File: Sound/Sound.kicad_pcb (KiCad board)
At the start: 2 copper layers, 295 x 300 mm, 18 parts, among them SW1 SW_DIP_x04, U1 7404

Commit message: new photos
Parts:
- moved C2 9.82 mm to (210.0, 287.5)
- moved R406 8.15 mm to (430.4, 311.1)
- moved R405 8.15 mm to (430.4, 308.0)
- moved R407 8.15 mm to (430.4, 314.3)
- moved C107 8.07 mm to (192.5, 315.5), turned to 90 degrees
- moved C108 5.39 mm to (203.5, 315.5), turned to 90 degrees
- moved SW1 4.24 mm to (198.9, 304.0)
- moved U1 3.78 mm to (253.8, 304.0)
- moved C109 2.70 mm to (399.5, 322.5)
- moved C1 2.50 mm to (192.5, 305.0)
- moved C110 1.05 mm to (411.0, 322.7)
- renumbered C4 to C107, C3 to C108, C5 to C109, C6 to C110
Other:
- board size 295 x 300 mm -> 300 x 300 mm
