File: Sound/Sound.kicad_sch (KiCad schematic)
At the start: 19 parts, among them J1 Conn_02x18_Counter_Clockwise, SW1 SW_DIP_x04, U1 7404

Commit message: new photos
Parts:
- renumbered C4 to C107, C3 to C108, C5 to C109, C6 to C110
Changed lines of the file:
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@@
   (symbol (lib_id "Device:C_Polarized") (at 132.08 352.425 0) (unit 1)
     (in_bom yes) (on_board yes) (dnp no) (fields_autoplaced)
-    (property "Reference" "C4" (at 135.89 350.266 0)
+    (property "Reference" "C107" (at 135.89 350.266 0)
       (effects (font (size 1.27 1.27)) (justify left))
     )
@@
       (project "Sound"
         (path "/a407fd57-8838-4f19-a49b-e173f62ac1a7"
-          (reference "C4") (unit 1)
+          (reference "C107") (unit 1)
         )
       )
@@
   (symbol (lib_id "Device:C_Polarized") (at 391.16 379.73 0) (unit 1)
     (in_bom yes) (on_board yes) (dnp no) (fields_autoplaced)
-    (property "Reference" "C5" (at 394.97 377.571 0)
+    (property "Reference" "C109" (at 394.97 377.571 0)
       (effects (font (size 1.27 1.27)) (justify left))
     )
@@
       (project "Sound"
         (path "/a407fd57-8838-4f19-a49b-e173f62ac1a7"
-          (reference "C5") (unit 1)
+          (reference "C109") (unit 1)
         )
       )
@@
   (symbol (lib_id "Device:C_Polarized") (at 402.59 380.365 0) (unit 1)
     (in_bom yes) (on_board yes) (dnp no) (fields_autoplaced)
-    (property "Reference" "C6" (at 406.4 378.206 0)
+    (property "Reference" "C110" (at 406.4 378.206 0)
       (effects (font (size 1.27 1.27)) (justify left))
     )
@@
       (project "Sound"
         (path "/a407fd57-8838-4f19-a49b-e173f62ac1a7"
-          (reference "C6") (unit 1)
+          (reference "C110") (unit 1)
         )
       )
@@
   (symbol (lib_id "Device:C_Polarized") (at 143.51 353.06 0) (unit 1)
     (in_bom yes) (on_board yes) (dnp no) (fields_autoplaced)
-    (property "Reference" "C3" (at 147.32 350.901 0)
+    (property "Reference" "C108" (at 147.32 350.901 0)
       (effects (font (size 1.27 1.27)) (justify left))
     )
@@
       (project "Sound"
         (path "/a407fd57-8838-4f19-a49b-e173f62ac1a7"
-          (reference "C3") (unit 1)
-        )
-      )
+          (reference "C108") (unit 1)
+        )
+      )
