File: Main/Main.kicad_sch (KiCad schematic)
At the start: 8 parts, among them U20 74LS192, U21 74LS192, U26 NE555P

Commit message: page 25
Parts:
- added AE1: Antenna, symbol Device:Antenna
- added C12: 0.01m, symbol Device:C_Polarized_US
- added C14: 47, symbol Device:C_Polarized_US
- added C15: 0.1m, symbol Device:C_Polarized_US
- added C19: 470m, symbol Device:C_Polarized
- added C24: 100m, symbol Device:C_Polarized_US
- added C27: 1000p, symbol Device:C
- added C3: TILT SW., symbol Device:C
- added C4: 470p, symbol Device:C_Polarized_US
- added D1: SiB01-02, Diode_THT:D_DO-35_SOD27_P7.62mm_Horizontal, symbol Device:D
- added D2: D, symbol Device:D
- added R13, R8, R9: 47k, symbol Device:R_US
- added R14, R3: 220, symbol Device:R_US
- added R4: R_US, symbol Device:R_US
- added R7: 100k, symbol Device:R_US
- added RA1: 560, symbol Device:R_US
- added RA2: 100, symbol Device:R_US
- added SW1: 1COIN 1PLAY/1COIN 2PLAY, symbol Switch:SW_SPDT
- added SW2: CREDIT, symbol Switch:SW_SPDT
- added SW3: TEST, symbol Switch:SW_SPDT
- added SW4: COIN, symbol Switch:SW_SPDT
- added U1: 74HC123, Package_DIP:DIP-16_W7.62mm, symbol 74xx:74HC123
- added U12: 74HC00, Package_DIP:DIP-14_W7.62mm, symbol 74xx:74HC00
- added U125: 74LS11, Package_DIP:DIP-14_W7.62mm, symbol 74xx:74LS11
- added U22: 74LS08, Package_DIP:DIP-14_W7.62mm, symbol 74xx:74LS08
- added U32: 74HC279, Package_DIP:DIP-16_W7.62mm, symbol 74xxMissing:74HC279
- added U37: 74LS74, Package_DIP:DIP-14_W7.62mm, symbol 74xx:74LS74
- added U38, U49: 74HC123, symbol 74xx:74HC123
- added U44: 74AHC04, Package_DIP:DIP-14_W7.62mm, symbol 74xx:74AHC04
- added U50: 74HC74, Package_DIP:DIP-14_W7.62mm, symbol 74xx:74HC74
- added U55, U61: 74LS32, Package_DIP:DIP-14_W7.62mm, symbol 74xx:74LS32
- added U73: 74AHC04, symbol 74xx:74AHC04
- added U74: 74LS27, Package_DIP:DIP-14_W7.62mm, symbol 74xx:74LS27
- added U79: 74LS393, symbol 74xx:74LS393
- added U85: 74LS11, symbol 74xx:74LS11
- U20, U21: footprint (none) -> Package_DIP:DIP-16_W7.62mm
Connections:
- net GNDPWR: now also U20.1 (B), U20.10 (C), U20.8 (GND), U21.8 (GND), C12.2, C14.2, C27.2, C3.2, C4.2, SW2.2 (B), SW3.2 (B), SW4.2 (B), U12.14 (VCC), U125.7 (GND), U22.7 (GND), U32.8 (GND), U37.7 (GND), U44.7 (GND), U50.7 (GND), U55.14 (VCC), U61.7 (GND)
- net VCC: now also U20.15 (A), U20.16 (VCC), U20.5 (UP), U20.9 (D), U21.16 (VCC), U21.5 (UP), D2.2 (A), R13.1, R4.1, R7.2, R8.1, R9.1, RA1.2, U1.2 (B), U1.3 (Clr), U37.2 (D), U37.4 (~{S}), U38.11 (Clr), U49.2 (B), U49.3 (Clr), U50.12 (D), U50.14 (VCC), U50.2 (D)
- net at U20.11 (~{LOAD}), U21.11 (~{LOAD}): now also U22.12
- net at U21.13 (~{BO}): now also U20.4 (DOWN)
- net at U21.14 (CLR): now also U20.14 (CLR), U74.9
- net at U21.4 (DOWN): now also U22.6
- net at U26.3 (Q): now also U22.4
- net at U26.4 (R): now also U37.9 (Q)
- net at U20.13 (~{BO}): now also U22.5, U55.5, U61.13
- new net: U37.12 (D), U37.5 (Q)
- new net: U22.13, U37.1 (~{R}), U37.13 (~{R}), U38.9 (A), U74.8
- new net: C19.1, R9.2, U1.15 (RCext)
- new net: C12.1, C14.1, R7.1, RA2.2, U1.1 (A)
- new net: R14.1, U44.8
- new net: C27.1, R14.2
- new net: R4.2, SW1.1 (A)
- new net: SW1.2 (B), U125.3
- new net: SW1.3 (C), U32.9 (Q)
- new net: R3.2, U12.8
- new net: U12.9, U32.11 (~{S1})
- new net: D2.1 (K), R3.1
- new net: C4.1, U79.1 (CP)
- new net: U55.9, U73.3, U79.2 (MR)
- new net: U55.13, U79.3 (Q0)
- new net: U125.5, U32.7 (Q)
- new net: U125.6, U37.3 (C)
- new net: U55.11, U55.2
- new net: U32.2 (~{S1}), U32.3 (~{S2})
- new net: C19.2, U1.14 (Cext)
- new net: C15.1, R8.2, U38.7 (RCext)
- new net: U61.11, U74.10
- new net: C24.1, R13.2, U49.15 (RCext)
- new net: D1.2 (A), RA1.1, RA2.1
- new net: C24.2, U49.14 (Cext)
- new net: C15.2, U38.6 (Cext)
- new net: AE1.1 (A), C3.1, D1.1 (K)
- new net: U44.9, U50.10 (~{S}), U55.6
- new net: U22.11, U50.1 (~{R}), U50.13 (~{R})
- new net: U38.10 (B), U50.9 (Q)
- new net: U50.5 (Q), U61.12
- new net: U50.6 (~{Q}), U55.4
- new net: U49.13 (Q), U85.2
- new net 8000: U79.6 (Q3)
- new net ACCEST: U37.11 (C)
- new net CAR_CONT_CL: U55.8
- new net EXTEND: U50.8 (~{Q})
- new net FX.SIGNAL: U49.4 (~{Q})
- new net GAME_OVER: U74.11
- no-connect marks 0 -> 2
Other:
- moved on the sheet: C1, R1, R2, RV1

Commit message: page 26 start
Parts:
- added C10, C11, C6, C7, C8, C9: 0.1m, symbol Device:C
- added C25: 1000p, symbol Device:C_Polarized_US
- added R15: 220, symbol Device:R_US
- added RA10, RA12, RA14, RA16, RA6, RA8: 100, symbol Device:R_US
- added RA11, RA13, RA15, RA5, RA7, RA9: 560, symbol Device:R_US
- added U10, U11, U17, U18: 74LS85, Package_DIP:DIP-16_W7.62mm, symbol 74xx:74LS85
- added U13: 74LS07, Package_DIP:DIP-14_W7.62mm, symbol 74xx:74LS07
- added U16: 74LS86, Package_DIP:DIP-14_W7.62mm, symbol 74xx:74LS86
- added U19, U5: 74LS393, Package_DIP:DIP-14_W7.62mm, symbol 74xx:74LS393
- added U24, U25: 74LS193, Package_DIP:DIP-16_W7.62mm, symbol 74xx:74LS193
- added U27: 74HC279, Package_DIP:DIP-16_W7.62mm, symbol 74xxMissing:74HC279
- added U33: 74LS74, Package_DIP:DIP-14_W7.62mm, symbol 74xx:74LS74
- added U4: 74LS151, Package_DIP:DIP-16_W7.62mm, symbol 74xx:74LS151
- added U8, U9: 74HC00, Package_DIP:DIP-14_W7.62mm, symbol 74xx:74HC00
- U38, U49: footprint (none) -> Package_DIP:DIP-16_W7.62mm
- U73, U79, U85: footprint (none) -> Package_DIP:DIP-14_W7.62mm
Connections:
- net GNDPWR: now also C10.2, C11.2, C25.2, C6.2, C7.2, C8.2, C9.2, U10.8 (GND), U11.1 (B3), U11.11 (B1), U11.14 (B2), U11.8 (GND), U11.9 (B0), U24.14 (CLR), U24.8 (GND), U25.1 (B), U25.10 (C), U25.14 (CLR), U25.15 (A), U25.8 (GND), U25.9 (D), U33.12 (D)
- net VCC: now also RA11.2, RA5.2, RA7.2, RA9.2, U10.1 (B3), U10.15 (A3), U10.16 (VCC), U11.16 (VCC), U11.2 (Ia<b), U11.3 (Ia=b), U11.4 (Ia>b), U16.1, U16.13, U17.1 (B3), U17.15 (A3), U17.2 (Ia<b), U17.4 (Ia>b), U18.2 (Ia<b), U18.4 (Ia>b), U24.1 (B), U24.10 (C), U24.15 (A), U24.16 (VCC), U24.7 (QD), U24.9 (D), U25.16 (VCC), U4.16 (VCC)
- net at SW1.2 (B), U125.3: now also U33.11 (C)
- net at U55.9, U73.3, U79.2 (MR): now also U73.2
- net at U55.13, U79.3 (Q0): now also U73.13
- net at U73.12: now also R15.1
- net at SW3.1 (A): now also RA13.1, RA14.1
- net at SW3.3 (C): now also RA11.1, RA12.1
- net at U125.4: now also U32.4 (Q)
- net at U125.5, U32.7 (Q): now also U33.10 (~{S})
- net at U55.1: now also C25.1, R15.2
- net at U55.3: now also U49.1 (A), U50.3 (C)
- net at U1.13 (Q): now also U20.14 (CLR), U21.14 (CLR), U74.9
- net INI.RESET: now reaches U1.4 (~{Q})
- net INI.RESET: now also U33.13 (~{R})
- net at U32.10 (~{R}): now also C7.1, RA8.2
- net COIN&TEST: now reaches U73.4
- net at SW2.1 (A): now also RA5.1, RA6.1
- net at SW2.3 (C): now also RA7.1, RA8.1
- net at U32.5 (~{R}): now also C8.1, RA10.2
- net at U32.6 (~{S}): now also C11.1, RA16.2
- net at SW4.1 (A): now also RA15.1, RA16.1
- net at SW4.3 (C): now also RA10.1, RA9.1
- new net: U24.11 (~{LOAD}), U25.11 (~{LOAD})
- new net: U24.5 (UP), U25.12 (~{CO})
- new net: U24.4 (DOWN), U25.13 (~{BO})
- new net: U11.12 (A1), U18.11 (B1), U25.2 (QB)
- new net: U11.10 (A0), U18.9 (B0), U25.3 (QA)
- new net: U11.13 (A2), U18.14 (B2), U25.6 (QC)
- new net: U11.15 (A3), U18.1 (B3), U25.7 (QD)
- new net: C6.1, RA6.2
- new net: U13.13, U16.11
- new net: U16.12, U16.2, U4.7 (~{E})
- new net: U4.5 (Z), U9.10
- new net: U13.11, U9.8
- new net: C9.1, RA12.2
- new net: U10.12 (A1), U17.11 (B1), U24.2 (QB)
- new net: U10.10 (A0), U17.9 (B0), U24.3 (QA)
- new net: U10.13 (A2), U17.14 (B2), U24.6 (QC)
- new net: U4.1 (I3), U4.2 (I2), U5.4 (Q1)
- new net: U10.11 (B1), U4.10 (S1)
- new net: U10.9 (B0), U4.11 (S0)
- new net: U4.12 (I7), U4.13 (I6), U5.6 (Q3)
- new net: U4.14 (I5), U4.15 (I4), U5.5 (Q2)
- new net: U4.3 (I1), U4.4 (I0), U5.3 (Q0)
- new net: U10.14 (B2), U4.9 (S2)
- new net: U17.10 (A0), U19.11 (Q0)
- new net: U17.12 (A1), U19.10 (Q1)
- new net: U17.13 (A2), U19.9 (Q2)
- new net: U17.3 (Ia=b), U18.6 (Oa=b)
- new net: C10.1, RA14.2
- new net: U19.12 (MR), U19.2 (MR)
- new net: U18.10 (A0), U19.3 (Q0)
- new net: U18.12 (A1), U19.4 (Q1)
- new net: U18.13 (A2), U19.5 (Q2)
- new net: U18.15 (A3), U19.13 (CP), U19.6 (Q3)
- new net: U10.4 (Ia>b), U11.5 (Oa>b)
- new net: U10.3 (Ia=b), U11.6 (Oa=b)
- new net: U10.2 (Ia<b), U11.7 (Oa<b)
- new net ACCI.: U16.3
- new net S-ACCE A: U13.8
- new net S-ACCE B: U13.6
- new net S-ACCE C: U13.4
- new net S-ACCE D: U13.2
- new net S-ACCI.: U13.12
- new net SCORE CP.: U13.10
- new net SCORE ST.: U9.9
- no-connect marks 2 -> 8
Other:
- note added: "25"
- note added: "26"
- note added: "27"
- note added: "28"
- moved on the sheet: SW2, SW3, SW4, U125B, U32A, U32B, U32C, U37A, U49C, U73A, U73F, U85B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

Commit message: first page almost done
Parts:
- removed C19: 470m, symbol Device:C_Polarized
- removed RA1, RA11, RA13, RA15, RA5, RA7, RA9: 560, symbol Device:R_US
- removed RA10, RA12, RA14, RA16, RA2, RA6, RA8: 100, symbol Device:R_US
- removed U1: 74HC123, Package_DIP:DIP-16_W7.62mm, symbol 74xx:74HC123
- removed U61: 74LS32, Package_DIP:DIP-14_W7.62mm, symbol 74xx:74LS32
- added C19: 470m, Capacitor_THT:CP_Radial_D10.0mm_P5.00mm, symbol Device:C_Polarized_US
- added IC28: 74LS10, Package_DIP:DIP-14_W7.62mm, symbol 74xx:74LS10
- added IC29, IC31: HD7417P, Package_DIP:DIP-14_W7.62mm, symbol 74xx:74HC7014
- added IC61, IC72: 74HC02, Package_DIP:DIP-14_W7.62mm, symbol 74xx:74HC02
- added IC67: 7450, Package_DIP:DIP-14_W7.62mm, symbol 74xxMissing:7450
- added L1: COIN METER, Diode_THT:D_DO-41_SOD81_P12.70mm_Horizontal, symbol Device:L
- added R1: 560, Resistor_THT:R_Axial_DIN0309_L9.0mm_D3.2mm_P12.70mm_Horizontal, symbol Device:R_US
- added R6: 1k, Resistor_THT:R_Axial_DIN0309_L9.0mm_D3.2mm_P12.70mm_Horizontal, symbol Device:R_US
- added RA1: R_Network08_US, Resistor_THT:R_Array_SIP9, symbol Device:R_Network08_US
- added RA2: R_Network07, Resistor_THT:R_Array_SIP8, symbol Device:R_Network07_US
- added TR1: Q_NPN_BEC, Package_TO_SOT_THT:TO-126-3_Vertical, symbol Device:Q_NPN_BCE
- AE1: footprint (none) -> Symbol:Symbol_ESD-Logo_CopperTop
- C10, C11, C12, C14, C15, C25, C27, C6, C7, C8, C9: footprint (none) -> Capacitor_THT:C_Disc_D9.0mm_W2.5mm_P5.00mm
- C24: footprint (none) -> Capacitor_THT:CP_Radial_D10.0mm_P5.00mm
- C3: footprint (none) -> Capacitor_THT:C_Disc_D4.3mm_W1.9mm_P5.00mm
- C4: renamed from C2; value C_Polarized -> 0.1u; footprint (none) -> Capacitor_THT:CP_Radial_Tantal_D4.5mm_P2.50mm; symbol Device:C_Polarized -> Device:C_Polarized_US
- C41: renamed from C4; footprint (none) -> Capacitor_THT:C_Disc_D9.0mm_W2.5mm_P5.00mm
- C5: renamed from C1; value C_Polarized -> 77u; footprint (none) -> Capacitor_THT:CP_Radial_Tantal_D4.5mm_P2.50mm; symbol Device:C_Polarized -> Device:C_Polarized_US
- D1: footprint Diode_THT:D_DO-35_SOD27_P7.62mm_Horizontal -> Diode_THT:D_DO-41_SOD81_P12.70mm_Horizontal
- D2: footprint (none) -> Diode_THT:D_DO-41_SOD81_P12.70mm_Horizontal
- R13, R14, R15, R3, R7, R8, R9: footprint (none) -> Resistor_THT:R_Axial_DIN0309_L9.0mm_D3.2mm_P12.70mm_Horizontal
- R22: renamed from R4; value R_US -> 1k; footprint (none) -> Resistor_THT:R_Axial_DIN0309_L9.0mm_D3.2mm_P12.70mm_Horizontal
- R4: renamed from R1; footprint (none) -> Resistor_THT:R_Axial_DIN0309_L9.0mm_D3.2mm_P12.70mm_Horizontal
- R5: renamed from R2; footprint (none) -> Resistor_THT:R_Axial_DIN0309_L9.0mm_D3.2mm_P12.70mm_Horizontal
- RV1: footprint (none) -> Potentiometer_THT:Potentiometer_Bourns_3386C_Horizontal
- SW1: footprint (none) -> Button_Switch_THT:SW_Slide_1P2T_CK_OS102011MS2Q
- SW2, SW3, SW4: footprint (none) -> TestPoint:TestPoint_Pad_1.0x1.0mm
- renumbered U10 to IC10, U11 to IC11, U12 to IC12, U125 to IC125, U13 to IC13, U16 to IC16, U17 to IC17, U18 to IC18, U19 to IC19, U20 to IC20, U21 to IC21, U22 to IC22, U24 to IC24, U25 to IC25, U26 to IC26, U27 to IC27, U32 to IC32, U33 to IC33, U37 to IC37, U38 to IC38, U4 to IC4, U44 to IC44, U49 to IC49, U5 to IC5, U50 to IC50, U55 to IC55, U73 to IC73, U74 to IC74, U79 to IC79, U9 to IC8, U8 to IC8, U85 to IC85
Connections:
- net INI.RESET is gone; now on net ~{INI. RESET} (B): IC33.13 (~{R})
- net GNDPWR: now also IC19.7 (GND), IC33.7 (GND), IC38.8 (GND), IC49.8 (GND), IC55.7 (GND), IC74.7 (GND), IC79.7 (GND), IC8.7 (GND), IC85.7 (GND), IC28.7 (GND), IC67.7 (GND); no longer IC55.14 (VCC)
- net VCC: now also IC12.7 (GND), IC125.14 (VCC), IC22.14 (VCC), IC32.16 (VCC), IC33.14 (VCC), IC37.14 (VCC), IC38.16 (VCC), IC38.2 (B), IC38.3 (Clr), IC44.14 (VCC), IC49.16 (VCC), IC74.14 (VCC), IC79.14 (VCC), IC85.14 (VCC), L1.1, R6.1, RA1.1 (common)
- net COIN IN (B): now reaches IC37.12 (D), IC37.5 (Q)
- net COIN IN (B): now also IC72.9
- net ~{GAME} (B): now reaches IC37.8 (~{Q})
- net ~{GAME} (B): now also IC55.13, IC31.9
- net at IC26.4 (R), IC37.9 (Q): now also IC31.5
- net at R9.2: now also IC38.15 (RCext), C19.1
- net at IC125.5, IC32.7 (Q), IC33.10 (~{S}): now also IC44.5
- net at IC33.8 (~{Q}): now also IC72.8
- net at C12.1, C14.1, R7.1: now also IC38.1 (A)
- net at C27.1, R14.2: now also IC61.6
- net Vs/16: now reaches IC12.10
- net Vs/16: now also IC85.1
- net at IC12.9, IC32.11 (~{S1}): now also IC72.10
- net at IC10.12 (A1), IC17.11 (B1), IC24.2 (QB): now also IC28.3
- net at IC10.10 (A0), IC17.9 (B0), IC24.3 (QA): now also IC28.4
- net at IC10.13 (A2), IC17.14 (B2), IC24.6 (QC): now also IC28.5
- net S-100-O: now reaches C41.1, IC79.1 (CP)
- net S-100-O: now also R6.2
- net at IC73.13, IC79.3 (Q0): now also IC55.12; no longer IC55.13
- net at IC73.8: now also IC67.13 (1B)
- net at IC73.9: now also IC67.10 (1D)
- net at IC73.1: now also IC125.6, IC20.11 (~{LOAD}), IC21.11 (~{LOAD}), IC22.12, IC37.3 (C), IC31.3
- net ~{EX.SIG???.??} (M): now reaches IC49.1 (A), IC50.3 (C), IC55.3
- net at IC20.14 (CLR), IC21.14 (CLR), IC74.9: now also IC38.13 (Q), IC31.1
- net at IC74.10: now also IC61.13
- net at IC55.10: now also IC61.4
- net at IC73.5: now also IC67.3 (2B)
- net at IC73.6: now also IC67.5 (2D)
- net at IC44.9, IC50.10 (~{S}), IC55.6: now also IC61.5
- net at IC44.6: now also R1.1
- net EXTEND (C): now reaches IC38.10 (B), IC50.9 (Q)
- net ~{COIN IN} (B): now reaches IC37.6 (~{Q})
- net ~{COIN IN} (B): now also IC31.11
- net at IC27.2 (~{S1}): now also IC28.6
- net at IC50.5 (Q): now also IC61.12
- net at IC20.13 (~{BO}), IC22.5, IC55.5: now also IC61.11
- net at IC5.1 (CP): now also IC67.6 (2Y)
- net at IC38.14 (Cext): now also C19.2
- net ~{INI. RESET} (B): now reaches IC38.4 (~{Q})
- net at IC85.12: now also IC29.13
- net V2: now reaches IC85.13
- net at IC38.12 (~{Q}): now also IC31.13
- net CAR_CONT_CL renamed CAR.CONT.CL (4)
- net COIN&TEST renamed ~{COIN&TEST} (F)
- net EXTEND renamed ~{EXTEND} (C)
- net FX.SIGNAL renamed ~{FX.SIGNAL} (B)
- new net: R1.2, TR1.1 (B)
- new net: L1.2, TR1.2 (C)
- new net EV.CP (S): IC29.12
- new net GAME (I): IC31.6
- new net MUTE (S): IC31.2
- new net RET1: TR1.3 (E)
- new net V6: IC67.1 (1A), IC67.2 (2A)
- new net V7: IC67.4 (2C), IC67.9 (1C)
- new net ~{COIN IN} (S): IC31.10
- new net ~{COIN&TEST} (I): IC31.4
- new net ~{GAME} (S): IC31.8
- new net ~{HISCORE} (S): IC31.12
- no-connect marks 8 -> 15
Other:
- moved on the sheet: IC33A, IC33C, IC38A, IC44C, IC50C, IC73C, IC73D, IC73E, IC73G

Commit message: stuff
Parts:
- added J1: Conn_01x36_Pin, BoardEdge:MainA, symbol Connector:Conn_01x36_Pin
Connections:
- net GNDPWR: now also J1.1 (Pin_1), J1.2 (Pin_2), J1.3 (Pin_3), J1.4 (Pin_4), J1.5 (Pin_5)
- net VCC: now also J1.33 (Pin_33), J1.34 (Pin_34), J1.35 (Pin_35), J1.36 (Pin_36)
Other:
- moved on the sheet: IC72D

Commit message: more page 2
Parts:
- removed C10, C11, C6, C7, C8, C9: 0.1m, Capacitor_THT:C_Disc_D9.0mm_W2.5mm_P5.00mm, symbol Device:C
- added C10, C7: 0.1u, Capacitor_THT:C_Disc_D7.5mm_W5.0mm_P7.50mm, symbol Device:C_Polarized_US
- added C31, C32: 100m, Capacitor_THT:CP_Radial_D10.0mm_P5.00mm, symbol Device:C_Polarized_US
- added Cp1, Cp10, Cp11, Cp12, Cp13, Cp14, Cp15, Cp16, Cp17, Cp18, Cp19, Cp2, Cp20, Cp3, Cp4, Cp5, Cp6, Cp7, Cp8, Cp9: 100n, Capacitor_THT:C_Disc_D7.5mm_W5.0mm_P7.50mm, symbol Device:C
- added IC14: 74LS20, Package_DIP:DIP-14_W7.62mm, symbol 74xx:74LS20
- added IC15, IC35, IC36: 74LS193, Package_DIP:DIP-16_W7.62mm, symbol 74xx:74LS193
- added IC2, IC34: 74LS08, Package_DIP:DIP-14_W7.62mm, symbol 74xx:74LS08
- added IC23: 74LS32, Package_DIP:DIP-14_W7.62mm, symbol 74xx:74LS32
- added IC30, IC68: 74LS00, Package_DIP:DIP-14_W7.62mm, symbol 74xx:74LS00
- added IC39, IC40: 74LS393, Package_DIP:DIP-14_W7.62mm, symbol 74xx:74LS393
- added IC41, IC42, IC7: 74LS85, Package_DIP:DIP-16_W7.62mm, symbol 74xx:74LS85
- added IC60: 74LS157, Package_DIP:DIP-16_W7.62mm, symbol 74xx:74LS157
- added IC69, IC9: 74LS153, Package_DIP:DIP-16_W7.62mm, symbol 74xx:74LS153
- C12, C25, C27, C41: footprint Capacitor_THT:C_Disc_D9.0mm_W2.5mm_P5.00mm -> Capacitor_THT:C_Disc_D7.5mm_W5.0mm_P7.50mm
- C14: footprint Capacitor_THT:C_Disc_D9.0mm_W2.5mm_P5.00mm -> Capacitor_THT:CP_Radial_Tantal_D8.0mm_P5.00mm
- C15: footprint Capacitor_THT:C_Disc_D9.0mm_W2.5mm_P5.00mm -> Capacitor_THT:CP_Radial_Tantal_D4.5mm_P5.00mm
- C3: footprint Capacitor_THT:C_Disc_D4.3mm_W1.9mm_P5.00mm -> Capacitor_THT:C_Disc_D7.5mm_W5.0mm_P7.50mm
- C4: footprint Capacitor_THT:CP_Radial_Tantal_D4.5mm_P2.50mm -> Capacitor_THT:C_Disc_D7.5mm_W5.0mm_P7.50mm
- TR1: footprint Package_TO_SOT_THT:TO-126-3_Vertical -> Package_TO_SOT_THT:TO-126-3_Horizontal_TabDown
Connections:
- net GNDPWR: now also IC17.8 (GND), IC18.8 (GND), C10.2, C7.2, Cp1.1, Cp10.1, Cp11.1, Cp12.1, Cp13.1, Cp14.1, Cp15.1, Cp16.1, Cp17.1, Cp18.1, Cp19.1, Cp2.1, Cp20.1, Cp3.1, Cp4.1, Cp5.1, Cp6.1, Cp7.1, Cp8.1, Cp9.1, IC15.1 (B), IC15.10 (C), IC15.15 (A), IC15.8 (GND), IC15.9 (D), IC35.1 (B), IC35.10 (C), IC35.14 (CLR), IC35.15 (A), IC35.8 (GND), IC35.9 (D), IC36.14 (CLR), IC36.8 (GND), IC41.8 (GND), IC42.8 (GND), IC69.1 (Ea), IC69.12 (I2b), IC69.15 (Eb), IC69.4 (I2a), IC7.8 (GND), IC9.1 (Ea), IC9.15 (Eb), IC9.6 (I0a), IC9.8 (GND)
- net VCC: now also IC33.4 (~{S}), RA2.1 (common), Cp1.2, Cp10.2, Cp11.2, Cp12.2, Cp13.2, Cp14.2, Cp15.2, Cp16.2, Cp17.2, Cp18.2, Cp19.2, Cp2.2, Cp20.2, Cp3.2, Cp4.2, Cp5.2, Cp6.2, Cp7.2, Cp8.2, Cp9.2, IC35.16 (VCC), IC36.1 (B), IC36.10 (C), IC36.15 (A), IC36.16 (VCC), IC36.9 (D), IC41.2 (Ia<b), IC41.4 (Ia>b), IC42.16 (VCC), IC42.2 (Ia<b), IC42.3 (Ia=b), IC42.4 (Ia>b), IC7.10 (A0), IC7.16 (VCC), IC7.2 (Ia<b), IC7.3 (Ia=b), IC7.4 (Ia>b), IC7.9 (B0); no longer RA1.1 (common)
- net at IC72.11: now also IC16.12, IC16.2, IC4.7 (~{E}), IC23.3
- net SP DOWN (G): now reaches IC72.12
- net at IC72.13: now also IC67.10 (1D), IC73.9
- net at IC24.11 (~{LOAD}), IC25.11 (~{LOAD}): now also IC35.11 (~{LOAD}), IC36.11 (~{LOAD})
- net at IC27.10 (~{R}): now also IC44.12
- net at IC27.11 (~{S1}): now also IC14.6
- net at IC27.9 (Q): now also IC16.10
- net A23: now reaches J1.23 (Pin_23)
- net A23: now also RA1.8 (R7), SW4.3 (C)
- net A24: now reaches J1.24 (Pin_24)
- net A24: now also RA1.5 (R4), RA2.5 (R4), SW3.3 (C)
- net A32: now reaches J1.32 (Pin_32)
- net A32: now also SW2.3 (C)
- net at IC8.1: now also IC60.6 (I1b)
- net at IC8.3: now also IC15.4 (DOWN)
- net at IC13.5: now also IC14.4, IC15.2 (QB), IC7.12 (A1)
- net at RA1.2 (R1): now also RA2.8 (R7)
- net at RA1.6 (R5): now also RA2.4 (R3)
- net at RA1.7 (R6): now also RA2.3 (R2)
- net at IC16.8: now also IC60.1 (S)
- net at IC16.9: now also IC28.9, IC32.13 (Q)
- net at IC33.1 (~{R}): now also IC23.11
- net EXTEND (A): now reaches IC33.2 (D)
- net at IC33.3 (C): now also IC27.7 (Q), IC23.13, IC23.2
- net EXPLO.ST.(G): now reaches IC33.5 (Q)
- net EXPLO.ST.(G): now also IC23.1, IC69.2 (S1)
- net ~{EXPLO.ST.}(G): now reaches IC33.6 (~{Q})
- net ~{EXPLO.ST.}(G): now also IC39.2 (MR)
- net at IC13.3: now also IC14.1, IC15.6 (QC), IC7.13 (A2)
- net at IC44.13: now also IC28.8
- net at IC27.2 (~{S1}), IC28.6: now also IC27.3 (~{S2})
- net at IC44.1: now also IC27.4 (Q)
- net at IC44.2: now also IC23.10
- net at IC67.3 (2B), IC73.5: now also IC8.11
- net at IC29.1: now also IC2.3
- net A20: now reaches IC29.2
- net ~{HOME POS.} (G): now reaches IC27.5 (~{R})
- net ~{HOME POS.} (G): now also IC23.8
- net at IC22.1: now also IC23.6, IC34.4
- net at IC22.3: now also IC7.1 (B3)
- net at IC13.9: now also IC14.2, IC15.3 (QA)
- net at IC32.15 (~{S}): now also C7.1
- net at IC16.4: now also IC2.13, IC23.4
- net at IC16.6: now also IC23.5, IC7.11 (B1)
- net at IC8.4: now also IC60.4 (Za)
- net at IC8.5: now also IC7.7 (Oa<b)
- net at IC8.6: now also IC15.5 (UP)
- net ~{COIN&TEST}: now reaches IC28.10
- new net: IC9.11 (I1b), IC9.13 (I3b)
- new net: IC9.3 (I3a), IC9.5 (I1a)
- new net: IC30.9, IC9.7 (Za)
- new net: IC30.1, IC9.9 (Zb)
- new net: IC34.8, IC39.1 (CP)
- new net: IC23.12, IC34.9, IC68.6
- new net: IC40.10 (Q1), IC41.11 (B1)
- new net: IC40.11 (Q0), IC41.9 (B0)
- new net: IC40.13 (CP), IC40.6 (Q3), IC42.1 (B3)
- new net: IC40.8 (Q3), IC41.1 (B3)
- new net: IC40.9 (Q2), IC41.14 (B2)
- new net: IC30.10, IC30.11
- new net: IC30.8, IC36.5 (UP)
- new net: IC36.3 (QA), IC42.10 (A0)
- new net: IC40.4 (Q1), IC42.11 (B1)
- new net: IC36.2 (QB), IC42.12 (A1)
- new net: IC36.6 (QC), IC42.13 (A2)
- new net: IC40.5 (Q2), IC42.14 (B2)
- new net: IC36.7 (QD), IC42.15 (A3)
- new net: IC41.3 (Ia=b), IC42.6 (Oa=b)
- new net: IC40.3 (Q0), IC42.9 (B0)
- new net: IC69.10 (I0b), IC69.11 (I1b)
- new net: IC69.13 (I3b), IC69.3 (I3a)
- new net: IC69.5 (I1a), IC69.6 (I0a)
- new net: IC15.7 (QD), IC7.15 (A3)
- new net: IC34.5, IC60.7 (Zb)
- new net: IC30.3, IC36.4 (DOWN)
- new net: IC35.5 (UP), IC36.12 (~{CO})
- new net: IC35.4 (DOWN), IC36.13 (~{BO})
- new net: IC2.11, IC7.14 (B2)
- new net: IC35.2 (QB), IC41.12 (A1)
- new net: IC35.3 (QA), IC41.10 (A0)
- new net: IC30.13, IC35.6 (QC), IC41.13 (A2)
- new net: IC30.12, IC35.7 (QD), IC41.15 (A3)
- new net ACCE.ST: IC34.6
- new net EXPLO. SEL. A (G): IC39.3 (Q0)
- new net EXPLO. SEL. B (G): IC39.4 (Q1)
- new net EXPLO. SEL. C (G): IC39.5 (Q2), IC68.4
- new net EXPLO. SEL. D (G): IC39.6 (Q3), IC68.5, IC69.14 (S0)
- new net PL-V-ST.: IC41.6 (Oa=b)
- no-connect marks 15 -> 23
Other:
- moved on the sheet: IC16B, IC16C, IC22A, IC27B, IC27C, IC27D, IC28C, IC29A, IC31G, IC32D, IC33A, IC44A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
