File: Main/Main.kicad_sch (KiCad schematic)
At the start: 114 parts, among them IC10 74LS85, IC11 74LS85, IC12 74HC00, IC125 74LS11, IC13 74LS07, IC14 74LS20, IC15 74LS193, IC16 74LS86, IC17 74LS85, IC18 74LS85, IC19 74LS393, IC2 74LS08, IC20 74LS192, IC21 74LS192, IC22 74LS08, IC23 74LS32, IC24 74LS193, IC25 74LS193, IC26 NE555P, IC27 74HC279, IC28 74LS10, IC29 HD7417P, IC30 74LS00, IC31 HD7417P, IC32 74HC279, IC33 74LS74, IC34 74LS08, IC35 74LS193, IC36 74LS193, IC37 74LS74, IC38 74HC123, IC39 74LS393, IC4 74LS151, IC40 74LS393, IC41 74LS85, IC42 74LS85, IC44 74AHC04, IC49 74HC123, IC5 74LS393, IC50 74HC74, IC55 74LS32, IC60 74LS157, IC61 74HC02, IC67 7450, IC68 74LS00, IC69 74LS153, IC7 74LS85, IC72 74HC02, IC73 74AHC04, IC74 74LS27, IC79 74LS393, IC8 74HC00, IC85 74LS11, IC9 74LS153, J1 Conn_01x36_Pin, SW1 1COIN 1PLAY/1COIN 2PLAY, SW2 CREDIT, SW3 TEST, SW4 COIN

Commit message: page 2 almost
Parts:
- removed C3: TILT SW., Capacitor_THT:C_Disc_D7.5mm_W5.0mm_P7.50mm, symbol Device:C
- added C1, C2: 4.7m, Capacitor_THT:CP_Radial_Tantal_D4.5mm_P2.50mm, symbol Device:C_Polarized_US
- added C17, C3: 470p, Capacitor_THT:C_Disc_D4.3mm_W1.9mm_P5.00mm, symbol Device:C_Polarized_US
- added C18: 15u, Capacitor_THT:CP_Radial_Tantal_D4.5mm_P2.50mm, symbol Device:C_Polarized_US
- added C20: 10u, Capacitor_THT:CP_Radial_Tantal_D4.5mm_P2.50mm, symbol Device:C_Polarized_US
- added C21: 22m, Capacitor_THT:CP_Radial_Tantal_D4.5mm_P2.50mm, symbol Device:C_Polarized_US
- added Cp21, Cp22, Cp23, Cp24, Cp25, Cp26, Cp27, Cp28, Cp29, Cp30, Cp31, Cp32, Cp33, Cp34, Cp35, Cp36, Cp37, Cp38, Cp39: 100n, Capacitor_THT:C_Disc_D7.5mm_W5.0mm_P7.50mm, symbol Device:C
- added Cp40: 100n, Capacitor_THT:CP_Radial_D10.0mm_P5.00mm, symbol Device:C
- added IC1, IC43: 74LS123, Package_DIP:DIP-16_W7.62mm, symbol 74xx:74LS123
- added IC3: 74LS153, Package_DIP:DIP-16_W7.62mm, symbol 74xx:74LS153
- added IC46, IC6: 74LS04, Package_DIP:DIP-14_W7.62mm, symbol 74xx:74LS04
- added IC47: 74LS20, Package_DIP:DIP-14_W7.62mm, symbol 74xx:74LS20
- added IC63: 74LS02, Package_DIP:DIP-14_W7.62mm, symbol 74xx:74LS02
- added IC66: 74LS08, Package_DIP:DIP-14_W7.62mm, symbol 74xx:74LS08
- added IC80: 74LS10, Package_DIP:DIP-14_W7.62mm, symbol 74xx:74LS10
- added R10, R11, R2, R3, R999: 47k, Resistor_THT:R_Axial_DIN0309_L9.0mm_D3.2mm_P12.70mm_Horizontal, symbol Device:R_US
- added SW5: TILT SW., Button_Switch_THT:SW_PUSH_6mm, symbol Switch:SW_SPST
- C25, C27: footprint Capacitor_THT:C_Disc_D7.5mm_W5.0mm_P7.50mm -> Capacitor_THT:C_Disc_D3.0mm_W1.6mm_P2.50mm
- C41: footprint Capacitor_THT:C_Disc_D7.5mm_W5.0mm_P7.50mm -> Capacitor_THT:C_Disc_D4.3mm_W1.9mm_P5.00mm
- D1: footprint Diode_THT:D_DO-41_SOD81_P12.70mm_Horizontal -> Diode_THT:D_DO-201AE_P15.24mm_Horizontal
- VR1: renamed from RV1; value R_Potentiometer_US -> 10k
- renumbered R3 to R998
Connections:
- net ACCEST is gone; now on net ACCE.ST: IC37.11 (C)
- net GNDPWR: now also IC13.7 (GND), IC14.7 (GND), IC16.7 (GND), IC2.7 (GND), IC23.7 (GND), IC27.8 (GND), IC29.7 (GND), IC30.7 (GND), IC31.7 (GND), IC34.7 (GND), IC39.7 (GND), IC5.7 (GND), IC60.15 (E), IC60.8 (GND), IC61.7 (GND), IC68.7 (GND), IC72.7 (GND), IC73.7 (GND), C17.2, C3.2, Cp21.1, Cp22.1, Cp23.1, Cp24.1, Cp25.1, Cp26.1, Cp27.1, Cp28.1, Cp29.1, Cp30.1, Cp31.1, Cp32.1, Cp33.1, Cp34.1, Cp35.1, Cp36.1, Cp37.1, Cp38.1, Cp39.1, Cp40.1, IC3.1 (Ea), IC3.10 (I0b), IC3.15 (Eb), IC3.6 (I0a), IC3.8 (GND), SW5.1 (A)
- net V6: now also IC47.10
- net V7: now also IC69.13 (I3b), IC69.3 (I3a), IC47.9
- net VCC: now also IC13.14 (VCC), IC14.14 (VCC), IC16.14 (VCC), IC19.14 (VCC), IC2.14 (VCC), IC23.14 (VCC), IC27.16 (VCC), IC28.14 (VCC), IC29.14 (VCC), IC34.14 (VCC), IC39.14 (VCC), IC5.14 (VCC), IC55.14 (VCC), IC60.16 (VCC), IC61.14 (VCC), IC67.14 (VCC), IC68.14 (VCC), IC72.14 (VCC), IC73.14 (VCC), IC8.14 (VCC), Cp21.2, Cp22.2, Cp23.2, Cp24.2, Cp25.2, Cp26.2, Cp27.2, Cp28.2, Cp29.2, Cp30.2, Cp31.2, Cp32.2, Cp33.2, Cp34.2, Cp35.2, Cp36.2, Cp37.2, Cp38.2, Cp39.2, Cp40.2, R10.1, R11.1, R2.1, R3.1, R999.1
- net Vs/16: now also IC60.2 (I0a)
- net ~{COIN&TEST}: now also IC28.11; no longer IC28.10
- net at IC9.10 (I0b): now also IC72.5, IC66.9
- net at IC9.11 (I1b), IC9.13 (I3b): now also IC3.9 (Zb)
- net at IC9.12 (I2b): now also IC66.8
- net at IC9.14 (S0): now also IC13.13, IC15.11 (~{LOAD}), IC16.11, IC28.10
- net at IC9.2 (S1): now also IC23.10, IC44.2
- net at IC9.3 (I3a), IC9.5 (I1a): now also IC3.7 (Za)
- net at IC9.4 (I2a): now also IC72.4
- net at IC16.12, IC16.2, IC4.7 (~{E})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: no longer IC23.3
- net A9: now reaches L1.2, TR1.2 (C)
- net Vs/8: now reaches IC60.6 (I1b), IC8.1
- net at IC40.12 (MR): now also IC40.2 (MR), C17.1, IC47.8
- net at IC13.5, IC14.4, IC15.2 (QB)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: now also IC6.5
- net at IC69.5 (I1a), IC69.6 (I0a): now also IC67.8 (1Y)
- net at IC74.3: now also IC68.11
- net at IC74.6: now also IC19.12 (MR), IC19.2 (MR), C3.1
- net ACCE D: now reaches IC13.1
- net ACCE D: now also IC6.12
- net at IC10.11 (B1), IC4.10 (S1): now also IC6.2
- net at IC10.9 (B0), IC4.11 (S0): now also IC6.6
- net at IC10.14 (B2), IC4.9 (S2): now also IC14.5, IC6.13, IC6.4
- net at IC13.3, IC14.1, IC15.6 (QC)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: now also IC6.3
- net PLAYER: now reaches IC44.10
- net PLAYER: now also IC49.10 (B), IC43.10 (B), IC43.2 (B), IC80.5
- net Vs/32: now reaches IC72.6
- net Vs/32: now also IC66.10
- net at IC23.9: now also IC30.2, IC46.2
- net ~{SP DOWN}: now reaches IC2.2
- net ~{SP DOWN}: now also IC2.12
- net at IC2.4: now also IC22.10
- net at IC2.5: now also IC1.5 (Q)
- net at IC2.6: now also IC3.11 (I1b)
- net at IC15.7 (QD), IC7.15 (A3): now also IC6.1
- net at IC34.1: now also IC80.6
- net ~{ACCI.PULSE}: now reaches IC34.2
- net at IC34.3: now also IC27.6 (~{S})
- net at AE1.1 (A), D1.1 (K): now also SW5.2 (B)
- net at IC19.1 (CP): now also IC18.3 (Ia=b), IC63.13
- net Vs/64: now reaches IC60.3 (I1a)
- net Vs/2: now reaches IC60.5 (I0b)
- net ~{BRIDGE(W)}: now reaches IC14.10
- net ROAD: now reaches IC14.12
- net ~{OTHER BODY}: now reaches IC14.13
- net at IC14.8: now also IC80.3
- net ~{RESCUE(Y)}: now reaches IC14.9
- net at IC35.2 (QB), IC41.12 (A1): now also IC47.4
- net at IC35.3 (QA), IC41.10 (A0): now also IC47.5
- net at IC30.13, IC35.6 (QC), IC41.13 (A2): now also IC47.2
- net at IC30.12, IC35.7 (QD), IC41.15 (A3): now also IC47.1
- net at IC49.11 (Clr): now also IC43.11 (Clr), IC43.3 (Clr)
- net at IC49.6 (Cext): now also C21.2
- net at IC49.7 (RCext): now also C21.1, R999.2
- net at IC49.9 (A): now also IC43.9 (A)
- net at IC22.8: now also IC3.5 (I1a)
- net at IC22.9: now also IC1.13 (Q)
- net at IC16.4, IC2.13, IC23.4: now also IC6.10
- net at IC16.5: now also IC6.8
- net at IC19.8 (Q3): now also IC63.11
- net GAME_OVER renamed B16
- net S-100-O renamed A30
- new net: IC1.1 (A), IC1.9 (A)
- new net: C2.2, IC1.14 (Cext)
- new net: C2.1, IC1.15 (RCext), R3.2
- new net: IC1.2 (B), IC3.3 (I3a)
- new net: IC1.12 (~{Q}), IC1.3 (Clr)
- new net: IC1.11 (Clr), IC1.4 (~{Q})
- new net: C1.1, IC1.7 (RCext), R2.2
- new net: C20.1, IC43.7 (RCext), R11.2
- new net: C18.1, IC43.15 (RCext), R10.2
- new net: C20.2, IC43.6 (Cext)
- new net: C1.2, IC1.6 (Cext)
- new net: IC46.1, IC47.6
- new net: C18.2, IC43.14 (Cext)
- new net: IC1.10 (B), IC3.13 (I3b)
- new net V4: IC47.13
- new net V5: IC47.12
- new net ~{ACCI.ST}: IC80.4
- no-connect marks 23 -> 32
Other:
- moved on the sheet: AE1, C10, C7, IC10, IC11, IC13A, IC13B, IC13C, IC13D, IC13E, IC13F, IC14A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

Commit message: first rom
Parts:
- added C22, C26, C39: 470p, Capacitor_THT:C_Disc_D4.3mm_W1.9mm_P5.00mm, symbol Device:C_Polarized_US
- added C6: C_Polarized_US, Capacitor_THT:C_Disc_D3.0mm_W1.6mm_P2.50mm, symbol Device:C_Polarized_US
- added IC119: 74LS123, Package_DIP:DIP-16_W7.62mm, symbol 74xx:74LS123
- added IC45: 74LS10, Package_DIP:DIP-14_W7.62mm, symbol 74xx:74LS10
- added IC48, IC56: 74HC00, Package_DIP:DIP-14_W7.62mm, symbol 74xx:74HC00
- added IC51: 74HC279, Package_DIP:DIP-16_W7.62mm, symbol 74xxMissing:74HC279
- added IC52, IC54: 74LS393, Package_DIP:DIP-14_W7.62mm, symbol 74xx:74LS393
- added IC53, IC58: 74LS85, Package_DIP:DIP-16_W7.62mm, symbol 74xx:74LS85
- added IC57: 74LS20, Package_DIP:DIP-14_W7.62mm, symbol 74xx:74LS20
- added IC59, IC71: MB7137, Package_DIP:DIP-24_W15.24mm, symbol Memory_PROM:MB7137
- added IC70: 74LS151, Package_DIP:DIP-16_W7.62mm, symbol 74xx:74LS151
- added J2: Conn_01x22, BoardEdge:MainB, symbol Connector_Generic:Conn_01x22
- added J3: Conn_01x28_Pin, BoardEdge:MainC, symbol Connector:Conn_01x28_Pin
- renumbered R999 to R12
Connections:
- net GNDPWR: now also C22.2, C26.2, C39.2, C6.2, IC53.8 (GND), IC59.12 (GND), IC59.21 (A10), IC59.22 (A9), IC59.23 (A8), IC70.8 (GND), IC71.12 (GND), IC71.20 (~{CE}1_(PVCE)), IC71.21 (A10), J3.25 (Pin_25), J3.26 (Pin_26), J3.27 (Pin_27), J3.28 (Pin_28)
- net VCC: now also IC53.16 (VCC), IC53.2 (Ia<b), IC53.4 (Ia>b), IC58.16 (VCC), IC58.2 (Ia<b), IC58.4 (Ia>b), IC59.24 (VCC_(PVCC)), IC71.18 (CE2), IC71.19 (CE3), IC71.24 (VCC_(PVCC)), J3.20 (Pin_20), J3.21 (Pin_21), J3.22 (Pin_22), J3.23 (Pin_23)
- net ~{ACCI.ST}: now also IC119.11 (Clr), IC51.7 (Q)
- net ~{HOME POS.} (G): now also IC51.5 (~{R})
- net at IC1.13 (Q): now also IC2.9; no longer IC22.9
- net at IC63.1: now also IC52.1 (CP)
- net at IC63.2: now also IC34.11
- net 7MHz: now reaches IC63.3
- net at IC34.12: now also IC46.5, IC52.8 (Q3), IC57.9, IC58.15 (A3)
- net at IC34.13: now also IC52.10 (Q1), IC57.12, IC57.4, IC58.12 (A1)
- net ~{ACC I.}: now reaches IC66.1
- net ~{ACC I.}: now also IC59.18 (CE2), IC59.19 (CE3)
- net at IC66.3: now also IC51.11 (~{S1})
- net H5: now reaches IC74.4
- net H8: now reaches IC74.5
- net at IC46.8: now also IC56.13, IC59.1 (A7)
- net at IC46.9: now also IC56.9, IC57.8
- net at IC2.4: now also IC2.10; no longer IC22.10
- net at IC63.4: now also IC54.1 (CP)
- net ~{H}s: now reaches IC63.5
- net at IC63.6: now also IC46.11, IC54.8 (Q3)
- net H4: now reaches IC68.12
- net H6: now reaches IC68.13
- net at IC43.13 (Q): now also IC61.3
- net at IC66.11: now also IC119.9 (A)
- net ~{GRAVEL}: now reaches IC66.12
- net ~{SLIDE}: now reaches IC66.13
- net at IC2.8: now also IC3.5 (I1a)
- net at IC22.8: no longer IC3.5 (I1a)
- net at IC46.6: now also IC57.2
- net at IC46.10: now also IC53.3 (Ia=b)
- net at IC46.3: now also IC48.2, IC54.9 (Q2), IC59.2 (A6)
- net at IC46.4: now also IC45.1
- net ~{SPLAY B}: now reaches IC49.5 (Q)
- net ~{SPLAY B}: now also IC48.10
- net at IC61.1: now also IC8.12
- net at IC61.2: now also IC43.5 (Q), IC48.9
- new net: IC45.10, IC51.13 (Q)
- new net: IC48.11, IC51.14 (~{R})
- new net: IC48.6, IC51.15 (~{S})
- new net: IC52.11 (Q0), IC58.10 (A0)
- new net: IC52.12 (MR), IC52.2 (MR)
- new net: IC52.9 (Q2), IC57.10, IC57.5, IC58.13 (A2)
- new net: IC45.9, IC56.5, IC57.6
- new net: IC45.13, IC48.1, IC48.12, IC48.4, IC54.11 (Q0), IC59.4 (A4)
- new net: IC52.3 (Q0), IC53.10 (A0)
- new net: IC52.4 (Q1), IC53.12 (A1)
- new net: IC52.5 (Q2), IC53.13 (A2)
- new net: IC52.6 (Q3), IC53.15 (A3)
- new net: IC53.11 (B1), IC59.10 (D1)
- new net: IC53.14 (B2), IC59.11 (D2)
- new net: IC53.1 (B3), IC59.13 (D3)
- new net: IC58.9 (B0), IC59.14 (D4)
- new net: IC58.11 (B1), IC59.15 (D5)
- new net: IC58.14 (B2), IC59.16 (D6)
- new net: IC58.1 (B3), IC59.17 (D7)
- new net: IC45.2, IC48.13, IC54.10 (Q1), IC59.3 (A5)
- new net: IC54.13 (CP), IC54.6 (Q3), IC59.5 (A3)
- new net: IC54.5 (Q2), IC59.6 (A2)
- new net: IC54.4 (Q1), IC59.7 (A1)
- new net: IC54.3 (Q0), IC59.8 (A0)
- new net: IC53.9 (B0), IC59.9 (D0)
- new net: IC70.1 (I3), IC71.13 (D3)
- new net: IC70.12 (I7), IC71.17 (D7)
- new net: IC70.13 (I6), IC71.16 (D6)
- new net: IC70.14 (I5), IC71.15 (D5)
- new net: IC70.15 (I4), IC71.14 (D4)
- new net: IC70.2 (I2), IC71.11 (D2)
- new net: IC70.3 (I1), IC71.10 (D1)
- new net: IC70.4 (I0), IC71.9 (D0)
- new net: IC45.8, IC70.7 (~{E})
- new net: IC48.3, IC51.1 (~{R})
- new net: IC45.12, IC51.2 (~{S1}), IC51.3 (~{S2})
- new net: IC51.4 (Q), IC56.4
- new net: C39.1, IC51.10 (~{R}), IC56.8
- new net: IC53.6 (Oa=b), IC58.3 (Ia=b)
- new net: C26.1, IC56.10, IC56.12, IC58.6 (Oa=b)
- new net: IC51.12 (~{S2}), IC56.11
- new net PL-V-ST: C6.1, IC54.12 (MR), IC54.2 (MR)
- new net SPLAY B: IC45.11
- new net ~{LIGHT}: C22.1, IC51.9 (Q)
- new net ~{SPLAY A}: IC48.8
- new net ~{SPLAY}: IC70.6 (~{Z})
- no-connect marks 32 -> 36
Other:
- moved on the sheet: IC22C, IC2C, IC30B, IC30E, IC34D, IC44B, IC46B, IC46C, IC46D, IC46E, IC46F, IC46G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

Commit message: edrjkghndrfkg
Parts:
- added IC62: 74LS32, Package_DIP:DIP-14_W7.62mm, symbol 74xx:74LS32
- added IC64: 74LS151, Package_DIP:DIP-16_W7.62mm, symbol 74xx:74LS151
- added IC65, IC77, IC84, IC91, IC98: MB7137, Package_DIP:DIP-24_W15.24mm, symbol Memory_PROM:MB7137
- added IC76: 74LS153, Package_DIP:DIP-16_W7.62mm, symbol 74xx:74LS153
Connections:
- net GNDPWR: now also IC64.8 (GND), IC65.12 (GND), IC65.21 (A10), IC77.12 (GND), IC84.12 (GND), IC91.12 (GND), IC98.12 (GND)
- net VCC: now also IC70.16 (VCC), IC64.16 (VCC), IC65.24 (VCC_(PVCC)), IC76.16 (VCC), IC77.24 (VCC_(PVCC)), IC84.24 (VCC_(PVCC)), IC91.24 (VCC_(PVCC)), IC98.24 (VCC_(PVCC))
- net ~{COIN IN}: now reaches IC57.1
- net ~{TUNNEL}: now reaches IC57.13
- net at IC44.4: now also IC64.7 (~{E})
- net at IC56.6: now also IC62.9
- net at IC71.4 (A4): now also IC65.4 (A4), IC77.4 (A4), IC84.4 (A4), IC91.4 (A4), IC98.4 (A4)
- net at IC71.5 (A3): now also IC65.5 (A3), IC77.5 (A3), IC84.5 (A3), IC91.5 (A3), IC98.5 (A3)
- net at IC71.6 (A2): now also IC65.6 (A2), IC77.6 (A2), IC84.6 (A2), IC91.6 (A2), IC98.6 (A2)
- net at IC71.7 (A1): now also IC65.7 (A1), IC77.7 (A1), IC84.7 (A1), IC91.7 (A1), IC98.7 (A1)
- net at IC71.8 (A0): now also IC65.8 (A0), IC77.8 (A0), IC84.8 (A0), IC91.8 (A0), IC98.8 (A0)
- new net: IC62.10, IC65.18 (CE2), IC65.19 (CE3)
- new net: IC64.3 (I1), IC65.10 (D1)
- new net: IC64.2 (I2), IC65.11 (D2)
- new net: IC64.1 (I3), IC65.13 (D3)
- new net: IC64.15 (I4), IC65.14 (D4)
- new net: IC64.14 (I5), IC65.15 (D5)
- new net: IC64.13 (I6), IC65.16 (D6)
- new net: IC64.12 (I7), IC65.17 (D7)
- new net: IC64.4 (I0), IC65.9 (D0)
- new net: IC76.5 (I1a), IC77.10 (D1), IC84.10 (D1), IC91.10 (D1), IC98.10 (D1)
- new net: IC76.4 (I2a), IC77.11 (D2), IC84.11 (D2), IC91.11 (D2), IC98.11 (D2)
- new net: IC76.3 (I3a), IC77.13 (D3), IC84.13 (D3), IC91.13 (D3), IC98.13 (D3)
- new net: IC76.10 (I0b), IC77.14 (D4), IC84.14 (D4), IC91.14 (D4), IC98.14 (D4)
- new net: IC76.11 (I1b), IC77.15 (D5), IC84.15 (D5), IC91.15 (D5), IC98.15 (D5)
- new net: IC76.12 (I2b), IC77.16 (D6), IC84.16 (D6), IC91.16 (D6), IC98.16 (D6)
- new net: IC76.13 (I3b), IC77.17 (D7), IC84.17 (D7), IC91.17 (D7), IC98.17 (D7)
- new net: IC76.6 (I0a), IC77.9 (D0), IC84.9 (D0), IC91.9 (D0), IC98.9 (D0)
Other:
- moved on the sheet: IC34D, IC44B
