File: Main/Main.kicad_sch (KiCad schematic)
At the start: 182 parts, among them IC1 74LS123, IC10 74LS85, IC11 74LS85, IC119 74LS123, IC12 74HC00, IC125 74LS11, IC13 74LS07, IC14 74LS20, IC15 74LS193, IC16 74LS86, IC17 74LS85, IC18 74LS85, IC19 74LS393, IC2 74LS08, IC20 74LS192, IC21 74LS192, IC22 74LS08, IC23 74LS32, IC24 74LS193, IC25 74LS193, IC26 NE555P, IC27 74HC279, IC28 74LS10, IC29 HD7417P, IC3 74LS153, IC30 74LS00, IC31 HD7417P, IC32 74HC279, IC33 74LS74, IC34 74LS08, IC35 74LS193, IC36 74LS193, IC37 74LS74, IC38 74HC123, IC39 74LS393, IC4 74LS151, IC40 74LS393, IC41 74LS85, IC42 74LS85, IC43 74LS123, IC44 74AHC04, IC45 74LS10, IC46 74LS04, IC47 74LS20, IC48 74HC00, IC49 74HC123, IC5 74LS393, IC50 74HC74, IC51 74HC279, IC52 74LS393, IC53 74LS85, IC54 74LS393, IC55 74LS32, IC56 74HC00, IC57 74LS20, IC58 74LS85, IC59 MB7137, IC6 74LS04, IC60 74LS157, IC61 74HC02, IC62 74LS32, IC63 74LS02, IC64 74LS151, IC65 MB7137, IC66 74LS08, IC67 7450, IC68 74LS00, IC69 74LS153, IC7 74LS85, IC70 74LS151, IC71 MB7137, IC72 74HC02, IC73 74AHC04, IC74 74LS27, IC76 74LS153, IC77 MB7137, IC79 74LS393, IC8 74HC00, IC80 74LS10, IC84 MB7137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

Commit message: fix speeds
Parts:
- IC12, IC48, IC56, IC8: value 74HC00 -> 74LS00; symbol 74xx:74HC00 -> 74xx:74LS00
- IC27, IC32, IC51: value 74HC279 -> 74LS279; symbol 74xxMissing:74HC279 -> 74xxMissing:74LS279
- IC29, IC31: value HD7417P -> 74LS07P; symbol 74xx:74HC7014 -> 74xx:74LS07
- IC38, IC49: value 74HC123 -> 74LS123; symbol 74xx:74HC123 -> 74xx:74LS123
- IC44, IC73: value 74AHC04 -> 74LS04; symbol 74xx:74AHC04 -> 74xx:74LS04
- IC50: value 74HC74 -> 74LS74; symbol 74xx:74HC74 -> 74xx:74LS74
- IC61, IC72: value 74HC02 -> 74LS02; symbol 74xx:74HC02 -> 74xx:74LS02

Commit message: rename stuff so the netlist works with nltool
Parts:
- C5: value 77u -> 47u
- C6: value C_Polarized_US -> 680p
- R4: value R_US -> 12k
- R5: value R_US -> 3.3k
- RA1: value R_Network08_US -> 560
- RA2: value R_Network07 -> 100
- renumbered VR1 to RV1, IC1 to U1, IC10 to U10, IC11 to U11, IC119 to U119, IC12 to U12, IC125 to U125, IC13 to U13, IC14 to U14, IC15 to U15, IC16 to U16, IC17 to U17, IC18 to U18, IC19 to U19, IC2 to U2, IC20 to U20, IC21 to U21, IC22 to U22, IC23 to U23, IC24 to U24, IC25 to U25, IC26 to U26, IC27 to U27, IC28 to U28, IC29 to U29, IC3 to U3, IC30 to U30, IC31 to U31, IC32 to U32, IC33 to U33, IC34 to U34, IC35 to U35, IC36 to U36, IC37 to U37, IC38 to U38, IC39 to U39, IC4 to U4, IC40 to U40, IC41 to U41, IC42 to U42, IC43 to U43, IC44 to U44, IC45 to U45, IC46 to U46, IC47 to U47, IC48 to U48, IC49 to U49, IC5 to U5, IC50 to U50, IC51 to U51, IC52 to U52, IC53 to U53, IC54 to U54, IC55 to U55, IC56 to U56, IC57 to U57, IC58 to U58, IC59 to U59, IC6 to U6, IC60 to U60, IC61 to U61, IC62 to U62, IC63 to U63, IC64 to U64, IC65 to U65, IC66 to U66, IC67 to U67, IC68 to U68, IC69 to U69, IC7 to U7, IC70 to U70, IC71 to U71, IC72 to U72, IC73 to U73, IC74 to U74, IC76 to U76, IC77 to U77, IC79 to U79, IC8 to U8, IC80 to U80, IC84 to U84, IC85 to U85, IC9 to U9, IC91 to U91, IC98 to U98

Commit message: page 4
Parts:
- added C30, C33: 10m, Capacitor_THT:CP_Radial_Tantal_D4.5mm_P2.50mm, symbol Device:C_Polarized_US
- added R16, R19: 47k, Resistor_THT:R_Axial_DIN0309_L9.0mm_D3.2mm_P12.70mm_Horizontal, symbol Device:R_US
- added RA3: 5.6k, Resistor_THT:R_Array_SIP9, symbol Device:R_Network08_US
- added U101, U102, U104, U109, U116, U117, U90, U96: 74LS161, Package_DIP:DIP-16_W7.62mm, symbol 74xx:74LS161
- added U103, U108, U118, U89: 74LS157, Package_DIP:DIP-16_W7.62mm, symbol 74xx:74LS157
- added U110, U124, U97: 74LS367, Package_DIP:DIP-16_W7.62mm, symbol 74xx:74LS367
- added U111: MB7137, Package_DIP:DIP-24_W15.24mm, symbol Memory_PROM:MB7137
- added U75: 74LS74, Package_DIP:DIP-14_W7.62mm, symbol 74xx:74LS74
- added U83: 74LS42, Package_DIP:DIP-16_W7.62mm, symbol 74xx:74LS42
- added U95: 74LS32, Package_DIP:DIP-14_W7.62mm, symbol 74xx:74LS32
Connections:
- net EV.CP (S) is gone; now on net A29: U29.12
- net EXTEND (C) is gone; now on net B8: U38.10 (B), U50.9 (Q)
- net GAME (I) is gone; now on net A27: U31.6
- net MUTE (S) is gone; now on net A26: U31.2
- net S-ACCE B is gone; now on net A13: U13.6
- net S-ACCE D is gone; now on net A12: U13.2
- net SCORE CP. is gone; now on net A14: U13.10
- net V6 is gone; now on net B12: U47.10, U67.1 (1A), U67.2 (2A)
- net ~{COIN IN} (S) is gone; now on net A28: U31.10
- net ~{EXTEND} (C) is gone; now on net B3: U50.8 (~{Q})
- net ~{GAME} (B) is gone; now on net B6: U31.9, U37.8 (~{Q}), U55.13
- net ~{SPLAY} is gone; now on net B10: U70.6 (~{Z})
- net 7MHz: now also U101.2 (CP), U102.2 (CP)
- net A20: now also J1.20 (Pin_20)
- net A30: now also J1.30 (Pin_30)
- net A9: now also J1.9 (Pin_9)
- net ACCE D: now also J2.14 (Pin_14)
- net B16: now also J2.16 (Pin_16)
- net GNDPWR: now also U65.20 (~{CE}1_(PVCE)), U76.8 (GND), U77.20 (~{CE}1_(PVCE)), U77.21 (A10), U101.8 (GND), U102.8 (GND), U103.11 (I0c), U103.2 (I0a), U103.5 (I0b), U103.8 (GND), U104.8 (GND), U108.10 (I1c), U108.3 (I1a), U108.6 (I1b), U108.8 (GND), U109.3 (D0), U109.4 (D1), U109.5 (D2), U109.6 (D3), U109.8 (GND), U116.3 (D0), U116.4 (D1), U116.5 (D2), U116.6 (D3), U116.8 (GND), U117.8 (GND), U83.8 (GND), U89.11 (I0c), U89.2 (I0a), U89.5 (I0b), U89.8 (GND), U90.8 (GND), U96.3 (D0), U96.4 (D1), U96.5 (D2), U96.6 (D3), U96.8 (GND)
- net H6: now also U75.12 (D)
- net VCC: now also U119.3 (Clr), R16.1, R19.1, RA3.1 (common), U101.1 (~{MR}), U101.16 (VCC), U101.7 (CEP), U102.1 (~{MR}), U102.10 (CET), U102.16 (VCC), U103.14 (I0d), U103.16 (VCC), U103.3 (I1a), U104.1 (~{MR}), U104.16 (VCC), U104.7 (CEP), U108.13 (I1d), U108.16 (VCC), U109.1 (~{MR}), U109.16 (VCC), U109.7 (CEP), U116.1 (~{MR}), U116.16 (VCC), U116.7 (CEP), U117.1 (~{MR}), U117.16 (VCC), U117.3 (D0), U117.7 (CEP), U83.16 (VCC), U89.14 (I0d), U89.16 (VCC), U89.3 (I1a), U90.1 (~{MR}), U90.16 (VCC), U90.7 (CEP), U96.1 (~{MR}), U96.16 (VCC), U96.7 (CEP), U97.16 (VCC)
- net Vs/16: now also U73.11, U95.4
- net ~{ACC I.}: now also U95.5, U95.9
- net ~{ACCI.ST}: now also U62.4
- net ~{SLIDE}: now also U119.1 (A)
- net ~{SP DOWN}: now also U72.1, U84.20 (~{CE}1_(PVCE)), U84.21 (A10)
- net at U34.13, U57.12, U57.4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: now also U52.4 (Q1); no longer U52.10 (Q1)
- net at U52.11 (Q0): now also U53.10 (A0), U64.11 (S0), U70.11 (S0), U76.14 (S0); no longer U58.10 (A0)
- net at U52.13 (CP): now also U63.1
- net at U34.12, U46.5, U57.9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: now also U52.6 (Q3), U65.2 (A6), U77.1 (A7), U84.1 (A7), U91.1 (A7), U98.1 (A7); no longer U52.8 (Q3)
- net at U57.10, U57.5, U58.13 (A2): now also U52.5 (Q2); no longer U52.9 (Q2)
- net at U119.13 (Q): now also U51.6 (~{S})
- net at U119.14 (Cext): now also C33.2
- net at U119.15 (RCext): now also C33.1, R19.2
- net at U119.2 (B): now also U68.3
- net ~{SCOKE.ST}: now reaches U119.4 (~{Q})
- net at U52.1 (CP): no longer U63.1
- net A10: now reaches J1.10 (Pin_10)
- net A11: now reaches J1.11 (Pin_11)
- net A11: now also U6.9
- net A12: now reaches J1.12 (Pin_12)
- net A13: now reaches J1.13 (Pin_13)
- net A14: now reaches J1.14 (Pin_14)
- net A15: now reaches J1.15 (Pin_15)
- net A15: now also U21.2 (QB)
- net A16: now reaches J1.16 (Pin_16)
- net A16: now also U21.6 (QC)
- net A17: now reaches J1.17 (Pin_17)
- net A17: now also U20.2 (QB)
- net A18: now reaches J1.18 (Pin_18)
- net A18: now also U20.6 (QC)
- net A19: now reaches J1.19 (Pin_19)
- net A19: now also U29.10
- net A21: now reaches J1.21 (Pin_21)
- net A21: now also U29.6
- net A22: now reaches J1.22 (Pin_22)
- net A25: now reaches J1.25 (Pin_25)
- net A26: now reaches J1.26 (Pin_26)
- net A27: now reaches J1.27 (Pin_27)
- net A28: now reaches J1.28 (Pin_28)
- net A29: now reaches J1.29 (Pin_29)
- net A31: now reaches J1.31 (Pin_31)
- net A6: now reaches J1.6 (Pin_6)
- net A7: now reaches J1.7 (Pin_7)
- net A8: now reaches J1.8 (Pin_8)
- net EXPLO.ST.(F): now reaches U62.8
- net EXPLO.ST.(F): now also U76.1 (Ea), U76.15 (Eb), U83.12 (A3), U83.13 (A2)
- net at U52.3 (Q0): now also U58.10 (A0); no longer U53.10 (A0)
- net at U53.12 (A1): now also U52.10 (Q1), U64.10 (S1), U70.10 (S1), U76.2 (S1); no longer U52.4 (Q1)
- net at U53.13 (A2): now also U52.9 (Q2), U64.9 (S2), U70.9 (S2), U77.3 (A5), U84.3 (A5), U91.3 (A5), U98.3 (A5); no longer U52.5 (Q2)
- net at U53.15 (A3): now also U52.8 (Q3), U65.3 (A5), U77.2 (A6), U84.2 (A6), U91.2 (A6), U98.2 (A6); no longer U52.6 (Q3)
- net at U66.2: now also U119.12 (~{Q})
- net at U72.2: now also U119.5 (Q)
- net at U68.1: now also U84.18 (CE2), U84.19 (CE3), U91.18 (CE2), U91.19 (CE3), U98.18 (CE2), U98.19 (CE3)
- net ~{PLAYER BODY}: now reaches U68.2
- net ~{PLAYER BODY}: now also U44.11, U83.2 (1)
- net at U119.6 (Cext): now also C30.2
- net at U119.7 (RCext): now also C30.1, R16.2
- net EXPLO.SGE A: now reaches U65.1 (A7)
- net EXPLO.SGE A: now also U63.9
- net EXPLO.SGE B: now reaches U65.23 (A8)
- net at U98.20 (~{CE}1_(PVCE)): now also U98.21 (A10), U95.8
- net at U98.23 (A8): now also U84.23 (A8), U91.23 (A8)
- net at U64.5 (Z): now also U56.2
- net C15: now reaches U64.6 (~{Z})
- net C15: now also U62.12
- net at U73.10: now also U95.10
- net at U77.18 (CE2): now also U77.19 (CE3)
- net ~{EXTEND} (A): now reaches U62.5
- net ~{EXPLO (R)}: now reaches U62.11
- net at U62.13: now also U56.1, U63.10
- net B4: now reaches U56.3
- net B4: now also J2.4 (Pin_4)
- net EXPLO.SGE C: now reaches U63.8
- net at U29.11: now also U75.8 (~{Q})
- net B1: now reaches J2.1 (Pin_1)
- net B10: now reaches J2.10 (Pin_10)
- net B11: now reaches J2.11 (Pin_11)
- net B12: now reaches J2.12 (Pin_12)
- net B13: now reaches J2.13 (Pin_13)
- net B15: now reaches J2.15 (Pin_15)
- net B17: now reaches J2.17 (Pin_17)
- net B18: now reaches J2.18 (Pin_18)
- net B19: now reaches J2.19 (Pin_19)
- net B19: now also U83.3 (2)
- net B2: now reaches J2.2 (Pin_2)
- net B20: now reaches J2.20 (Pin_20)
- net B21: now reaches J2.21 (Pin_21)
- net B22: now reaches J2.22 (Pin_22)
- net B3: now reaches J2.3 (Pin_3)
- net B5: now reaches J2.5 (Pin_5)
- net B6: now reaches J2.6 (Pin_6)
- net B7: now reaches J2.7 (Pin_7)
- net B8: now reaches J2.8 (Pin_8)
- net B9: now reaches J2.9 (Pin_9)
- net B9: now also U61.10
- net at U61.8: now also U76.7 (Za), U83.15 (A0)
- net at U61.9: now also U76.9 (Zb), U83.14 (A1)
- net at U91.20 (~{CE}1_(PVCE)): now also U91.21 (A10), U95.6
- net V2 renamed C6
- new net: U102.3 (D0), U108.4 (Za)
- new net: U102.4 (D1), U108.7 (Zb)
- new net: U102.5 (D2), U108.9 (Zc)
- new net: U102.6 (D3), U108.12 (Zd)
- new net: RA3.5 (R4), U110.3 (O1a), U111.8 (A0), U124.3 (O1a), U97.3 (O1a)
- new net: RA3.4 (R3), U110.5 (O2a), U111.7 (A1), U124.5 (O2a), U97.5 (O2a)
- new net: RA3.3 (R2), U110.7 (O3a), U111.6 (A2), U124.7 (O3a), U97.7 (O3a)
- new net: RA3.2 (R1), U110.9 (O4a), U111.5 (A3), U124.9 (O4a), U97.9 (O4a)
- new net: U116.10 (CET), U117.15 (TC)
- new net: U104.2 (CP), U109.2 (CP), U116.2 (CP), U117.2 (CP), U90.2 (CP), U96.2 (CP)
- new net: U90.15 (TC), U96.10 (CET)
- new net: U104.15 (TC), U109.10 (CET)
- new net: U103.4 (Za), U104.3 (D0)
- new net: U103.7 (Zb), U104.4 (D1)
- new net: U103.9 (Zc), U104.5 (D2)
- new net: U103.12 (Zd), U104.6 (D3)
- new net: U118.15 (E), U124.13 (O6b)
- new net: U90.11 (Q3), U97.10 (I4)
- new net: U90.12 (Q2), U97.6 (I3)
- new net: U90.13 (Q1), U97.4 (I2)
- new net: U90.14 (Q0), U97.2 (I1)
- new net: U89.4 (Za), U90.3 (D0)
- new net: U89.7 (Zb), U90.4 (D1)
- new net: U89.9 (Zc), U90.5 (D2)
- new net: U89.12 (Zd), U90.6 (D3)
- new net: U111.15 (D5), U118.10 (I1c)
- new net: U111.14 (D4), U118.11 (I0c)
- new net: U111.17 (D7), U118.13 (I1d)
- new net: U111.16 (D6), U118.14 (I0d)
- new net: U111.9 (D0), U118.2 (I0a)
- new net: U111.10 (D1), U118.3 (I1a)
- new net: U111.11 (D2), U118.5 (I0b)
- new net: U111.13 (D3), U118.6 (I1b)
- new net: U117.4 (D1), U117.5 (D2)
- new net H3: U75.13 (~{R})
- new net ~{PLAYER (BL)}: U83.4 (3)
- no-connect marks 36 -> 46
Other:
- moved on the sheet: U119A, U119B, U29E, U44E, U45C, U51B, U52A, U52B, U56A, U61C, U63C, U66D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

Commit message: got new pics of the bottom
Connections:
- net 7MHz: now also U63.12
- net A6: now also R998.2, U12.8
- net B12: now also U69.10 (I0b), U69.11 (I1b)
- net COIN IN (B): now also U72.8; no longer U72.9
- net V5: now also U69.13 (I3b), U69.3 (I3a)
- net V7: no longer U69.13 (I3b), U69.3 (I3a)
- net Vs/8: now also U34.10
- net ~{H}s: now also U40.1 (CP)
- net at U66.9, U72.5, U9.10 (I0b): now also U69.9 (Zb)
- net at U12.4: now also U34.5, U60.7 (Zb)
- net at U12.5: now also U10.5 (Oa>b)
- net at U12.6: now also U25.4 (DOWN)
- net at U25.5 (UP): now also U12.3
- net at U69.7 (Za): now also U12.1
- net at U33.8 (~{Q}): now also U72.9; no longer U72.8
- net at C20.1, R11.2: now also U43.15 (RCext); no longer U43.7 (RCext)
- net at C20.2: now also U43.14 (Cext); no longer U43.6 (Cext)
- net at U12.2: now also U10.7 (Oa<b)
- net at U2.1: now also U3.14 (S0), U43.12 (~{Q})
- net A4: now reaches SW2.1 (A)
- net at C18.2: now also R10.2, U43.7 (RCext); no longer U43.14 (Cext)
- net ~{SLIP}: now reaches U43.1 (A)
- net at U43.4 (~{Q}): now also U29.3, U3.2 (S1)
- net ~{SLIPZONE}: now reaches U29.4
- net ~{POOL}: now reaches U43.9 (A), U49.9 (A)
- new net: C18.1, U43.6 (Cext)
Other:
- moved on the sheet: C18, C20, R10, R11, U12A, U12B, U29B, U72C

Commit message: add led board
Parts:
- added C34, C35: 470m, Capacitor_THT:CP_Radial_D10.0mm_P5.00mm, symbol Device:C_Polarized_US
- added R17, R18, R20, R21: 47k, Resistor_THT:R_Axial_DIN0309_L9.0mm_D3.2mm_P12.70mm_Horizontal, symbol Device:R_US
- added U107: 74LS10, Package_DIP:DIP-14_W7.62mm, symbol 74xx:74LS10
- added U114: 74LS04, Package_DIP:DIP-14_W7.62mm, symbol 74xx:74LS04
- added U120, U121: 74LS123, Package_DIP:DIP-16_W7.62mm, symbol 74xx:74LS123
- added U81: 74LS279, Package_DIP:DIP-16_W7.62mm, symbol 74xxMissing:74LS279
- C31, C32: value 100m -> 470m
- C6: footprint Capacitor_THT:C_Disc_D3.0mm_W1.6mm_P2.50mm -> Capacitor_THT:C_Disc_D7.5mm_W5.0mm_P7.50mm
Connections:
- net A23: now also D1.2 (A)
- net GNDPWR: now also U110.8 (GND), U111.12 (GND), U118.8 (GND), U124.8 (GND), U97.8 (GND)
- net VCC: now also U1.16 (VCC), U110.16 (VCC), U111.24 (VCC_(PVCC)), U118.16 (VCC), U124.16 (VCC), R17.1, R18.1, R20.2, R21.1
- net Vs/2: now also U30.5
- net Vs/32: now also U72.5; no longer U72.6
- net at U66.9, U69.9 (Zb), U9.10 (I0b): now also U72.6; no longer U72.5
- net at U66.8, U9.12 (I2b): now also U3.12 (I2b)
- net at U72.4, U9.4 (I2a): now also U3.4 (I2a)
- net at U75.1 (~{R}): now also U75.4 (~{S})
- net at U110.13 (O6b): now also RA3.6 (R5), U118.15 (E), U124.13 (O6b), U75.11 (C), U97.13 (O6b)
- net at U10.11 (B1), U4.10 (S1), U6.2: now also U14.5, U6.13
- net at U10.14 (B2), U4.9 (S2), U6.4: no longer U14.5, U6.13
- net at U95.11: now also U81.2 (~{S1}), U81.3 (~{S2})
- net at U95.13: now also U95.1
- net at U101.14 (Q0): now also U111.1 (A7)
- net at C32.1: now also R18.2, U121.7 (RCext)
- net at C32.2: now also U121.6 (Cext)
- net at U118.12 (Zd): now also U114.11
- net at U118.7 (Zb): now also U114.1
- net at U118.9 (Zc): now also U114.13
- net at U95.3: now also U81.1 (~{R})
- net at U89.1 (S): now also U107.12
- net at U103.1 (S): now also U107.8
- net Vs/4: now reaches U30.4
- net Vs/4: now also U111.23 (A8)
- net at C31.1: now also R17.2, U120.7 (RCext)
- net at C31.2: now also U120.6 (Cext)
- new net: U107.1, U121.13 (Q)
- new net: U107.13, U121.1 (A), U121.5 (Q)
- new net: U107.10, U120.5 (Q)
- new net: U107.9, U120.13 (Q)
- new net: C35.2, U121.14 (Cext)
- new net: C35.1, R21.2, U121.15 (RCext)
- new net: U121.2 (B), U121.9 (A)
- new net: U120.11 (Clr), U120.3 (Clr), U121.11 (Clr), U121.3 (Clr)
- new net: C34.1, R20.1, U120.15 (RCext)
- new net: C34.2, U120.14 (Cext)
- new net: U120.2 (B), U120.9 (A)
- no-connect marks 46 -> 49
Other:
- moved on the sheet: U29E, U30B, U75B

Commit message: more page 4 and redo of the pcb
Parts:
- added U100: 7450, Package_DIP:DIP-14_W7.62mm, symbol 74xxMissing:7450
- added unit 3 of U40
- added U78: 74LS393, Package_DIP:DIP-14_W7.62mm, symbol 74xx:74LS393
- added U82: 74LS04, Package_DIP:DIP-14_W7.62mm, symbol 74xx:74LS04
- added U86: 74LS02, Package_DIP:DIP-14_W7.62mm, symbol 74xx:74LS02
- added U87: 74LS107, Package_DIP:DIP-14_W7.62mm, symbol 74xx:74LS107
- added U88: 74LS32, Package_DIP:DIP-14_W7.62mm, symbol 74xx:74LS32
- added U92, U99: 74LS74, Package_DIP:DIP-14_W7.62mm, symbol 74xx:74LS74
- added U93: 74LS08, Package_DIP:DIP-14_W7.62mm, symbol 74xx:74LS08
- added U94: 74LS259, Package_DIP:DIP-16_W7.62mm, symbol 74xx:74LS259
Connections:
- net B15: now also U114.10, U114.2
- net GNDPWR: now also U101.5 (D2), U101.6 (D3), U79.12 (MR), U89.15 (E), U78.12 (MR), U78.2 (MR)
- net VCC: now also U101.3 (D0), U101.4 (D1), U87.10 (~{R}), U87.11 (K), U87.8 (J), U92.1 (~{R}), U92.10 (~{S}), U92.13 (~{R}), U92.4 (~{S}), U99.1 (~{R}), U99.10 (~{S}), U99.13 (~{R}), U99.4 (~{S})
- net Vs/16: now also U79.8 (Q3), U78.1 (CP)
- net Vs/2: now also U79.11 (Q0)
- net Vs/32: now also U78.3 (Q0)
- net Vs/4: now also U79.10 (Q1)
- net Vs/64: now also U78.4 (Q1)
- net Vs/8: now also U79.9 (Q2)
- net ~{OTHER BODY}: now also U114.12
- net at U81.4 (Q): now also U121.2 (B), U121.9 (A), U89.13 (I1d), U82.5
- net at U102.11 (Q3): now also U111.2 (A6)
- net at U102.12 (Q2): now also U111.3 (A5)
- net at U102.13 (Q1): now also U111.4 (A4)
- net at U102.14 (Q0): now also U118.1 (S)
- net at U102.15 (TC): now also U101.10 (CET), U80.9
- net at U102.7 (CEP): now also U81.9 (Q)
- net at U102.9 (~{PE}): now also U101.9 (~{PE}), U80.8
- net at U110.1 (OEa): now also U110.15 (OEb), U100.6 (2Y)
- net at U110.10 (I4): now also U104.11 (Q3)
- net at U110.2 (I1): now also U104.14 (Q0)
- net at U110.4 (I2): now also U104.13 (Q1)
- net at U110.6 (I3): now also U104.12 (Q2)
- net at U107.2: now also U30.6
- net at U81.13 (Q): now also U103.13 (I1d), U120.2 (B), U120.9 (A), U82.9
- net at U81.14 (~{R}): now also U88.11
- net at U81.15 (~{S}): now also U88.3
- net at U85.6: now also U95.12, U88.1, U88.4
- net at U81.5 (~{R}): now also U88.8
- net at U81.6 (~{S}): now also U88.6
- net at U124.1 (OEa): now also U124.15 (OEb)
- net at U124.10 (I4): now also U117.11 (Q3)
- net at U124.2 (I1): now also U117.14 (Q0)
- net at U124.4 (I2): now also U117.13 (Q1)
- net at U124.6 (I3): now also U117.12 (Q2)
- net at U95.1, U95.13: now also U97.14 (I6)
- net at U80.10: now also U101.15 (TC), U87.9 (C)
- net at U80.11: now also U87.5 (Q)
- net at U101.11 (Q3): now also U94.3 (A2)
- net at U101.12 (Q2): now also U94.2 (A1)
- net at U101.13 (Q1): now also U94.1 (A0)
- net at U85.8: now also U95.2, U88.13
- net at U97.1 (OEa): now also U97.15 (OEb), U100.8 (1Y)
- net at U89.10 (I1c): now also U89.6 (I1b), U82.6
- net at U103.10 (I1c): now also U103.6 (I1b), U82.8
- net C12: now reaches U79.13 (CP)
- net C12: now also U86.12
- net at U117.4 (D1), U117.5 (D2): now also U82.2
- new net: U100.1 (1A), U99.5 (Q)
- new net: U100.10 (1D), U93.12
- new net: U100.13 (1B), U93.1
- new net: U100.9 (1C), U99.9 (Q)
- new net: U87.6 (~{Q}), U94.14 (E)
- new net: U92.3 (C), U93.8
- new net: U100.2 (2A), U92.5 (Q)
- new net: U88.5, U88.9
- new net: U86.13, U93.10, U93.13, U93.2, U93.4
- new net: U93.3, U99.3 (C)
- new net: U100.5 (2D), U93.5
- new net: U92.11 (C), U93.6
- new net: U88.12, U88.2
- new net: U100.4 (2C), U92.9 (Q)
- new net: U100.3 (2B), U93.9
- new net: U93.11, U99.11 (C)
- new net Vs/1k: U78.10 (Q1)
- new net Vs/256: U78.13 (CP), U78.6 (Q3)
- new net Vs/512: U78.11 (Q0)
- new net ~{H}5: U86.11
- no-connect marks 49 -> 61
Other:
- moved on the sheet: J1, J2, J3, U79B, U80C, U81A, U81B, U81C, U81D, U85B, U85C, U95A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
