File: Main/Main.kicad_sch (KiCad schematic)
At the start: 227 parts, among them J1 Conn_01x36_Pin, J2 Conn_01x22, J3 Conn_01x28_Pin, SW1 1COIN 1PLAY/1COIN 2PLAY, SW2 CREDIT, SW3 TEST, SW4 COIN, SW5 TILT SW., U1 74LS123, U10 74LS85, U100 7450, U101 74LS161, U102 74LS161, U103 74LS157, U104 74LS161, U107 74LS10, U108 74LS157, U109 74LS161, U11 74LS85, U110 74LS367, U111 MB7137, U114 74LS04, U116 74LS161, U117 74LS161, U118 74LS157, U119 74LS123, U12 74LS00, U120 74LS123, U121 74LS123, U124 74LS367, U125 74LS11, U13 74LS07, U14 74LS20, U15 74LS193, U16 74LS86, U17 74LS85, U18 74LS85, U19 74LS393, U2 74LS08, U20 74LS192, U21 74LS192, U22 74LS08, U23 74LS32, U24 74LS193, U25 74LS193, U26 NE555P, U27 74LS279, U28 74LS10, U29 74LS07P, U3 74LS153, U30 74LS00, U31 74LS07P, U32 74LS279, U33 74LS74, U34 74LS08, U35 74LS193, U36 74LS193, U37 74LS74, U38 74LS123, U39 74LS393, U4 74LS151, U40 74LS393, U41 74LS85, U42 74LS85, U43 74LS123, U44 74LS04, U45 74LS10, U46 74LS04, U47 74LS20, U48 74LS00, U49 74LS123, U5 74LS393, U50 74LS74, U51 74LS279, U52 74LS393, U53 74LS85, U54 74LS393, U55 74LS32, U56 74LS00, U57 74LS20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

Commit message: prom and power
Parts:
- added C36: 0.01m, Capacitor_THT:C_Disc_D7.5mm_W5.0mm_P7.50mm, symbol Device:C_Polarized_US
- added U105, U115: 74S288, Package_DIP:DIP-16_W7.62mm, symbol 74xxMissing:74S288
- added U106: 74LS08, Package_DIP:DIP-14_W7.62mm, symbol 74xx:74LS08
- added U112: 74LS393, Package_DIP:DIP-14_W7.62mm, symbol 74xx:74LS393
- added U113: 74LS85, Package_DIP:DIP-16_W7.62mm, symbol 74xx:74LS85
- added U122: 74LS02, Package_DIP:DIP-14_W7.62mm, symbol 74xx:74LS02
- added U123: 74LS10, Package_DIP:DIP-14_W7.62mm, symbol 74xx:74LS10
- added unit 3 of U78
Connections:
- net GNDPWR: now also U1.8 (GND), U100.7 (GND), U107.7 (GND), U114.7 (GND), U119.8 (GND), U120.16 (VCC), U121.16 (VCC), U40.7 (GND), U43.8 (GND), U45.7 (GND), U46.7 (GND), U47.7 (GND), U48.7 (GND), U51.8 (GND), U52.7 (GND), U54.7 (GND), U56.7 (GND), U57.7 (GND), U6.7 (GND), U62.7 (GND), U63.7 (GND), U66.7 (GND), U75.7 (GND), U80.7 (GND), U81.8 (GND), U82.7 (GND), U86.7 (GND), U87.7 (GND), U88.7 (GND), U92.7 (GND), U93.7 (GND), U94.8 (GND), U95.14 (VCC), U99.7 (GND), U105.8 (GND), U106.7 (GND), U113.2 (Ia<b), U113.4 (Ia>b), U113.8 (GND), U115.8 (GND), U122.7 (GND), U123.7 (GND), U78.7 (GND)
- net VCC: now also U100.14 (VCC), U107.14 (VCC), U114.14 (VCC), U119.16 (VCC), U120.8 (GND), U121.8 (GND), U30.14 (VCC), U31.14 (VCC), U40.14 (VCC), U43.16 (VCC), U45.14 (VCC), U46.14 (VCC), U47.14 (VCC), U48.14 (VCC), U51.16 (VCC), U52.14 (VCC), U54.14 (VCC), U56.14 (VCC), U57.14 (VCC), U6.14 (VCC), U62.14 (VCC), U63.14 (VCC), U66.14 (VCC), U75.14 (VCC), U80.14 (VCC), U81.16 (VCC), U82.14 (VCC), U86.14 (VCC), U87.14 (VCC), U88.14 (VCC), U92.14 (VCC), U93.14 (VCC), U94.16 (VCC), U95.7 (GND), U99.14 (VCC), U105.16 (VCC), U106.14 (VCC), U113.16 (VCC), U113.3 (Ia=b), U115.16 (VCC), U122.14 (VCC), U123.14 (VCC), U78.14 (VCC)
- net at U116.11 (Q3): now also U123.9
- net at U116.12 (Q2): now also U122.12
- net at U116.13 (Q1): now also U123.11
- net at U116.14 (Q0): now also U122.11
- net at U116.9 (~{PE}): now also U117.9 (~{PE})
- net at U96.11 (Q3): now also U123.2
- net at U96.12 (Q2): now also U122.9
- net at U96.13 (Q1): now also U123.1
- net at U96.14 (Q0): now also U122.8
- net at U124.14 (I6): now also U88.5, U88.9, U123.8
- net at U109.11 (Q3): now also U123.5
- net at U109.12 (Q2): now also U122.2
- net at U109.13 (Q1): now also U123.3
- net at U109.14 (Q0): now also U122.3
- new net: C36.1, U115.14 (A4)
- new net: C36.2, U115.15 (~{G})
- new net: U122.13, U123.10
- new net: U112.11 (Q0), U113.1 (B3)
- new net: U112.9 (Q2), U113.11 (B1)
- new net: U113.12 (A1), U115.11 (A1)
- new net: U112.10 (Q1), U113.14 (B2)
- new net: U113.15 (A3), U115.13 (A3)
- new net: U112.8 (Q3), U113.9 (B0)
- new net: U122.1, U123.4
- new net: U122.10, U123.13
- no-connect marks 61 -> 62
Other:
- moved on the sheet: U12D, U49C, U66E, U72E, U85D, U86E, U94, U95E

Commit message: fix schematic errors
Parts:
- added C28, C29, C8, C9: 470m, Capacitor_THT:C_Disc_D4.3mm_W1.9mm_P5.00mm, symbol Device:C_Polarized_US
- U105, U115: footprint Package_DIP:DIP-16_W7.62mm -> Package_DIP:DIP-16_W15.24mm
Connections:
- net ACCE D is gone; now on net ACCE. D: J2.14 (Pin_14), U13.1, U6.12
- net ~{COIN&TEST} (F) is gone; now on net ~{COIN&TEST}: U73.4
- net ~{COIN&TEST} (I) is gone; now on net ~{COIN&TEST}: U31.4
- net ~{GAME} (S) is gone; now on net B6: U31.8
- net 8000: now also U62.1
- net B6: now also U15.14 (CLR)
- net CAR.CONT.CL (4): now also U112.2 (MR); no longer U55.8
- net GNDPWR: now also U103.15 (E), U105.15 (~{G}), U108.15 (E), U94.15 (Clr), C28.2, C29.2, C8.2, C9.2; no longer U105.8 (GND)
- net H5: now also U74.2; no longer U74.4
- net H8: now also U74.13; no longer U74.5
- net PL-V-ST: now also U52.12 (MR), U52.2 (MR)
- net VCC: now also U17.16 (VCC), U18.16 (VCC), U3.16 (VCC), U41.16 (VCC), U75.1 (~{R}), U75.4 (~{S}), U9.16 (VCC), U94.13 (D)
- net Vs/1k: now also U105.12 (A2)
- net Vs/2: now also U107.11
- net Vs/256: now also U105.10 (A0)
- net Vs/512: now also U105.11 (A1)
- net ~{ACCI.ST}: now also U80.3; no longer U80.4
- net ~{TUNNEL}: now also U8.13
- net at U112.1 (CP): now also U86.4, C29.1
- net at U112.3 (Q0): now also U105.13 (A3), U106.10
- net at U112.4 (Q1): now also U105.14 (A4), U106.9
- net at U52.8 (Q3), U53.15 (A3), U65.3 (A5)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: now also U52.1 (CP), U71.3 (A5)
- net at U75.2 (D): now also U106.6
- net at U75.3 (C): now also U66.6, C8.1
- net at U75.5 (Q): now also U68.9
- net at U16.12, U16.2, U4.7 (~{E})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: now also U23.3
- net SP. CONT.: now reaches C36.1, U115.14 (A4)
- net at U101.9 (~{PE}), U102.9 (~{PE}), U80.8: now also U104.2 (CP), U109.2 (CP), U116.2 (CP), U117.2 (CP), U86.8, U90.2 (CP), U96.2 (CP)
- net at U110.14 (I6): now also U123.6, U88.12, U88.2
- net at U34.12, U46.5, U52.6 (Q3)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: now also U71.2 (A6)
- net at U56.6, U62.9: now also U74.5
- net at U8.2: now also U7.5 (Oa>b)
- net ACCE. B: now reaches U13.5, U14.4, U15.2 (QB), U6.5, U7.12 (A1)
- net ACCE. B: now also U113.12 (A1), U115.11 (A1)
- net at U72.3: now also U45.5
- net at U100.13 (1B), U93.1: now also U94.9 (Q4), C28.1
- net at U82.10: now also U90.9 (~{PE}), U96.9 (~{PE})
- net at U82.11: now also U96.15 (TC)
- net at U116.15 (TC): now also U82.13
- net at U116.9 (~{PE}), U117.9 (~{PE}): now also U82.12
- net at U46.3, U48.2, U54.9 (Q2)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: now also U71.23 (A8)
- net at U113.13 (A2): now also U106.11
- net ACCE. D: now reaches U113.15 (A3), U115.13 (A3)
- net at U113.6 (Oa=b): now also U114.5
- net at U68.11: now also U74.1; no longer U74.3
- net at C3.1, U19.12 (MR), U19.2 (MR): now also U74.12; no longer U74.6
- net AREA 1: now reaches U94.10 (Q5)
- net AREA 1: now also U66.5, U68.10
- net AREA 5: now reaches U94.12 (Q7)
- net AREA 5: now also U100.3 (2B), U93.9
- net AREA 2: now reaches U94.4 (Q0)
- net AREA 2: now also U100.5 (2D), U93.5
- net ~{L1-SIDE}: now reaches U85.4
- net C4: now reaches U85.5
- net C16: now reaches U115.1 (D0)
- net ACCE. A: now reaches U115.10 (A0)
- net ACCE. A: now also U13.9, U14.2, U15.3 (QA)
- net ACCE. C: now reaches U115.12 (A2)
- net ACCE. C: now also U106.13, U13.3, U14.1, U15.6 (QC), U6.3, U7.13 (A2)
- net SP. B: now reaches U115.2 (D1)
- net C17: now reaches U115.3 (D2)
- net SP. D: now reaches U115.4 (D3)
- net at U115.5 (D4): now also U108.2 (I0a)
- net at U115.6 (D5): now also U108.5 (I0b)
- net at U115.7 (D6): now also U108.11 (I0c)
- net at U115.9 (D7): now also U108.14 (I0d)
- net at U92.2 (D): now also U105.3 (D2)
- net at U104.10 (CET): now also U117.10 (CET), U90.10 (CET)
- net at U104.9 (~{PE}): now also U109.9 (~{PE}), U82.4
- net at U81.7 (Q): now also U117.6 (D3), U82.1
- net at U86.10: now also U112.12 (MR), U114.3
- net at U86.9: now also U108.1 (S)
- net at U16.9, U28.9, U32.13 (Q): now also U22.2, U29.9
- net at U106.8: now also U86.6
- net at U10.14 (B2), U4.9 (S2), U6.4: now also U80.13
- net at U107.10, U120.5 (Q): now also U120.1 (A)
- net at U109.15 (TC): now also U82.3
- net at U121.4 (~{Q}): now also U121.10 (B)
- net 14MHz: now reaches U112.13 (CP)
- net at U66.4: now also U86.13, U93.10, U93.13, U93.2, U93.4
- net at U14.8: now also U80.4; no longer U80.3
- net at U81.10 (~{R}): now also U114.4
- net at U81.11 (~{S1}): now also U114.6, U81.12 (~{S2})
- net at U99.2 (D): now also U105.2 (D1)
- net at U120.4 (~{Q}): now also U120.10 (B)
- net at U44.3: now also U74.6
- net SHIFT: now reaches U29.8
- net C3: now reaches U86.5
- net ~{SP IRREG.}: now reaches U106.12
- net ~{SP IRREG.}: now also U80.12
- net ~{R2-SIDE}: now reaches U85.10
- net ~{R-L-SIDE}: now reaches U85.11
- net ~{R1-SIDE}: now reaches U85.9
- net at U105.1 (D0): now also U92.12 (D)
- net at U105.4 (D3): now also U99.12 (D)
- net at U105.5 (D4): now also U106.5
- net EXT.CAR CONT.: now reaches U80.1
- net at U80.2: now also U62.3
- net at U32.14 (~{R}): now also C10.1
- net ~{EXT. 500}: now reaches U62.2
- net ~{EXT. 500}: now also U106.4
- net at U68.8: now also C9.1
- net EXPLO. SEL. A (G) renamed EXPLO. SEL. A
- net EXPLO. SEL. B (G) renamed EXPLO. SEL. B
- net EXPLO. SEL. C (G) renamed EXPLO. SEL. C
- net EXPLO. SEL. D (G) renamed EXPLO. SEL. D
- net EXPLO. SEL. D: now also U74.4
- net EXPLO.SGE A renamed EXPLO.SEL. A
- net EXPLO.SGE B renamed EXPLO.SEL. B
- net EXPLO.SGE C renamed EXPLO.SEL. C
- net EXPLO.ST.(F) renamed EXPLO.ST.
- net S-ACCE A renamed S-ACCE. A
- net S-ACCE C renamed S-ACCE. C
- net SCORE ST. renamed ~{SCORE ST.}
- net SP DOWN (G) renamed SP. DOWN
- net ~{EX.SIG???.??} (M) renamed ~{EX.SIGNAL CP}
- net ~{FX.SIGNAL} (B) renamed ~{FX.SIGNAL}
- net ~{INI. RESET} (B) renamed ~{INI. RESET}
- net ~{SCOKE.ST} renamed ~{SCORE.ST}
- new net CAR.CONT.CL: U55.8
- new net ~{EXPLO.ST.}: U74.3
- no-connect marks 62 -> 79
Other:
- moved on the sheet: U105, U106B, U106C, U106D, U112A, U114B, U114C, U29D, U45B, U62A, U66B, U68C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

Commit message: my wrist hurts
Parts:
- added C11: 470m, Capacitor_THT:C_Disc_D4.3mm_W1.9mm_P5.00mm, symbol Device:C_Polarized_US
Connections:
- net CAR.CONT.CL (4) is gone; now on net CAR.CONT.CL: U112.2 (MR)
- net SPLAY B is gone; now on net ~{SPLAY B}: U45.11
- net ~{FX.SIGNAL} is gone; now on net C1: U49.4 (~{Q})
- net AREA 5: now also J3.10 (Pin_10)
- net B10: now also U71.1 (A7)
- net C12: now also J3.12 (Pin_12)
- net C3: now also J3.3 (Pin_3)
- net C4: now also J3.4 (Pin_4)
- net C6: now also J3.6 (Pin_6)
- net GNDPWR: now also C11.2
- net SP. DOWN: now also U119.5 (Q), U72.2
- net Vs/16: now also U29.5
- net at U1.1 (A), U1.9 (A): now also U29.3, U3.2 (S1), U43.4 (~{Q})
- net at U48.12, U48.4, U54.11 (Q0)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: now also U45.2, U48.2, U65.4 (A4), U71.4 (A4), U77.4 (A4), U84.4 (A4), U91.4 (A4), U98.4 (A4); no longer U45.13, U48.1
- net AREA 4: now reaches U100.10 (1D), U93.12
- net AREA 4: now also U106.3, C11.1
- net AREA 3: now reaches C28.1, U100.13 (1B), U93.1, U94.9 (Q4)
- net at U46.3, U54.9 (Q2), U59.2 (A6)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: now also U48.1; no longer U48.2
- net at U48.13, U54.10 (Q1), U59.3 (A5): no longer U45.2
- net at U54.13 (CP), U54.6 (Q3), U59.5 (A3): now also U65.5 (A3), U71.5 (A3), U77.5 (A3), U84.5 (A3), U91.5 (A3), U98.5 (A3)
- net at U54.5 (Q2), U59.6 (A2): now also U65.6 (A2), U71.6 (A2), U77.6 (A2), U84.6 (A2), U91.6 (A2), U98.6 (A2)
- net at U54.4 (Q1), U59.7 (A1): now also U65.7 (A1), U71.7 (A1), U77.7 (A1), U84.7 (A1), U91.7 (A1), U98.7 (A1)
- net at U54.3 (Q0), U59.8 (A0): now also U65.8 (A0), U71.8 (A0), U77.8 (A0), U84.8 (A0), U91.8 (A0), U98.8 (A0)
- net at U106.1: now also U107.6
- net at U106.2: now also U101.11 (Q3), U94.3 (A2)
- net at U101.13 (Q1), U94.1 (A0): now also U107.4
- net at U101.12 (Q2), U94.2 (A1): now also U107.5
- net C1: now reaches J3.1 (Pin_1)
- net C11: now reaches J3.11 (Pin_11)
- net C13: now reaches J3.13 (Pin_13)
- net C2: now reaches J3.2 (Pin_2)
- net C5: now reaches J3.5 (Pin_5)
- net C7: now reaches J3.7 (Pin_7)
- net C8: now reaches J3.8 (Pin_8)
- net C9: now reaches J3.9 (Pin_9)
- net at U80.11, U87.5 (Q): now also U107.3
- net at U101.14 (Q0), U111.1 (A7): now also U111.15 (D5), U111.17 (D7), U118.10 (I1c), U118.13 (I1d)
- net at U15.7 (QD), U6.1, U7.15 (A3): now also U43.11 (Clr), U43.3 (Clr), U49.11 (Clr)
- net at U85.8, U88.13, U95.2: now also U88.10
- net ~{SP DOWN} renamed ~{SP. DOWN}
Other:
- moved on the sheet: U106A, U107B, U29C

Commit message: another error
Parts:
- C36: footprint Capacitor_THT:C_Disc_D7.5mm_W5.0mm_P7.50mm -> Capacitor_THT:C_Disc_D4.3mm_W1.9mm_P5.00mm
- U105, U115: footprint Package_DIP:DIP-16_W15.24mm -> Package_DIP:DIP-16_W7.62mm
Connections:
- net ACCE. A: now also U7.10 (A0)
- net GNDPWR: now also C36.2, U105.8 (GND), U115.15 (~{G})
- net VCC: no longer U7.10 (A0)
- net at U113.1 (B3): now also U112.8 (Q3); no longer U112.11 (Q0)
- net at U113.11 (B1): now also U112.10 (Q1); no longer U112.9 (Q2)
- net at U113.14 (B2): now also U112.9 (Q2); no longer U112.10 (Q1)
- net at U113.9 (B0): now also U112.11 (Q0); no longer U112.8 (Q3)
- net at U92.3 (C): now also U93.6; no longer U93.8
- net at U92.5 (Q): now also U100.4 (2C); no longer U100.2 (2A)
- net ~{Vb}: now reaches U104.10 (CET), U117.10 (CET), U90.10 (CET)
- net at U92.11 (C): now also U93.8; no longer U93.6
- net at U92.9 (Q): now also U100.2 (2A); no longer U100.4 (2C)
Other:
- moved on the sheet: U112B, U92A, U92B

Commit message: fix some of my own mistakes
Parts:
- added C37: 0.1m, Capacitor_THT:C_Disc_D4.3mm_W1.9mm_P5.00mm, symbol Device:C_Polarized_US
- added R23: 560, Resistor_THT:R_Axial_DIN0309_L9.0mm_D3.2mm_P12.70mm_Horizontal, symbol Device:R_US
- added R24: 100, Resistor_THT:R_Axial_DIN0309_L9.0mm_D3.2mm_P12.70mm_Horizontal, symbol Device:R_US
- J1: symbol Connector:Conn_01x36_Pin -> Connector_Generic:Conn_02x36_Top_Bottom
Connections:
- net A22 is gone; now on net GNDPWR: J1.22 (Pin_22)
- net A7 is gone; now on net GNDPWR: J1.7 (Pin_7)
- net COIN IN (B) is gone; now on net B1: U37.12 (D), U37.5 (Q), U72.8
- net EXTEND (A) is gone; now on net B9: U33.2 (D)
- net RET1 is gone; now on net GNDPWR: TR1.3 (E)
- net ROAD is gone; now on net B7: U14.12
- net ~{COIN IN} (B) is gone; now on net ~{COIN IN}: U31.11, U37.6 (~{Q})
- net ~{EX.SIGNAL CP} is gone; now on net B2: U49.1 (A), U50.3 (C), U55.3
- net ~{RESCUE(Y)} is gone; now on net B8: U14.9
- net ~{SCORE.ST} is gone; now on net ~{SCORE ST.}: U119.4 (~{Q})
- net A23: now also RA1.6 (R5), RA2.4 (R3); no longer D1.2 (A), RA1.8 (R7)
- net A24: now also RA1.4 (R3), RA2.6 (R5); no longer RA1.5 (R4), RA2.5 (R4)
- net A25: now also RA1.3 (R2), RA2.7 (R6)
- net A32: now also R23.2, R24.1; no longer SW2.3 (C)
- net A8: now also U1.2 (B), U3.3 (I3a)
- net B8: no longer U38.10 (B), U50.9 (Q)
- net B9: now also U38.10 (B), U50.9 (Q)
- net GNDPWR: now also J1.37 (Pin_37), J1.38 (Pin_38), J1.39 (Pin_39), J1.40 (Pin_40), J1.41 (Pin_41), J1.45 (Pin_45), J1.57 (Pin_57), J1.58 (Pin_58), U4.8 (GND), C37.2
- net VCC: now also J1.69 (Pin_69), J1.70 (Pin_70), J1.71 (Pin_71), J1.72 (Pin_72), RA1.1 (common), R23.1
- net ~{COIN&TEST}: now also U24.11 (~{LOAD}), U25.11 (~{LOAD}), U35.11 (~{LOAD}), U36.11 (~{LOAD})
- net at U27.10 (~{R}): no longer U44.12
- net at U27.11 (~{S1}): no longer U14.6
- net at U27.9 (Q): no longer U16.10
- net at U39.10 (Q1): now also U45.3
- net at U39.8 (Q3): now also U45.5, U72.3
- net at U39.9 (Q2): now also U45.4
- net Af: now reaches RA1.7 (R6), RA2.3 (R2)
- net Af: now also J1.68 (Pin_68)
- net at U10.11 (B1), U4.10 (S1), U6.2: now also U80.13; no longer U14.5, U6.13
- net at U10.14 (B2), U4.9 (S2), U6.4: no longer U80.13
- net at U17.10 (A0): now also U19.3 (Q0); no longer U19.11 (Q0)
- net at U17.12 (A1): now also U19.4 (Q1); no longer U19.10 (Q1)
- net at U17.13 (A2): now also U19.5 (Q2); no longer U19.9 (Q2)
- net at U32.10 (~{R}): now also C37.1, R24.2
- net at U63.11: now also U19.6 (Q3); no longer U19.8 (Q3)
- net at U18.3 (Ia=b), U63.13: now also U19.13 (CP); no longer U19.1 (CP)
- net at U18.10 (A0): now also U19.11 (Q0); no longer U19.3 (Q0)
- net at U18.12 (A1): now also U19.10 (Q1); no longer U19.4 (Q1)
- net at U18.13 (A2): now also U19.9 (Q2); no longer U19.5 (Q2)
- net at U27.13 (Q): now also U16.10
- net at U27.14 (~{R}): now also U44.12
- net at U27.15 (~{S}): now also U14.6
- net A4: no longer names the net of SW2.1 (A)
- net ~{BRIDGE(W)} renamed BH
- new net: RA1.5 (R4), RA2.5 (R4)
- new net: D1.2 (A), RA1.8 (R7)
- new net: U14.5, U6.13
- new net: U18.15 (A3), U19.1 (CP), U19.8 (Q3)
- new net AF: J1.42 (Pin_42)
- new net AG: J1.43 (Pin_43)
- new net AH: J1.44 (Pin_44)
- new net AJ: J1.46 (Pin_46)
- new net AK: J1.47 (Pin_47)
- new net AL: J1.48 (Pin_48)
- new net AM: J1.49 (Pin_49)
- new net AN: J1.50 (Pin_50)
- new net AO: J1.51 (Pin_51)
- new net AP: J1.52 (Pin_52)
- new net AQ: J1.53 (Pin_53)
- new net AR: J1.54 (Pin_54)
- new net AS: J1.55 (Pin_55)
- new net AT: J1.56 (Pin_56)
- new net AW: J1.59 (Pin_59)
- new net AX: J1.60 (Pin_60)
- new net AY: J1.61 (Pin_61)
- new net AZ: J1.62 (Pin_62)
- new net Aa: J1.63 (Pin_63)
- new net Ab: J1.64 (Pin_64)
- new net Ac: J1.65 (Pin_65)
- new net Ad: J1.66 (Pin_66)
- new net Ae: J1.67 (Pin_67)
- no-connect marks 79 -> 81
Other:
- moved on the sheet: J2, J3, U19A, U19B, U27C, U27D, U39B

Commit message: aaaaaaaaaaaaaa
Parts:
- removed RA2: 100, Resistor_THT:R_Array_SIP8, symbol Device:R_Network07_US
- removed SW2: CREDIT, TestPoint:TestPoint_Pad_1.0x1.0mm, symbol Switch:SW_SPDT
- removed SW3: TEST, TestPoint:TestPoint_Pad_1.0x1.0mm, symbol Switch:SW_SPDT
- removed SW4: COIN, TestPoint:TestPoint_Pad_1.0x1.0mm, symbol Switch:SW_SPDT
- added C13: 0.01m, Capacitor_THT:CP_Radial_Tantal_D4.5mm_P2.50mm, symbol Device:C_Polarized_US
- added C16: 470p, Capacitor_THT:C_Disc_D4.3mm_W1.9mm_P5.00mm, symbol Device:C_Polarized_US
- added C36: 0.1m, Capacitor_THT:C_Disc_D7.5mm_W5.0mm_P7.50mm, symbol Device:C_Polarized_US
- added C38: 680p, Capacitor_THT:C_Disc_D4.7mm_W2.5mm_P5.00mm, symbol Device:C_Polarized_US
- added C6: 680p, Capacitor_THT:C_Disc_D7.5mm_W5.0mm_P7.50mm, symbol Device:C_Polarized_US
- added C8, C9: 0.1u, Capacitor_THT:C_Disc_D7.5mm_W5.0mm_P7.50mm, symbol Device:C_Polarized_US
- added RN2: R_Pack08_Split, Package_DIP:DIP-16_W7.62mm, symbol Device:R_Pack08_Split
- added unit 3 of U112
- added V1: 1, Capacitor_THT:C_Disc_D7.5mm_W5.0mm_P7.50mm, symbol Simulation_SPICE:VDC
- C11, C37: footprint Capacitor_THT:C_Disc_D4.3mm_W1.9mm_P5.00mm -> Capacitor_THT:C_Disc_D7.5mm_W5.0mm_P7.50mm
- C12: footprint Capacitor_THT:C_Disc_D7.5mm_W5.0mm_P7.50mm -> Capacitor_THT:CP_Radial_Tantal_D4.5mm_P5.00mm
- C14: footprint Capacitor_THT:CP_Radial_Tantal_D8.0mm_P5.00mm -> Capacitor_THT:C_Disc_D7.5mm_W5.0mm_P10.00mm
- Cp1, Cp10, Cp11, Cp12, Cp13, Cp14, Cp15, Cp16, Cp17, Cp18, Cp19, Cp2, Cp20, Cp21, Cp22, Cp23, Cp24, Cp25, Cp26, Cp27, Cp28, Cp29, Cp3, Cp30, Cp31, Cp32, Cp33, Cp34, Cp35, Cp36, Cp37, Cp38, Cp39, Cp4, Cp5, Cp6, Cp7, Cp8, Cp9: footprint Capacitor_THT:C_Disc_D7.5mm_W5.0mm_P7.50mm -> Capacitor_THT:C_Disc_D7.5mm_W5.0mm_P10.00mm
- renumbered C6 to C40, C9 to C42, C8 to C66, C36 to C86
Connections:
- net A10 is gone; now on net GNDPWR: J1.10 (Pin_10)
- net AG is gone; now on net VCC: J1.43 (Pin_43)
- net AJ is gone; now on net VCC: J1.46 (Pin_46)
- net AO is gone; now on net AS: J1.51 (Pin_51)
- net AP is gone; now on net AT: J1.52 (Pin_52)
- net AQ is gone; now on net AU: J1.53 (Pin_53)
- net AR is gone; now on net AV: J1.54 (Pin_54)
- net EXPLO.SEL. A is gone; now on net EXPLO. SEL. A: U63.9, U65.1 (A7)
- net EXPLO.SEL. B is gone; now on net EXPLO. SEL. B: U65.23 (A8)
- net EXPLO.SEL. C is gone; now on net EXPLO. SEL. C: U63.8
- net ~{ACC I.} is gone; now on net ~{ACCI.}: U59.18 (CE2), U59.19 (CE3), U66.1, U95.5, U95.9
- net ~{ACCI.PULSE} is gone; now on net ~{ACCI. PULSE}: U34.2
- net ~{EXPLO.ST.} is gone; now on net ~{EXPLO. ST.}: U74.3
- net ~{EXPLO.ST.}(G) is gone; now on net ~{EXPLO. ST.}: U33.6 (~{Q}), U39.2 (MR)
- net A23: now also RN2.12 (R5.2)
- net A24: now also RN2.14 (R3.2)
- net A25: now also RN2.15 (R2.2)
- net A26: now also C7.1, RA1.2 (R1), RN2.16 (R1.2)
- net ACCE.ST: no longer U37.11 (C)
- net AM: now also U6.11
- net AREA 4: no longer C11.1
- net AS: now also U21.3 (QA); no longer J1.55 (Pin_55)
- net AT: now also U21.7 (QD); no longer J1.56 (Pin_56)
- net AW: now also J1.55 (Pin_55); no longer J1.59 (Pin_59)
- net AX: now also J1.56 (Pin_56); no longer J1.60 (Pin_60)
- net AY: now also J1.59 (Pin_59); no longer J1.61 (Pin_61)
- net AZ: now also J1.60 (Pin_60); no longer J1.62 (Pin_62)
- net Aa: now also J1.61 (Pin_61); no longer J1.63 (Pin_63)
- net Ab: now also J1.62 (Pin_62); no longer J1.64 (Pin_64)
- net Ac: now also J1.63 (Pin_63); no longer J1.65 (Pin_65)
- net Ad: now also J1.64 (Pin_64); no longer J1.66 (Pin_66)
- net Ae: now also J1.65 (Pin_65); no longer J1.67 (Pin_67)
- net Af: now also J1.66 (Pin_66), RN2.11 (R6.2); no longer J1.68 (Pin_68)
- net B15: no longer U114.2
- net B6: now also U5.2 (MR)
- net C15: now also J3.15 (Pin_15)
- net C16: now also J3.16 (Pin_16)
- net C17: now also J3.17 (Pin_17)
- net GNDPWR: now also U111.20 (~{CE}1_(PVCE)), U58.8 (GND), U69.8 (GND), C16.2, C36.2, C38.2, C6.2, C8.2, C9.2, U112.7 (GND), V1.2
- net PL-V-ST: no longer U52.12 (MR), U52.2 (MR)
- net VCC: now also U111.18 (CE2), U111.19 (CE3), U15.16 (VCC), U69.16 (VCC), U112.14 (VCC), V1.1
- net Vs/32: now also U39.13 (CP), C38.1
- net Vs/4: now also U77.23 (A8)
- net ~{ACCI.ST}: no longer U119.11 (Clr), U51.7 (Q), U62.4
- net at U119.2 (B), U68.3: now also U119.10 (B)
- net at U34.8, U39.1 (CP): now also C16.1
- net at U39.12 (MR): now also U62.6
- net at U48.5: now also U46.12
- net ~{EXPLO. ST.}: now reaches U68.1, U84.18 (CE2), U84.19 (CE3), U91.18 (CE2), U91.19 (CE3), U98.18 (CE2), U98.19 (CE3)
- net at U32.15 (~{S}): now also RN2.1 (R1.1); no longer C7.1
- net at U48.13, U54.10 (Q1), U59.3 (A5): now also U45.13, U46.13
- net at C12.1, R7.1, U38.1 (A): no longer C14.1
- net C14: now reaches J3.14 (Pin_14)
- net C18: now reaches J3.18 (Pin_18)
- net C19: now reaches J3.19 (Pin_19)
- net ~{ACCI. PULSE}: now reaches U45.6
- net at RA1.5 (R4): now also RN2.13 (R4.2)
- net at U124.1 (OEa), U124.15 (OEb): now also C42.1, U68.8
- net at U4.10 (S1), U6.2: now also U6.13; no longer U10.11 (B1), U80.13
- net at U4.11 (S0), U6.6: no longer U10.9 (B0)
- net at U4.9 (S2), U6.4: no longer U10.14 (B2)
- net at U14.5: no longer U6.13
- net at U95.1, U95.13, U97.14 (I6): now also U123.12
- net at U32.1 (~{R}): now also C11.1
- net at U32.2 (~{S1}), U32.3 (~{S2}): now also C8.1
- net PL-H-ST.: now reaches U17.6 (Oa=b)
- net at U32.5 (~{R}): now also C6.1
- net at U32.6 (~{S}): now also C9.1, RN2.5 (R5.1)
- net AU: now reaches U20.3 (QA)
- net AV: now reaches U20.7 (QD)
- net ACCI. renamed ~{ACCI.}
- net CAR.CONT.CL renamed CAR CONT. CL
- net EXPLO.ST.(G) renamed EXPLO. ST.
- net ~{EXTEND} (A) renamed ~{EXTEND}
- new net: C36.1, RN2.10 (R7.2)
- new net: C14.1, RN2.8 (R8.1)
- new net: U10.14 (B2), U80.13
- new net ACCE. ST.: U37.11 (C)
- new net Ag: J1.67 (Pin_67)
- new net Ah: J1.68 (Pin_68)
- new net PL-H-ST: U52.12 (MR), U52.2 (MR)
- new net ~{ACCI. ST}: U119.11 (Clr), U51.7 (Q), U62.4
- new net ~{OTHER TIRE}: U114.2
- no-connect marks 81 -> 114
Other:
- title: (none) -> 97091X-P
- moved on the sheet: C11, C14, C7, U27C, U32B, U46F, U6F
