File: Main/Main.kicad_sch (KiCad schematic)
At the start: 248 parts, among them J1 Conn_01x36_Pin, J2 Conn_01x22, J3 Conn_01x28_Pin, SW1 1COIN 1PLAY/1COIN 2PLAY, SW5 TILT SW., U1 74LS123, U10 74LS85, U100 7450, U101 74LS161, U102 74LS161, U103 74LS157, U104 74LS161, U105 74S288, U106 74LS08, U107 74LS10, U108 74LS157, U109 74LS161, U11 74LS85, U110 74LS367, U111 MB7137, U112 74LS393, U113 74LS85, U114 74LS04, U115 74S288, U116 74LS161, U117 74LS161, U118 74LS157, U119 74LS123, U12 74LS00, U120 74LS123, U121 74LS123, U122 74LS02, U123 74LS10, U124 74LS367, U125 74LS11, U13 74LS07, U14 74LS20, U15 74LS193, U16 74LS86, U17 74LS85, U18 74LS85, U19 74LS393, U2 74LS08, U20 74LS192, U21 74LS192, U22 74LS08, U23 74LS32, U24 74LS193, U25 74LS193, U26 NE555P, U27 74LS279, U28 74LS10, U29 74LS07P, U3 74LS153, U30 74LS00, U31 74LS07P, U32 74LS279, U33 74LS74, U34 74LS08, U35 74LS193, U36 74LS193, U37 74LS74, U38 74LS123, U39 74LS393, U4 74LS151, U40 74LS393, U41 74LS85, U42 74LS85, U43 74LS123, U44 74LS04, U45 74LS10, U46 74LS04, U47 74LS20, U48 74LS00, U49 74LS123, U5 74LS393, U50 74LS74, U51 74LS279, U52 74LS393, U53 74LS85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

Commit message: power hookup
Connections:
- net A26: no longer C7.1
- net at RN2.1 (R1.1), U32.15 (~{S}): now also C7.1
Other:
- moved on the sheet: C7
Changed lines of the file:
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@@
   (junction (at 715.01 422.275) (diameter 0) (color 0 0 0 0)
   )
+  (junction (at 700.405 75.565) (diameter 0) (color 0 0 0 0)
+  )
   (junction (at 887.095 200.025) (diameter 0) (color 0 0 0 0)
   )
@@
     )
   )
-  (symbol (lib_id "Device:C_Polarized_US") (at 692.785 79.375 0) (unit 1)
+  (symbol (lib_id "Device:C_Polarized_US") (at 700.405 79.375 0) (unit 1)
     (in_bom yes) (on_board yes) (dnp no)
-    (property "Reference" "C7" (at 693.42 82.55 0)
+    (property "Reference" "C7" (at 701.04 82.55 0)
       (effects (font (size 1.27 1.27)) (justify left))
     )
-    (property "Value" "0.1u" (at 692.785 84.455 0)
+    (property "Value" "0.1u" (at 700.405 84.455 0)
       (effects (font (size 1.27 1.27)) (justify left))
     )
-    (property "Footprint" "Capacitor_THT:C_Disc_D7.5mm_W5.0mm_P7.50mm" (at 692.785 79.375 0)
+    (property "Footprint" "Capacitor_THT:C_Disc_D7.5mm_W5.0mm_P7.50mm" (at 700.405 79.375 0)
       (effects (font (size 1.27 1.27)) hide)
     )
-    (property "Datasheet" "~" (at 692.785 79.375 0)
+    (property "Datasheet" "~" (at 700.405 79.375 0)
       (effects (font (size 1.27 1.27)) hide)
     )
@@
     )
   )
-  (symbol (lib_id "power:GNDPWR") (at 692.785 83.185 0) (unit 1)
+  (symbol (lib_id "power:GNDPWR") (at 700.405 83.185 0) (unit 1)
     (in_bom yes) (on_board yes) (dnp no) (fields_autoplaced)
-    (property "Reference" "#PWR0112" (at 692.785 88.265 0)
+    (property "Reference" "#PWR0112" (at 700.405 88.265 0)
       (effects (font (size 1.27 1.27)) hide)
     )
-    (property "Value" "GNDPWR" (at 692.658 86.995 0)
+    (property "Value" "GNDPWR" (at 700.278 86.995 0)
       (effects (font (size 1.27 1.27)))
     )
-    (property "Footprint" "" (at 692.785 84.455 0)
+    (property "Footprint" "" (at 700.405 84.455 0)
       (effects (font (size 1.27 1.27)) hide)
     )
-    (property "Datasheet" "" (at 692.785 84.455 0)
+    (property "Datasheet" "" (at 700.405 84.455 0)
       (effects (font (size 1.27 1.27)) hide)
     )

Commit message: card edge B
Parts:
- J2: symbol Connector_Generic:Conn_01x22 -> Connector_Generic:Conn_02x22_Top_Bottom
- J3: symbol Connector:Conn_01x28_Pin -> Connector_Generic:Conn_02x28_Top_Bottom
Connections:
- net AH is gone; now on net AJ: J1.44 (Pin_44)
- net AK is gone; now on net AM: J1.47 (Pin_47)
- net AL is gone; now on net AN: J1.48 (Pin_48)
- net B17 is gone; now on net B12: J2.17 (Pin_17)
- net C11 is gone; now on net AREA 5: J3.11 (Pin_11)
- net C13 is gone; now on net 7MHz: J3.13 (Pin_13)
- net C14 is gone; now on net ~{GRAVEL}: J3.14 (Pin_14)
- net C9 is gone; now on net AREA 3: J3.9 (Pin_9)
- net H4 is gone; now on net C8: U68.12
- net H5 is gone; now on net C7: U74.2
- net S-ACCE. C is gone; now on net AN: U13.4
- net SHIFT is gone; now on net AW: U29.8
- net SP. CONT. is gone; now on net Ah: C86.1, U115.14 (A4)
- net V7 is gone; now on net B18: U47.9, U67.4 (2C), U67.9 (1C)
- net Vs/16 is gone; now on net B21: U12.10, U29.5, U60.2 (I0a), U73.11, U78.1 (CP), U79.8 (Q3), U85.1, U95.4
- net Vs/2 is gone; now on net B2: U107.11, U30.5, U60.5 (I0b), U79.11 (Q0)
- net Vs/32 is gone; now on net B20: C38.1, U39.13 (CP), U66.10, U72.5, U78.3 (Q0)
- net ~{ACCI.ST} is gone; now on net ~{ACCI. ST}: U80.3
- net ~{HISCORE} (S) is gone; now on net Af: U31.12
- net ~{SLIPZONE} is gone; now on net AX: U29.4
- net 8000: now also J2.31 (Pin_31)
- net A23: now also RA1.7 (R6), RN2.11 (R6.2); no longer RA1.6 (R5), RN2.12 (R5.2)
- net A24: now also RA1.5 (R4), RN2.13 (R4.2); no longer RA1.4 (R3), RN2.14 (R3.2)
- net A26: no longer RA1.2 (R1), RN2.16 (R1.2)
- net AM: no longer J1.49 (Pin_49)
- net AN: no longer J1.50 (Pin_50)
- net AREA 4: now also J3.10 (Pin_10)
- net AREA 5: no longer J3.10 (Pin_10)
- net AY: no longer J1.59 (Pin_59)
- net AZ: no longer J1.60 (Pin_60)
- net Aa: now also J1.59 (Pin_59), RA1.6 (R5), RN2.12 (R5.2); no longer J1.61 (Pin_61)
- net Ab: now also J1.60 (Pin_60), RA1.4 (R3), RN2.14 (R3.2); no longer J1.62 (Pin_62)
- net Ac: now also J1.61 (Pin_61), RA1.2 (R1), RN2.16 (R1.2); no longer J1.63 (Pin_63)
- net Ad: now also J1.62 (Pin_62), U31.4; no longer J1.64 (Pin_64)
- net Ae: now also J1.63 (Pin_63), U31.8; no longer J1.65 (Pin_65)
- net Af: now also J1.64 (Pin_64); no longer J1.66 (Pin_66), RA1.7 (R6), RN2.11 (R6.2)
- net Ag: no longer J1.67 (Pin_67)
- net Ah: now also J1.65 (Pin_65); no longer J1.68 (Pin_68)
- net B18: now also J2.35 (Pin_35)
- net B6: no longer U31.8
- net BH: now also J2.30 (Pin_30)
- net GNDPWR: now also J3.53 (Pin_53), J3.54 (Pin_54), J3.55 (Pin_55), J3.56 (Pin_56), U12.7 (GND), U120.8 (GND), U121.8 (GND), U95.7 (GND); no longer U12.14 (VCC), U120.16 (VCC), U121.16 (VCC), U95.14 (VCC)
- net VCC: now also J3.48 (Pin_48), J3.49 (Pin_49), J3.50 (Pin_50), J3.51 (Pin_51), U12.14 (VCC), U120.16 (VCC), U121.16 (VCC), U95.14 (VCC); no longer U12.7 (GND), U120.8 (GND), U121.8 (GND), U95.7 (GND)
- net ~{COIN&TEST}: no longer U31.4
- net at C12.1, R7.1, U38.1 (A): now also C13.1, C13.2, C14.1, RN2.8 (R8.1)
- net at D1.2 (A), RA1.8 (R7): now also RN2.9 (R8.2)
- net Al: now reaches RA1.9 (R8)
- net Al: now also J1.68 (Pin_68), RN2.7 (R7.1)
- net at RN2.2 (R2.1): now also C10.1, U32.14 (~{R})
- net at U6.13, U6.2: no longer U4.10 (S1)
- net at U4.11 (S0), U6.6: now also U10.9 (B0)
- net at U6.4: now also U10.11 (B1), U4.10 (S1); no longer U4.9 (S2)
- net at C8.1, U32.2 (~{S1}), U32.3 (~{S2}): now also RN2.3 (R3.1)
- net at C6.1, U32.5 (~{R}): now also RN2.4 (R4.1)
- net Aj: now reaches AE1.1 (A), D1.1 (K), SW5.2 (B)
- net Aj: now also J1.66 (Pin_66)
- net AJ: now reaches U1.10 (B), U3.13 (I3b)
- net at U10.14 (B2), U80.13: now also U4.9 (S2)
- net EXPLO. SEL. D renamed BM
- net BM: now also J2.34 (Pin_34)
- net H6 renamed CH
- net H8 renamed CF
- net S-ACCE. A renamed AP
- net AP: now also J1.49 (Pin_49)
- net S-ACCI. renamed AR
- net AR: now also J1.50 (Pin_50)
- net V4 renamed BT
- net BT: now also J2.38 (Pin_38)
- net V5 renamed BU
- net BU: now also J2.39 (Pin_39)
- net Vs/4 renamed BY
- net Vs/64 renamed BX
- net ~{EXT. 500} renamed BZ
- net BZ: now also J2.44 (Pin_44)
- net ~{INI. RESET} renamed Ak
- net Ak: now also J1.67 (Pin_67)
- net ~{POOL} renamed CM
- net ~{SLIP} renamed CA
- net CA: now also J3.29 (Pin_29)
- net ~{TUNNEL} renamed BF
- net BF: now also J2.28 (Pin_28)
- new net BA: J2.23 (Pin_23)
- new net BB: J2.24 (Pin_24)
- new net BC: J2.25 (Pin_25)
- new net BD: J2.26 (Pin_26)
- new net BE: J2.27 (Pin_27)
- new net BG: J2.29 (Pin_29)
- new net BK: J2.32 (Pin_32)
- new net BL: J2.33 (Pin_33)
- new net BP: J2.36 (Pin_36)
- new net BQ: J2.37 (Pin_37)
- new net BV: J2.40 (Pin_40)
- no-connect marks 114 -> 115
Other:
- moved on the sheet: C13, C14, RN2B, RN2H, U120C, U121C, U12E, U4, U6A, U6B, U95E
