File: Video/Video.kicad_sch (KiCad schematic)
At the start: 28 parts, among them Q1 Q_NPN_BCE, U1 74LS07, U10 74LS32, U13 74LS30, U16 74LS07, U19 74LS12, U2 74LS147, U3 74LS04, U4 74LS30, U5 74LS157, U6 74LS42, U7 74LS06, U79 74LS174, U8 74LS12, U86 74LS368, U9 74LS00

Commit message: mroe chips
Parts:
- added RN1: 560, Resistor_THT:R_Array_SIP9, symbol Device:R_Network08_US
- added U11, U20: 74LS157, Package_DIP:DIP-16_W7.62mm, symbol 74xx:74LS157
- added U12, U17: MB7137, Package_DIP:DIP-24_W15.24mm, symbol Memory_PROM:MB7137
- added U14: 74LS20, Package_DIP:DIP-14_W7.62mm, symbol 74xx:74LS20
- added U15: 74LS09, Package_DIP:DIP-14_W7.62mm, symbol 74xx:74LS09
- added U18: 74LS123, Package_DIP:DIP-16_W7.62mm, symbol 74xx:74LS123
- added U21: 74LS11, Package_DIP:DIP-14_W7.62mm, symbol 74xx:74LS11
- Q1: footprint Package_TO_SOT_THT:TO-92 -> Package_TO_SOT_THT:TO-92L_Inline
Connections:
- net VCC: now also RN1.1 (common)
- net at U13.3, U8.12, U9.10: now also U14.5
- net at U9.9: now also U14.8
- net at U3.10: now also U2.10 (E9)
- net at D1.1 (K), D2.1 (K), D3.1 (K)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: now also RN1.6 (R5)
- net ~{LIGHT}: now reaches U19.3
- net ~{LIGHT}: now also U15.2
- net TUNNEL AP: now reaches U19.4
- net at U2.4 (E7): now also U3.4
- net at U2.5 (E8): now also U3.2
- net at U19.1: now also U10.8
- net at U10.2: now also U15.3
- net at U10.3: now also U20.5 (I0b)
- net at Q1.1 (B), U7.4: now also RN1.5 (R4)
- net ~{TV-BLANKING}: now reaches U7.3
- net at U5.7 (Zb): now also U10.9
- net ~{SYNCRO}: now reaches U7.5
- net ~{EXTEND}: now reaches U10.10
- net at U4.3: now also U20.12 (Zd)
- net at U19.10: now also U21.6
- net at U19.11: now also U20.13 (I1d)
- net at U19.8: now also U20.14 (I0d)
- net ~{ROAD}: now reaches U19.9
- net ~{ROAD}: now also U15.1
- new net: U12.1 (A7), U17.1 (A7)
- new net: U11.5 (I0b), U12.10 (D1), U17.10 (D1)
- new net: U11.11 (I0c), U12.11 (D2), U17.11 (D2)
- new net: U11.14 (I0d), U12.13 (D3), U12.17 (D7), U17.13 (D3)
- new net: U11.3 (I1a), U12.14 (D4), U17.14 (D4)
- new net: U11.6 (I1b), U12.15 (D5), U17.15 (D5)
- new net: U11.10 (I1c), U12.16 (D6), U17.16 (D6)
- new net: U11.13 (I1d), U17.17 (D7)
- new net: U12.2 (A6), U17.2 (A6)
- new net: U12.3 (A5), U17.3 (A5)
- new net: U12.4 (A4), U17.4 (A4)
- new net: U12.5 (A3), U17.5 (A3)
- new net: U12.6 (A2), U17.6 (A2)
- new net: U12.7 (A1), U17.7 (A1)
- new net: U12.8 (A0), U17.8 (A0)
- new net: U11.2 (I0a), U12.9 (D0), U17.9 (D0)
- new net E10: U14.10
- new net ~{GRASSAREA}: U21.4
- new net ~{HOUSE ST}: U21.3
- new net ~{SLIP}: U14.9
- new net ~{TREE&GRASS}: U20.2 (I0a), U20.6 (I1b), U21.5
Other:
- note added: "TV-BLUE"
- note added: "TV-GREEN"
- note added: "TV-RED"
- note added: "TV-SYNC"
- moved on the sheet: D1, D2, D3, Q1, R1, R13, R14, R15, R2, R3, R4, R5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

Commit message: aaaaaaaaaaaaaa
Parts:
- added U22: 74LS06, Package_DIP:DIP-14_W7.62mm, symbol 74xx:74LS06
- added U23: 74LS86, Package_DIP:DIP-14_W7.62mm, symbol 74xx:74LS86
- added U24: 74LS42, Package_DIP:DIP-16_W7.62mm, symbol 74xx:74LS42
Connections:
- net D10: now also RN1.9 (R8)
- net D13: no longer D2.2 (A), R14.2, R3.2, R4.2, U16.10
- net at U11.14 (I0d), U12.13 (D3), U17.13 (D3): no longer U12.17 (D7)
- net at U11.13 (I1d), U17.17 (D7): now also U12.17 (D7)
- net at U17.20 (~{CE}1_(PVCE)): now also U12.19 (CE3)
- net at U17.23 (A8): now also U12.23 (A8)
- net at U12.4 (A4), U17.4 (A4): now also U21.8
- net at U12.5 (A3), U17.5 (A3): now also U23.3
- net at U12.6 (A2), U17.6 (A2): now also U23.11
- net at U12.7 (A1), U17.7 (A1): now also U23.6
- net at U12.8 (A0), U17.8 (A0): now also U23.8
- new net D12: D2.2 (A), R14.2, R3.2, R4.2, U16.10

Commit message: vidoeodeoeo
Parts:
- added U201, U49: 74LS393, Package_DIP:DIP-14_W7.62mm, symbol 74xx:74LS393
- added U202, U29, U43, U50: 74LS157, Package_DIP:DIP-16_W7.62mm, symbol 74xx:74LS157
- added U25, U31, U35, U38, U40: 74LS74, Package_DIP:DIP-14_W7.62mm, symbol 74xx:74LS74
- added U26: 74LS20, Package_DIP:DIP-14_W7.62mm, symbol 74xx:74LS20
- added U27, U33: 74LS30, Package_DIP:DIP-14_W7.62mm, symbol 74xx:74LS30
- added U28: 74LS86, Package_DIP:DIP-14_W7.62mm, symbol 74xx:74LS86
- added U30, U51: MB7137, Package_DIP:DIP-24_W15.24mm, symbol Memory_PROM:MB7137
- added U32: 74LS21, Package_DIP:DIP-14_W7.62mm, symbol 74xx:74LS21
- added U34: 74LS02, Package_DIP:DIP-14_W7.62mm, symbol 74xx:74LS02
- added U36, U37: 74LS161, Package_DIP:DIP-16_W7.62mm, symbol 74xx:74LS161
- added U39: 74LS32, Package_DIP:DIP-14_W7.62mm, symbol 74xx:74LS32
- added U41, U48: 74LS151, Package_DIP:DIP-16_W7.62mm, symbol 74xx:74LS151
- added U42, U44, U55, U66: 74LS10, Package_DIP:DIP-14_W7.62mm, symbol 74xx:74LS10
- added U45, U56: 74LS00, Package_DIP:DIP-14_W7.62mm, symbol 74xx:74LS00
- added U46: 74LS193, Package_DIP:DIP-16_W7.62mm, symbol 74xx:74LS193
- added U47, U52, U58: 74LS08, Package_DIP:DIP-14_W7.62mm, symbol 74xx:74LS08
- added U53: 74LS153, Package_DIP:DIP-16_W7.62mm, symbol 74xx:74LS153
- added U54: 74LS42, Package_DIP:DIP-16_W7.62mm, symbol 74xx:74LS42
- added U57: 74LS107, Package_DIP:DIP-14_W7.62mm, symbol 74xx:74LS107
- added unit 4 of U9
- added unit 5 of U9
- Q1: footprint Package_TO_SOT_THT:TO-92L_Inline -> Package_TO_SOT_THT:TO-92L_Inline_Wide; symbol Device:Q_NPN_BCE -> Device:Q_NPN_ECB
Connections:
- net D11: now also U7.8; no longer U16.8
- net D12: now also U7.10; no longer U16.10
- net D13: now also U7.12; no longer U16.12
- net GNDPWR: now also Q1.1 (E), U1.7 (GND), U10.7 (GND), U11.8 (GND), U12.12 (GND), U13.7 (GND), U14.7 (GND), U15.7 (GND), U16.7 (GND), U17.12 (GND), U18.8 (GND), U19.7 (GND), U20.8 (GND), U21.7 (GND), U22.7 (GND), U23.7 (GND), U24.8 (GND), U3.7 (GND), U4.7 (GND), U5.15 (E), U7.7 (GND), U8.7 (GND), U25.7 (GND), U26.7 (GND), U27.7 (GND), U28.7 (GND), U29.8 (GND), U30.12 (GND), U31.7 (GND), U51.12 (GND); no longer Q1.3 (E)
- net VCC: now also U1.14 (VCC), U10.14 (VCC), U11.16 (VCC), U12.24 (VCC_(PVCC)), U13.14 (VCC), U14.14 (VCC), U15.14 (VCC), U16.14 (VCC), U17.24 (VCC_(PVCC)), U18.16 (VCC), U19.14 (VCC), U20.16 (VCC), U21.14 (VCC), U22.14 (VCC), U23.14 (VCC), U24.16 (VCC), U3.14 (VCC), U4.14 (VCC), U5.16 (VCC), U6.16 (VCC), U7.14 (VCC), U8.14 (VCC), U201.14 (VCC), U202.16 (VCC), U25.14 (VCC), U27.14 (VCC), U28.14 (VCC), U29.16 (VCC), U30.24 (VCC_(PVCC)), U31.14 (VCC), U32.14 (VCC), U33.14 (VCC), U34.14 (VCC), U35.14 (VCC), U36.16 (VCC), U37.16 (VCC), U38.14 (VCC), U39.14 (VCC), U40.14 (VCC), U41.16 (VCC), U41.4 (I0), U42.14 (VCC), U43.16 (VCC), U44.14 (VCC), U47.1, U47.14 (VCC), U48.1 (I3), U48.16 (VCC), U51.24 (VCC_(PVCC)), U9.14 (VCC)
- net ~{TV-BLANKING}: now also U7.1; no longer U7.3
- net at U16.13: no longer U2.6 (S2)
- net ~{OTHER CAR}: now reaches U8.1
- net ~{GRAVEL}: now reaches U8.13
- net ~{GRAVEL}: now also U15.4
- net at U8.2: now also U19.5, U45.13, U66.12
- net V-(H): now reaches U9.4
- net ~{BRIDGE (DBu)}: now reaches U9.5
- net at U9.6: now also U5.3 (I1a)
- net at U2.10 (E9), U3.10: now also U13.5
- net at U3.11: now also U33.8
- net at D1.1 (K), D2.1 (K), D3.1 (K)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: now also RN1.5 (R4); no longer RN1.6 (R5)
- net at U22.2: now also U11.15 (E)
- net at U10.11: now also U12.18 (CE2)
- net ~{GREEN BELT}: now reaches U13.11
- net at U13.2: now also U19.11, U20.13 (I1d)
- net ~{Y-LINE}: now reaches U13.4
- net ~{Y-LINE}: now also U5.11 (I0c)
- net at U23.5: now also U23.12, U23.2, U23.9
- net ~{RESCUE(Bc)}: now reaches U15.5
- net at U15.6: now also U14.1
- net at U7.9: now also U2.9 (S0)
- net at U19.6: now also U26.5
- net at U2.13 (E3): now also U58.8
- net at U2.7 (S1): now also U7.11; no longer U16.11
- net at U16.9: no longer U2.9 (S0)
- net at U3.3: now also U27.8
- net at U7.13: now also U2.6 (S2)
- net at U8.3: now also U20.4 (Za)
- net at U22.9: now also U29.7 (Zb)
- net at U10.3, U20.5 (I0b): now also U34.3
- net at U79.5 (Q1): now also U58.10
- net at U7.2: now also Q1.3 (B), RN1.6 (R5)
- net at U10.6: now also U29.15 (E)
- net at U22.13: now also U29.4 (Za)
- net BRIDGE AP: now reaches U5.1 (S)
- net ~{BRIDGE (Y)}: now reaches U5.10 (I1c)
- net at U5.12 (Zd): now also U27.3
- net ~{BRIDGE (W)}: now reaches U5.13 (I1d)
- net ~{SIDE LINE}: now reaches U5.14 (I0d)
- net at U5.4 (Za): now also U14.2
- net ~{BRIDGE Bu}: now reaches U5.6 (I1b)
- net EXTEND: now reaches U20.1 (S)
- net EXTEND: now also U34.2
- net at U20.10 (I1c): now also U14.6
- net at U20.7 (Zb): now also U27.6
- net at U3.13: now also U34.1
- net at U3.1: now also U26.6
- net ~{RESCUE}: now reaches U22.10
- net ~{RESCUE}: now also U27.2
- net at U22.11: now also U29.12 (Zd)
- net ~{OTHER BODY}: now reaches U86.1 (OEa), U86.15 (OEb)
- net AREA 4: now reaches U86.10 (I4)
- net AREA 5: now reaches U86.12 (I5)
- net AREA 1: now reaches U86.2 (I1)
- net AREA 2: now reaches U86.4 (I2)
- net AREA 3: now reaches U86.6 (I3)
- new net: U201.12 (MR), U201.2 (MR)
- new net: U201.13 (CP), U201.6 (Q3)
- new net: U57.11 (K), U57.4 (K)
- new net: U40.12 (D), U41.1 (I3), U41.13 (I6), U41.14 (I5), U41.15 (I4), U41.2 (I2), U41.3 (I1)
- new net: U40.11 (C), U41.12 (I7)
- new net: U25.2 (D), U25.9 (Q)
- new net: U29.3 (I1a), U30.10 (D1)
- new net: U29.5 (I0b), U30.11 (D2)
- new net: U29.6 (I1b), U30.13 (D3)
- new net: U29.11 (I0c), U30.14 (D4)
- new net: U29.10 (I1c), U30.15 (D5)
- new net: U29.14 (I0d), U30.16 (D6)
- new net: U29.13 (I1d), U30.17 (D7)
- new net: U29.2 (I0a), U30.9 (D0)
- new net: U44.12, U45.12
- new net: U33.11, U45.11
- new net DUMMY: U33.2
- new net EXPLO: U33.5
- new net PLAYER BODY: U33.6
- new net RESCUE: U33.1
- new net ~{BRIDGE}: U44.1
- new net ~{DUMMY}: U26.2, U27.1, U66.1
- new net ~{EXPLO. AREA}: U66.13
- new net ~{HOUSE}: U27.12, U44.13, U58.9
- new net ~{OTHER TIRE}: U27.11
- new net ~{PLAYER TIRE}: U27.5
- new net ~{PLAYER}: U26.4, U66.2
- new net ~{SIG}: U26.1
- new net ~{WALL}: U44.2
- now unconnected: U7.4
- no-connect marks 6 -> 7
Other:
- moved on the sheet: U10B, U10D, U15B, U16D, U16E, U16F, U22A, U22D, U22E, U22F, U3E, U7A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

Commit message: video
Parts:
- removed U16: 74LS07, Package_DIP:DIP-14_W7.62mm, symbol 74xx:74LS07
- added C1, C2: 470p, Capacitor_THT:C_Disc_D3.0mm_W1.6mm_P2.50mm, symbol Device:C_Polarized_US
- added C16: 100p, Capacitor_THT:C_Disc_D4.3mm_W1.9mm_P5.00mm, symbol Device:C
- added C17: 0,1u, Capacitor_THT:C_Disc_D7.5mm_W5.0mm_P7.50mm, symbol Device:C
- added Cp1, Cp10, Cp11, Cp12, Cp13, Cp14, Cp15, Cp16, Cp17, Cp18, Cp2, Cp3, Cp4, Cp5, Cp6, Cp7, Cp8, Cp9: C, Capacitor_THT:C_Disc_D7.5mm_W5.0mm_P7.50mm, symbol Device:C
- added Cp19, Cp20, Cp21, Cp22, Cp23, Cp24, Cp25, Cp26, Cp27, Cp28, Cp29, Cp30, Cp31, Cp32, Cp33, Cp34, Cp35, Cp36: C, Capacitor_THT:C_Disc_D7.5mm_W5.0mm_P10.00mm, symbol Device:C
- added J1, J2: Conn_02x22_Top_Bottom, BoardEdge:EdgeD, symbol Connector_Generic:Conn_02x22_Top_Bottom
- added R17, R18: 330, Resistor_THT:R_Axial_DIN0309_L9.0mm_D3.2mm_P12.70mm_Horizontal, symbol Device:R
- added U100, U102, U103, U107, U108, U118, U76, U77, U85, U91: 74LS161, Package_DIP:DIP-16_W7.62mm, symbol 74xx:74LS161
- added U101, U71, U78, U90: 74LS20, Package_DIP:DIP-14_W7.62mm, symbol 74xx:74LS20
- added U104, U70: 74LS32, Package_DIP:DIP-14_W7.62mm, symbol 74xx:74LS32
- added U105, U112, U119: 74LS153, Package_DIP:DIP-16_W7.62mm, symbol 74xx:74LS153
- added U106, U113, U120, U64, U99: MB7137, Package_DIP:DIP-24_W15.24mm, symbol Memory_PROM:MB7137
- added U109, U116: 74LS107, Package_DIP:DIP-14_W7.62mm, symbol 74xx:74LS107
- added U110, U16, U72, U81: 74LS00, Package_DIP:DIP-14_W7.62mm, symbol 74xx:74LS00
- added U111, U67, U83, U84, U92, U98: 74LS157, Package_DIP:DIP-16_W7.62mm, symbol 74xx:74LS157
- added U114, U117, U59, U62, U82, U93: 74LS06, Package_DIP:DIP-14_W7.62mm, symbol 74xx:74LS06
- added U115, U75, U94: 74LS10, Package_DIP:DIP-14_W7.62mm, symbol 74xx:74LS10
- added U60, U61, U73, U89: 74LS27, Package_DIP:DIP-14_W7.62mm, symbol 74xx:74LS27
- added U63: 74LS151, Package_DIP:DIP-16_W7.62mm, symbol 74xx:74LS151
- added U65, U80: 74LS02, Package_DIP:DIP-14_W7.62mm, symbol 74xx:74LS02
- added U68: 74LS279, Package_DIP:DIP-16_W7.62mm, symbol 74xxMissing:74LS279
- added U69, U74, U88: 74LS74, Package_DIP:DIP-14_W7.62mm, symbol 74xx:74LS74
- added U87, U95: 74LS08, Package_DIP:DIP-14_W7.62mm, symbol 74xx:74LS08
- added U96, U97: 74LS42, Package_DIP:DIP-16_W7.62mm, symbol 74xx:74LS42
- added Y1: 14,305, Crystal:Crystal_HC18-U_Horizontal_1EP_style2, symbol Device:Crystal_GND3
Connections:
- net BRIDGE AP: now also U58.5, U16.10
- net D10: now also J1.10 (Pin_10)
- net D11: now also J1.11 (Pin_11)
- net D12: now also J1.12 (Pin_12)
- net D13: now also J1.13 (Pin_13)
- net GNDPWR: now also U12.20 (~{CE}1_(PVCE)), U12.21 (A10), U201.7 (GND), U202.8 (GND), U32.7 (GND), U33.7 (GND), U34.7 (GND), U35.7 (GND), U36.8 (GND), U37.8 (GND), U38.7 (GND), U39.7 (GND), U40.7 (GND), U41.8 (GND), U42.7 (GND), U43.8 (GND), U44.7 (GND), U45.7 (GND), U46.8 (GND), U47.7 (GND), U48.8 (GND), U49.7 (GND), U50.15 (E), U50.8 (GND), U51.20 (~{CE}1_(PVCE)), U51.21 (A10), U52.7 (GND), U53.8 (GND), U54.12 (A3), U54.8 (GND), U55.7 (GND), U56.7 (GND), U57.7 (GND), U58.7 (GND), U6.8 (GND), U66.7 (GND), U9.7 (GND), C1.2, C2.2, Cp1.1, Cp10.1, Cp11.1, Cp12.1, Cp13.1, Cp14.1, Cp15.1, Cp16.1, Cp17.1, Cp18.1, Cp19.1, Cp2.1, Cp20.1, Cp21.1, Cp22.1, Cp23.1, Cp24.1, Cp25.1, Cp26.1, Cp27.1, Cp28.1, Cp29.1, Cp3.1, Cp30.1, Cp31.1, Cp32.1, Cp33.1, Cp34.1, Cp35.1, Cp36.1, Cp4.1, Cp5.1, Cp6.1, Cp7.1, Cp8.1, Cp9.1, J1.1 (Pin_1), J1.2 (Pin_2), J1.3 (Pin_3), J1.4 (Pin_4), J1.5 (Pin_5), U100.8 (GND), U101.7 (GND), U102.8 (GND), U103.8 (GND), U104.7 (GND), U105.8 (GND), U106.12 (GND), U107.8 (GND), U108.8 (GND), U109.7 (GND), U110.7 (GND), U111.8 (GND), U112.8 (GND), U113.12 (GND), U114.7 (GND), U115.7 (GND), U116.7 (GND), U117.7 (GND), U118.8 (GND), U119.8 (GND), U120.12 (GND), U120.20 (~{CE}1_(PVCE)), U16.7 (GND), U59.7 (GND), U60.7 (GND), U61.7 (GND), U62.7 (GND), U63.8 (GND), U64.12 (GND), U64.20 (~{CE}1_(PVCE)), U64.21 (A10), U65.7 (GND), U67.15 (E), U67.8 (GND), U68.8 (GND), U69.7 (GND), U70.7 (GND), U71.7 (GND), U72.7 (GND), U73.7 (GND), U74.7 (GND), U75.7 (GND), U76.3 (D0), U76.4 (D1), U76.5 (D2), U76.6 (D3), U76.8 (GND), U77.3 (D0), U77.4 (D1), U77.5 (D2), U77.6 (D3), U77.8 (GND), U78.7 (GND), U80.7 (GND), U81.7 (GND), U82.7 (GND), U83.10 (I1c), U83.15 (E), U83.3 (I1a), U83.6 (I1b), U83.8 (GND), U84.10 (I1c), U84.15 (E), U84.6 (I1b), U84.8 (GND), U85.8 (GND), U87.7 (GND), U88.7 (GND), U89.7 (GND), U90.7 (GND), U91.8 (GND), U92.15 (E), U92.8 (GND), U93.7 (GND), U94.7 (GND), U95.7 (GND), U96.8 (GND), U97.12 (A3), U97.8 (GND), U98.8 (GND), U99.12 (GND), Y1.3
- net VCC: now also U17.19 (CE3), U26.14 (VCC), U36.1 (~{MR}), U36.10 (CET), U36.7 (CEP), U43.13 (I1d), U43.14 (I0d), U43.5 (I0b), U45.14 (VCC), U46.16 (VCC), U48.13 (I6), U48.14 (I5), U48.15 (I4), U48.2 (I2), U49.14 (VCC), U50.16 (VCC), U51.18 (CE2), U51.19 (CE3), U52.14 (VCC), U53.16 (VCC), U53.3 (I3a), U54.16 (VCC), U55.14 (VCC), U56.14 (VCC), U57.1 (J), U57.13 (~{R}), U57.14 (VCC), U57.4 (K), U58.14 (VCC), U66.14 (VCC), Cp1.2, Cp10.2, Cp11.2, Cp12.2, Cp13.2, Cp14.2, Cp15.2, Cp16.2, Cp17.2, Cp18.2, Cp19.2, Cp2.2, Cp20.2, Cp21.2, Cp22.2, Cp23.2, Cp24.2, Cp25.2, Cp26.2, Cp27.2, Cp28.2, Cp29.2, Cp3.2, Cp30.2, Cp31.2, Cp32.2, Cp33.2, Cp34.2, Cp35.2, Cp36.2, Cp4.2, Cp5.2, Cp6.2, Cp7.2, Cp8.2, Cp9.2, J1.19 (Pin_19), J1.20 (Pin_20), J1.21 (Pin_21), J1.22 (Pin_22), U100.16 (VCC), U101.14 (VCC), U102.16 (VCC), U103.16 (VCC), U104.14 (VCC), U105.16 (VCC), U106.19 (CE3), U106.24 (VCC_(PVCC)), U107.16 (VCC), U108.16 (VCC), U109.10 (~{R}), U109.11 (K), U109.14 (VCC), U109.8 (J), U110.14 (VCC), U111.16 (VCC), U112.16 (VCC), U113.24 (VCC_(PVCC)), U114.14 (VCC), U115.14 (VCC), U116.14 (VCC), U117.14 (VCC), U118.16 (VCC), U119.16 (VCC), U120.18 (CE2), U120.24 (VCC_(PVCC)), U16.14 (VCC), U59.14 (VCC), U60.14 (VCC), U61.14 (VCC), U62.14 (VCC), U63.16 (VCC), U64.18 (CE2), U64.19 (CE3), U64.24 (VCC_(PVCC)), U65.14 (VCC), U67.16 (VCC), U68.16 (VCC), U69.14 (VCC), U70.14 (VCC), U71.14 (VCC), U72.14 (VCC), U73.14 (VCC), U74.14 (VCC), U75.14 (VCC), U76.1 (~{MR}), U76.16 (VCC), U76.7 (CEP), U77.1 (~{MR}), U77.16 (VCC), U77.7 (CEP), U78.14 (VCC), U80.14 (VCC), U81.14 (VCC), U82.14 (VCC), U83.16 (VCC), U83.2 (I0a), U84.13 (I1d), U84.16 (VCC), U84.2 (I0a), U85.1 (~{MR}), U85.16 (VCC), U85.7 (CEP), U87.14 (VCC), U88.14 (VCC), U89.14 (VCC), U90.14 (VCC), U91.1 (~{MR}), U91.16 (VCC), U91.7 (CEP), U92.16 (VCC), U93.14 (VCC), U94.14 (VCC), U95.1, U95.14 (VCC), U96.16 (VCC), U97.16 (VCC), U98.16 (VCC), U99.19 (CE3), U99.24 (VCC_(PVCC))
- net ~{GRAVEL}: now also U72.11
- net ~{OTHER CAR}: now also U21.13
- net ~{WALL}: now also U72.3
- net V7: now reaches U54.13 (A2)
- net V6: now reaches U54.14 (A1)
- net V6: now also U28.4, U64.3 (A5)
- net V5: now reaches U54.15 (A0)
- net V5: now also U64.4 (A4)
- net at U54.2 (1): now also U61.13
- net at U54.3 (2): now also U61.3, U68.15 (~{S})
- net at U54.6 (5): now also U70.2
- net at U54.7 (6): now also U68.14 (~{R})
- net at U54.9 (7): now also U61.9
- net SIG: now reaches U9.12
- net SIG: now also U4.12, U9.3
- net at U9.13: now also U66.8, U9.2
- net at U48.10 (S1): now also U39.11, U41.10 (S1)
- net at U48.11 (S0): now also U41.11 (S0), U49.11 (Q0)
- net at U48.12 (I7): now also U40.12 (D), U41.1 (I3), U41.13 (I6), U41.14 (I5), U41.15 (I4), U41.2 (I2), U41.3 (I1), U48.4 (I0)
- net at U48.9 (S2): now also U41.9 (S2), U47.13, U49.8 (Q3)
- net MH3: now reaches U12.1 (A7), U17.1 (A7)
- net MH2: now reaches U12.2 (A6), U17.2 (A6)
- net MH4: now reaches U12.23 (A8), U17.23 (A8)
- net MH1: now reaches U12.3 (A5), U17.3 (A5)
- net at U66.10: now also U59.8
- net at U66.11: now also U65.1
- net at U57.11 (K): no longer U57.4 (K)
- net S-100-C: now reaches RN1.4 (R3)
- net S-100-C: now also U24.12 (A3)
- net V-4: now reaches U22.1
- net V-4: now also U21.1
- net at U24.1 (0): now also U40.3 (C)
- net S-100-D: now reaches U24.13 (A2)
- net S-100-B: now reaches U24.14 (A1)
- net S-100-A: now reaches U24.15 (A0)
- net at U24.2 (1): now also U47.4
- net at U24.3 (2): now also U31.3 (C)
- net at U24.5 (4): now also U25.11 (C)
- net at U24.7 (6): now also U47.5
- net at U24.9 (7): now also U31.11 (C)
- net at U55.10: now also U57.12 (C)
- net at U55.11: now also U57.3 (Q)
- net V1: now reaches U23.4
- net V1: now also U30.7 (A1), U51.7 (A1), U64.8 (A0)
- net at U23.12, U23.2, U23.5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: now also U28.1, U28.5
- net at U55.1: now also U56.6
- net at U55.13: now also U56.8
- net at U55.2: now also U52.10, U59.4
- net ~{BRIDGE AP}: now reaches U58.1
- net ~{M.ROAD}: now reaches U58.2
- net at U58.3: now also U65.5
- net MH0: now reaches U11.1 (S)
- net at U11.4 (Za): now also U15.10, U6.15 (A0)
- net at U11.7 (Zb): now also U6.14 (A1)
- net at U11.9 (Zc): now also U6.13 (A2)
- net V4: now reaches U28.2
- net V4: now also U51.4 (A4), U61.1, U64.5 (A3), U73.8
- net at U28.3: now also U21.11
- net at U25.9 (Q): no longer U25.2 (D)
- net at U31.1 (~{R}): now also U31.13 (~{R}), U34.10
- net at U31.2 (D): now also U38.6 (~{Q}), U89.4
- net at U31.5 (Q): now also U32.5
- net at U31.6 (~{Q}): now also U31.12 (D)
- net at U21.12: now also U16.9
- net ~{DUMMY AREA}: now reaches U21.2
- net ~{DUMMY AREA}: now also U26.8, U59.3
- net V3: now reaches U30.5 (A3)
- net V3: now also U23.1, U51.5 (A3), U64.6 (A2)
- net V2: now reaches U30.6 (A2)
- net V2: now also U23.13, U51.6 (A2), U64.7 (A1)
- net V0: now reaches U30.8 (A0)
- net V0: now also U23.10, U51.8 (A0)
- net at U58.6: now also U65.6
- net at U31.9 (Q): now also U32.2, U34.6
- net at U6.12 (A3): now also U16.8
- net at U37.4 (D1): now also U37.7 (CEP)
- net V-2: now reaches U21.10
- net at U21.9: now also U28.6
- net at U34.8: now also U47.11
- net ~{COIN IN}: now reaches U34.9
- net ~{COIN IN}: now also C1.1, U64.23 (A8)
- net at U56.3: now also U56.12
- net at U47.12: now also U39.13, U49.9 (Q2)
- net at U43.15 (E): now also U43.2 (I0a)
- net H3: now reaches U51.1 (A7)
- net H3: now also U64.2 (A6)
- net at U51.10 (D1): now also U50.3 (I1a)
- net at U51.11 (D2): now also U50.5 (I0b)
- net at U51.13 (D3): now also U50.6 (I1b)
- net at U51.14 (D4): now also U50.11 (I0c)
- net at U51.15 (D5): now also U50.10 (I1c)
- net at U51.16 (D6): now also U50.14 (I0d)
- net at U51.17 (D7): now also U50.13 (I1d)
- net H2: now reaches U51.2 (A6)
- net H2: now also U63.9 (S2)
- net H4: now reaches U51.23 (A8)
- net H4: now also U71.1
- net H1: now reaches U51.3 (A5)
- net H1: now also U63.10 (S1)
- net at U51.9 (D0): now also U50.2 (I0a)
- net at U40.5 (Q): now also U32.1
- net at U38.11 (C): now also U47.6
- net at U38.13 (~{R}): now also U45.3
- net at U38.9 (Q): now also U38.2 (D)
- net at U52.4: now also U55.6, U70.9
- net at U52.5: now also U70.13, U71.8
- net at U52.6: now also U70.5
- net at U9.1: now also U50.12 (Zd)
- net at U38.5 (Q): now also U45.2
- net ~{GAME}: now reaches U55.3
- net ~{GAME}: now also U73.10
- net H8: now reaches U55.4
- net H8: now also U64.1 (A7)
- net ~{H5}: now reaches U55.5
- net at U49.10 (Q1): now also U39.12
- net at U49.12 (MR): now also U32.6
- net at U49.13 (CP): now also U40.8 (~{Q}), U45.1, C2.1
- net at U15.8: now also U16.13, U16.2
- net H6: now reaches U42.1
- net H6: now also U71.4
- net at U42.12: now also U73.11
- net ~{H8}: now reaches U42.13
- net ~{H8}: now also U71.9
- net H5: now reaches U42.2
- net H5: now also U71.12
- net at U58.13: now also U72.13, U72.2
- net at U56.4: now also U52.8, U56.10
- net at U56.5: now also U50.7 (Zb)
- net Vs/16: now reaches U52.9
- net Vs/16: now also U71.10, U73.9
- net ~{TUNNEL}: now reaches U34.4
- net at U34.5: now also U32.4
- net at U56.9: now also U50.4 (Za)
- net H9: now reaches U50.1 (S)
- new net: U70.4, U71.6
- new net: U63.7 (~{E}), U70.6
- new net: U71.13, U72.6
- new net: C16.1, Y1.2
- new net: C16.2, R18.2, U117.10
- new net: U62.12, U69.1 (~{R})
- new net: U69.4 (~{S}), U70.3
- new net: U69.5 (Q), U84.11 (I0c), U84.5 (I0b)
- new net: U69.6 (~{Q}), U84.14 (I0d)
- new net: U88.6 (~{Q}), U89.3
- new net: U75.8, U89.5
- new net: U89.6, U89.9
- new net: U76.10 (CET), U85.15 (TC)
- new net: U83.4 (Za), U85.3 (D0)
- new net: U83.7 (Zb), U85.4 (D1)
- new net: U83.9 (Zc), U85.5 (D2)
- new net: U83.12 (Zd), U85.6 (D3)
- new net: U61.11, U62.8, U70.1
- new net: U62.9, U77.15 (TC)
- new net: U98.10 (I1c), U99.15 (D5)
- new net: U98.11 (I0c), U99.14 (D4)
- new net: U98.13 (I1d), U99.17 (D7)
- new net: U98.14 (I0d), U99.16 (D6)
- new net: U98.2 (I0a), U99.9 (D0)
- new net: U98.3 (I1a), U99.10 (D1)
- new net: U97.15 (A0), U98.4 (Za)
- new net: U98.5 (I0b), U99.11 (D2)
- new net: U98.6 (I1b), U99.13 (D3)
- new net: U97.14 (A1), U98.7 (Zb)
- new net: U97.13 (A2), U98.9 (Zc)
- new net: U62.10, U69.10 (~{S})
- new net: U61.12, U62.11
- new net: U61.8, U62.13
- new net: U88.1 (~{R}), U95.11
- new net: U67.1 (S), U92.1 (S)
- new net: U62.2, U69.13 (~{R})
- new net: U69.8 (~{Q}), U83.14 (I0d)
- new net: U69.9 (Q), U83.11 (I0c), U83.5 (I0b)
- new net: U105.10 (I0b), U106.14 (D4)
- new net: U105.11 (I1b), U106.15 (D5)
- new net: U105.12 (I2b), U106.16 (D6)
- new net: U105.13 (I3b), U106.17 (D7)
- new net: U105.3 (I3a), U106.13 (D3)
- new net: U105.4 (I2a), U106.11 (D2)
- new net: U105.5 (I1a), U106.10 (D1)
- new net: U105.6 (I0a), U106.9 (D0)
- new net: U95.4, U96.6 (5)
- new net: U95.5, U96.7 (6)
- new net: U77.10 (CET), U91.15 (TC)
- new net: U61.6, U62.1
- new net: U112.5 (I1a), U113.10 (D1)
- new net: U112.4 (I2a), U113.11 (D2)
- new net: U112.3 (I3a), U113.13 (D3)
- new net: U112.10 (I0b), U113.14 (D4)
- new net: U112.11 (I1b), U113.15 (D5)
- new net: U112.12 (I2b), U113.16 (D6)
- new net: U112.13 (I3b), U113.17 (D7)
- new net: U112.6 (I0a), U113.9 (D0)
- new net: U109.9 (C), U117.12
- new net: C17.1, R17.2, U117.13, U117.8
- new net: C17.2, R18.1, U117.11
- new net: U68.13 (Q), U71.5
- new net: U62.3, U76.15 (TC)
- new net: U63.1 (I3), U64.13 (D3)
- new net: U63.12 (I7), U64.17 (D7)
- new net: U63.13 (I6), U64.16 (D6)
- new net: U63.14 (I5), U64.15 (D5)
- new net: U63.15 (I4), U64.14 (D4)
- new net: U63.2 (I2), U64.11 (D2)
- new net: U63.3 (I1), U64.10 (D1)
- new net: U63.4 (I0), U64.9 (D0)
- new net: U63.6 (~{Z}), U70.10, U70.12
- new net: U119.10 (I0b), U120.14 (D4)
- new net: U119.11 (I1b), U120.15 (D5)
- new net: U119.12 (I2b), U120.16 (D6)
- new net: U119.13 (I3b), U120.17 (D7)
- new net: U119.3 (I3a), U120.13 (D3)
- new net: U119.4 (I2a), U120.11 (D2)
- new net: U119.5 (I1a), U120.10 (D1)
- new net: U119.6 (I0a), U120.9 (D0)
- new net: U84.4 (Za), U91.3 (D0)
- new net: U84.7 (Zb), U91.4 (D1)
- new net: U84.9 (Zc), U91.5 (D2)
- new net: U84.12 (Zd), U91.6 (D3)
- new net: U109.5 (Q), U117.5
- new net: R17.1, U117.9, Y1.1
- new net: U75.11, U82.4
- new net COIN IN: U72.5
- new net D14: J1.14 (Pin_14)
- new net D15: J1.15 (Pin_15)
- new net D16: J1.16 (Pin_16)
- new net D17: J1.17 (Pin_17)
- new net D18: J1.18 (Pin_18)
- new net D6: J1.6 (Pin_6)
- new net D7: J1.7 (Pin_7)
- new net D8: J1.8 (Pin_8)
- new net D9: J1.9 (Pin_9)
- new net H0: U63.11 (S0)
- new net H7: U71.2
- new net M1V0: U85.14 (Q0), U92.2 (I0a)
- new net M1V1: U85.13 (Q1), U92.5 (I0b)
- new net M1V2: U85.12 (Q2), U92.11 (I0c)
- new net M1V3: U85.11 (Q3), U92.14 (I0d)
- new net M1V4: U67.2 (I0a), U76.14 (Q0)
- new net M1V5: U76.13 (Q1)
- new net M1V6: U76.12 (Q2)
- new net M1V7: U76.11 (Q3)
- new net M2V0: U91.14 (Q0), U92.3 (I1a)
- new net M2V1: U91.13 (Q1), U92.6 (I1b)
- new net M2V2: U91.12 (Q2), U92.10 (I1c)
- new net M2V3: U91.11 (Q3), U92.13 (I1d)
- new net M2V4: U67.3 (I1a), U77.14 (Q0)
- new net M2V5: U75.9, U77.13 (Q1)
- new net M2V6: U77.12 (Q2), U82.3
- new net M2V7: U75.10, U77.11 (Q3)
- new net MH5: U88.3 (C)
- new net MH6: U88.2 (D)
- new net MH7: U95.13
- new net MH8: U95.12
- new net ~{CAR NO CONT}: U59.9
- new net ~{EX.SIGNAL}: U72.4
- new net ~{EXT.500}: U65.2
- new net ~{Hs}: U76.2 (CP), U77.2 (CP), U85.2 (CP), U91.2 (CP)
- new net ~{M1VL0}: U61.2, U61.4, U62.4, U76.9 (~{PE}), U85.9 (~{PE})
- new net ~{M2VL0}: U77.9 (~{PE}), U91.9 (~{PE})
- new net ~{POOL}: U72.8
- new net ~{SLIDE}: U65.4
- new net ~{V4}: U61.10, U61.5
- new net ~{Vb}: U85.10 (CET), U91.10 (CET)
- no-connect marks 7 -> 27
Other:
- moved on the sheet: U10D, U11, U12, U15C, U17, U21A, U21C, U22A, U22C, U23A, U23B, U23C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

Commit message: video board all chips
Parts:
- added C10, C22, C25, C6, C7: 470p, Capacitor_THT:C_Disc_D3.0mm_W1.6mm_P2.50mm, symbol Device:C
- added R16: 47k, Resistor_THT:R_Axial_DIN0309_L9.0mm_D3.2mm_P12.70mm_Horizontal, symbol Device:R_US
- added U206: 74LS74, Package_DIP:DIP-14_W7.62mm, symbol 74xx:74LS74
- C24: renamed from C2; footprint Capacitor_THT:C_Disc_D3.0mm_W1.6mm_P2.50mm -> Capacitor_THT:C_Disc_D4.3mm_W1.9mm_P5.00mm
- renumbered C1 to C20
Connections:
- net H9 is gone; now on net H0: U50.1 (S)
- net PLAYER BODY is gone; now on net E7: U33.6
- net ROAD is gone; now on net E7: U5.2 (I0a), U5.5 (I0b)
- net ~{PLAYER} is gone; now on net E9: U26.4, U66.2
- net BRIDGE AP: now also U22.5, U80.1, U80.6
- net D10: now also RN1.2 (R1); no longer RN1.9 (R8)
- net E10: now also J2.10 (Pin_10)
- net EXTEND: now also U25.12 (D), U26.12, U40.2 (D)
- net GNDPWR: now also J1.23 (Pin_23), J1.24 (Pin_24), J1.25 (Pin_25), J1.26 (Pin_26), J1.27 (Pin_27), U101.2, U102.5 (D2), U103.5 (D2), U108.5 (D2), U111.15 (E), U111.3 (I1a), U111.6 (I1b), U118.3 (D0), U120.21 (A10), U30.20 (~{CE}1_(PVCE)), U37.6 (D3), U43.11 (I0c), U43.3 (I1a), U43.6 (I1b), U53.10 (I0b), U84.3 (I1a), C10.2, C22.2, C25.2, C6.2, C7.2, U206.7 (GND)
- net M1V0: now also U78.1
- net M1V1: now also U78.2
- net M1V2: now also U90.13
- net M1V3: now also U78.5
- net M1V4: now also U78.4
- net M1V5: now also U90.12
- net M1V6: now also U90.10
- net M1V7: now also U90.9
- net M2V0: now also U90.2
- net M2V1: now also U90.1
- net M2V2: now also U117.3
- net M2V4: now also U90.5
- net M2V5: now also U78.9, U82.5
- net M2V6: now also U75.3, U78.10
- net M2V7: now also U75.4, U78.12
- net MH0: now also U105.14 (S0), U112.14 (S0), U118.14 (Q0), U119.14 (S0), U98.1 (S)
- net MH1: now also U105.2 (S1), U112.2 (S1), U118.13 (Q1), U119.2 (S1), U99.3 (A5)
- net MH2: now also U106.3 (A5), U113.3 (A5), U118.12 (Q2), U120.3 (A5), U99.2 (A6)
- net MH3: now also U106.2 (A6), U113.2 (A6), U118.11 (Q3), U120.2 (A6), U99.1 (A7)
- net MH4: now also U103.14 (Q0), U104.9, U106.1 (A7), U113.1 (A7), U120.1 (A7), U99.23 (A8)
- net MH5: now also U103.13 (Q1), U89.1, U96.15 (A0)
- net MH6: now also U103.12 (Q2), U89.2, U96.14 (A1)
- net MH7: now also U103.11 (Q3), U89.13, U96.13 (A2)
- net MH8: now also U104.13, U110.10
- net S-100-A: now also RN1.9 (R8), U202.4 (Za)
- net S-100-B: now also RN1.8 (R7), U202.7 (Zb)
- net S-100-C: now also U202.12 (Zd); no longer RN1.4 (R3)
- net S-100-D: now also RN1.4 (R3), U202.9 (Zc)
- net TUNNEL AP: now also U80.13, U80.5, U87.5
- net V7: now also U104.1
- net VCC: now also U100.1 (~{MR}), U102.1 (~{MR}), U102.10 (CET), U102.7 (CEP), U103.1 (~{MR}), U103.4 (D1), U103.7 (CEP), U107.1 (~{MR}), U107.10 (CET), U107.6 (D3), U108.1 (~{MR}), U108.10 (CET), U108.7 (CEP), U109.1 (J), U109.13 (~{R}), U109.4 (K), U111.13 (I1d), U118.1 (~{MR}), U18.10 (B), U18.11 (Clr), U37.1 (~{MR}), U37.3 (D0), U57.10 (~{R}), U57.11 (K), U57.8 (J), U83.13 (I1d), R16.2, U206.14 (VCC)
- net ~{BRIDGE AP}: now also U22.6
- net ~{COIN & START}: now also U70.8
- net ~{DUMMY AREA}: no longer U26.8, U59.3
- net ~{DUMMY}: now also U26.8, U55.12, U59.3
- net ~{EXT.500}: now also U25.2 (D), U25.9 (Q)
- net ~{EXTEND}: now also U49.2 (MR)
- net ~{HOUSE}: now also U14.13
- net ~{Hs}: now also U35.2 (D), U47.2
- net ~{M1VL0}: now also U67.5 (I0b), U74.3 (C)
- net ~{M2VL0}: now also U61.11, U62.8, U67.6 (I1b), U70.1, U74.1 (~{R}), C10.1
- net ~{POOL}: now also U14.12
- net ~{ROAD}: now also U74.6 (~{Q}), U87.10, U87.4
- net ~{TUNNEL}: now also U31.8 (~{Q}), U38.12 (D), U80.11
- net ~{V4}: now also U60.13
- net ~{Vb}: now also U74.2 (D), U88.12 (D)
- net at U54.7 (6), U68.14 (~{R}): now also C22.1
- net V-CA: now reaches U42.3
- net Vb: now reaches U42.4
- net at U42.5: now also U35.5 (Q)
- net at U42.6: now also U43.1 (S)
- net at U80.4: now also U87.9, U94.5, U94.9
- net at U103.10 (CET): now also U118.15 (TC), U55.9
- net at U103.15 (TC): now also U55.10, U57.12 (C), C25.1
- net 7M: now reaches U103.2 (CP)
- net 7M: now also U118.2 (CP), U14.4, U79.9 (Cp)
- net at U103.3 (D0): now also U111.12 (Zd)
- net at U82.10: now also U66.4
- net at U82.11: now also U89.12
- net at U68.5 (~{R}): now also U41.5 (Z)
- net at U68.6 (~{S}): now also U48.5 (Z)
- net at U111.11 (I0c): now also U110.13
- net at U111.14 (I0d): now also U110.12
- net at U111.4 (Za): now also U118.4 (D1)
- net at U111.7 (Zb): now also U118.5 (D2)
- net at U111.9 (Zc): now also U118.6 (D3)
- net M2V8: now reaches U78.13
- net at U78.8: now also U82.1
- net at U81.12: now also U90.8
- net at U81.13: now also U82.12
- net at U47.3: now also U40.12 (D), U41.1 (I3), U41.13 (I6), U41.14 (I5), U41.15 (I4), U41.2 (I2), U41.3 (I1), U48.12 (I7), U48.4 (I0)
- net at U89.6, U89.9: now also U72.10
- net EX: now reaches U42.10
- net EX: now also U49.4 (Q1)
- net at U42.11: now also U49.3 (Q0)
- net at U42.8: now also U35.4 (~{S}), C6.1
- net at U42.9: now also U35.8 (~{Q})
- net at U94.10: now also U88.8 (~{Q})
- net E7: now reaches U94.11
- net E7: now also J2.7 (Pin_7), U74.5 (Q)
- net at U94.8: now also U80.8
- net at U57.5 (Q): now also U44.11, U44.3
- net at U57.9 (C): now also U37.15 (TC), U44.10
- net at U110.11: now also U95.10
- net at U116.10 (~{R}): now also U116.8 (J)
- net at U116.11 (K): now also U116.3 (Q)
- net at U55.8: now also U118.9 (~{PE})
- net at U13.12: now also U19.10, U21.6
- net at U117.4: now also U90.4
- net at U88.9 (Q): now also U104.2, U96.12 (A3)
- net at U104.11: now also U56.2
- net at U104.12: now also U95.6
- net at U35.10 (~{S}): now also U49.5 (Q2)
- net at U35.11 (C): now also U47.8
- net 100-C: now reaches U35.12 (D)
- net at U35.9 (Q): now also U18.9 (A)
- net at U67.1 (S), U92.1 (S): now also U104.3
- net at U92.12 (Zd): now also U106.5 (A3), U113.5 (A3), U120.5 (A3), U99.5 (A3)
- net at U92.4 (Za): now also U106.8 (A0), U113.8 (A0), U120.8 (A0), U99.8 (A0)
- net at U92.7 (Zb): now also U106.7 (A1), U113.7 (A1), U120.7 (A1), U99.7 (A1)
- net at U92.9 (Zc): now also U106.6 (A2), U113.6 (A2), U120.6 (A2), U99.6 (A2)
- net at U72.1: now also U117.1, U87.6, U89.10
- net at U58.13, U72.13, U72.2: now also U119.7 (Za), U119.9 (Zb), U58.11, U60.11, U72.9
- net at U65.11: now also U81.9, U82.8
- net at U65.12: now also U56.12, U56.3
- net at U65.13: now also U81.4
- net at U75.5: now also U82.6
- net at U75.6: now also U66.3
- net at U82.2: now also U81.1
- net ~{RESCUE(W)}: now reaches U22.8
- net at U60.1: now also U35.6 (~{Q})
- net at U60.12: now also U59.11
- net E18: now reaches U16.4
- net E18: now also J2.18 (Pin_18)
- net at U16.5: now also U29.9 (Zc)
- net ~{RESCUE(R)}: now reaches U16.6
- net at U82.9: now also U94.3, U96.1 (0)
- net at U25.13 (~{R}): now also U38.13 (~{R}), U45.3
- net EXT.500: now reaches U25.8 (~{Q})
- net at U31.1 (~{R}), U31.13 (~{R}), U34.10: now also U25.1 (~{R}), U40.1 (~{R})
- net at U60.10: now also U105.7 (Za)
- net at U60.9: now also U112.9 (Zb)
- net at U46.1 (B): now also U46.15 (A)
- net at U59.10: now also U10.4
- net at U19.13: now also U20.9 (Zc)
- net at U30.1 (A7): now also U37.13 (Q1)
- net at U30.18 (CE2): now also U37.4 (D1), U37.7 (CEP)
- net at U30.2 (A6): now also U37.14 (Q0)
- net at U30.3 (A5): now also U36.11 (Q3)
- net at U30.4 (A4): now also U36.12 (Q2)
- net at U99.4 (A4): now also U106.4 (A4), U113.4 (A4), U120.4 (A4), U67.4 (Za)
- net at U105.1 (Ea): now also U105.15 (Eb), U56.11
- net at U105.9 (Zb): now also U22.3, U34.12
- net at U96.3 (2): now also U110.4
- net at U96.5 (4): now also U110.5
- net at U90.6: now also U81.2
- net at U37.10 (CET): now also U44.9
- net at U37.11 (Q3): now also U44.5
- net at U37.12 (Q2): now also U44.4
- net at U37.9 (~{PE}): now also U44.8
- net at U66.5: now also U73.6
- net at U66.6: now also U104.5, U72.12
- net at U29.1 (S): now also U36.13 (Q1)
- net at U95.8: now also U94.13
- net ~{TUNNEL&BRIDGE}: now reaches U95.9
- net at U104.10: now also U67.7 (Zb)
- net Vs/64: now reaches U47.10
- net Vs/64: now also U49.1 (CP)
- net at U47.9: now also U45.8
- net at U83.1 (S): now also U84.1 (S), U87.3
- net at U113.23 (A8): now also U110.8
- net at U104.4: now also U58.12, U80.10
- net at U104.6: now also U89.11
- net at U18.5 (Q): now also U7.3
- net at U18.7 (RCext): now also R16.1
- net at U10.5: now also U35.3 (C), U44.6, C7.1
- net at U43.12 (Zd): now also U36.6 (D3)
- net at U43.4 (Za): now also U36.3 (D0)
- net at U43.7 (Zb): now also U36.4 (D1)
- net at U43.9 (Zc): now also U36.5 (D2)
- net at U73.4: now also U40.6 (~{Q})
- net at U94.12: now also U87.2
- net at U49.6 (Q3): now also U45.10
- net E8: now reaches U22.12
- net E8: now also J2.8 (Pin_8), U27.2, U4.1
- net E1: now reaches J2.1 (Pin_1)
- net E11: now reaches J2.11 (Pin_11)
- net E12: now reaches J2.12 (Pin_12)
- net E13: now reaches J2.13 (Pin_13)
- net ACCE.D: now reaches J2.14 (Pin_14)
- net ACCE.D: now also U45.9
- net E15: now reaches J2.15 (Pin_15)
- net E16: now reaches J2.16 (Pin_16)
- net E17: now reaches J2.17 (Pin_17)
- net E19: now reaches J2.19 (Pin_19)
- net E2: now reaches J2.2 (Pin_2)
- net E20: now reaches J2.20 (Pin_20)
- net E21: now reaches J2.21 (Pin_21)
- net E22: now reaches J2.22 (Pin_22)
- net E3: now reaches J2.3 (Pin_3)
- net E4: now reaches J2.4 (Pin_4)
- net E5: now reaches J2.5 (Pin_5)
- net E6: now reaches J2.6 (Pin_6)
- net E9: now reaches J2.9 (Pin_9)
- net at U38.3 (C): now also U40.9 (Q)
- net at U119.1 (Ea): now also U119.15 (Eb), U89.8
- net at U81.5: now also U56.13, U87.8
- net at U81.6: now also U112.1 (Ea), U112.15 (Eb)
- net ~{GAME OVER}: now reaches U70.11
- net ~{GAME OVER}: now also U33.12
- net at U25.5 (Q): now also U32.4, U34.5
- net ~{EXPLO.}: now reaches U4.5
- net EA: now reaches U87.1
- net at U78.6: now also U82.13
- net at U112.7 (Za): now also U34.11
- net at U110.9: now also U110.6
- net at U117.2: now also U120.23 (A8)
- net T.P: now reaches U33.4
- net EXPLO renamed EK
- net ~{RESCUE} renamed ~{RESCUE(Bl)}
- net ~{RESCUE(Bl)}: no longer U27.2
- new net: U206.11 (C), U206.2 (D), U206.6 (~{Q})
- new net: U206.1 (~{R}), U206.13 (~{R})
- no-connect marks 27 -> 47
Other:
- moved on the sheet: C20, C24, U103, U104B, U104C, U104D, U105, U106, U10B, U110B, U110C, U110D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
