File: Video/Video.kicad_sch (KiCad schematic)
At the start: 188 parts, among them J1 Conn_02x22_Top_Bottom, J2 Conn_02x22_Top_Bottom, Q1 Q_NPN_BCE, U1 74LS07, U10 74LS32, U100 74LS161, U101 74LS20, U102 74LS161, U103 74LS161, U104 74LS32, U105 74LS153, U106 MB7137, U107 74LS161, U108 74LS161, U109 74LS107, U11 74LS157, U110 74LS00, U111 74LS157, U112 74LS153, U113 MB7137, U114 74LS06, U115 74LS10, U116 74LS107, U117 74LS06, U118 74LS161, U119 74LS153, U12 MB7137, U120 MB7137, U13 74LS30, U14 74LS20, U15 74LS09, U16 74LS00, U17 MB7137, U18 74LS123, U19 74LS12, U2 74LS147, U20 74LS157, U201 74LS393, U202 74LS157, U206 74LS74, U21 74LS11, U22 74LS06, U23 74LS86, U24 74LS42, U25 74LS74, U26 74LS20, U27 74LS30, U28 74LS86, U29 74LS157, U3 74LS04, U30 MB7137, U31 74LS74, U32 74LS21, U33 74LS30, U34 74LS02, U35 74LS74, U36 74LS161, U37 74LS161, U38 74LS74, U39 74LS32, U4 74LS30, U40 74LS74, U41 74LS151, U42 74LS10, U43 74LS157, U44 74LS10, U45 74LS00, U46 74LS193, U47 74LS08, U48 74LS151, U49 74LS393, U5 74LS157, U50 74LS157, U51 MB7137, U52 74LS08, U53 74LS153, U54 74LS42, U55 74LS10, U56 74LS00, U57 74LS107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

Commit message: schem
Parts:
- added C4: 1,5uF, Capacitor_THT:C_Disc_D3.0mm_W1.6mm_P2.50mm, symbol Device:C
- added J3: Conn_02x22_Top_Bottom, BoardEdge:EdgeD, symbol Connector_Generic:Conn_02x22_Top_Bottom
- C22: footprint Capacitor_THT:C_Disc_D3.0mm_W1.6mm_P2.50mm -> Capacitor_THT:C_Disc_D4.3mm_W1.9mm_P5.00mm
Connections:
- net E1 is gone; now on net COIN IN: J2.1 (Pin_1)
- net EXTEND is gone; now on net EB: U20.1 (S), U25.12 (D), U26.12, U34.2, U40.2 (D)
- net H4 is gone; now on net F8: U51.23 (A8), U71.1
- net H5 is gone; now on net F7: U42.2, U71.12
- net H6 is gone; now on net FH: U42.1, U71.4
- net Vs/16 is gone; now on net E19: U52.9, U71.10, U73.9
- net ~{BRIDGE (W)} is gone; now on net EH: U5.13 (I1d)
- net ~{BRIDGE Bu} is gone; now on net ~{BRIDGE (Bu)}: U5.6 (I1b)
- net ~{BRIDGE} is gone; now on net ~{BRIDGE (R)}: U44.1
- net ~{COIN IN} is gone; now on net ED: C20.1, U34.9, U64.23 (A8)
- net ~{DUMMY} is gone; now on net ~{DUMMY AREA}: U26.2, U26.8, U27.1, U55.12, U59.3, U66.1
- net ~{EX.SIGNAL} is gone; now on net F1: U72.4
- net ~{EXPLO.} is gone; now on net E4: U4.5
- net ~{EXTEND} is gone; now on net E3: U10.10, U49.2 (MR)
- net ~{GAME} is gone; now on net E6: U55.3, U73.10
- net ~{LIGHT} is gone; now on net EC: U15.2, U19.3
- net ~{OTHER CAR} is gone; now on net E15: U21.13, U8.1
- net ~{OTHER TIRE} is gone; now on net E5: U27.11
- net ~{PLAYER TIRE} is gone; now on net E17: U27.5
- net ~{TUNNEL} is gone; now on net ~{TUNNEL&BRIDGE}: U31.8 (~{Q}), U34.4, U38.12 (D), U80.11
- net AREA 3: now also J3.9 (Pin_9)
- net AREA 4: now also J3.10 (Pin_10)
- net AREA 5: now also J3.11 (Pin_11)
- net E16: now also U59.6
- net E18: now also U30.23 (A8)
- net E20: now also U94.2
- net E8: no longer U27.2
- net EA: now also J2.23 (Pin_23)
- net EXT.500: now also U25.2 (D), U25.9 (Q); no longer U25.8 (~{Q})
- net GNDPWR: now also U20.15 (E), U46.1 (B), U46.10 (C), U46.15 (A), U46.9 (D), U53.6 (I0a), U99.20 (~{CE}1_(PVCE)); no longer U120.21 (A10)
- net H7: now also U107.11 (Q3)
- net H8: now also U53.1 (Ea)
- net S-100-D: no longer RN1.4 (R3)
- net TUNNEL AP: now also U68.7 (Q), U73.13, U73.3, U80.12, U80.3
- net V0: now also U102.14 (Q0)
- net V1: now also U102.13 (Q1)
- net V2: now also U102.12 (Q2)
- net V3: now also U102.11 (Q3), U114.13
- net V4: now also U100.14 (Q0), U101.9, U93.1; no longer U73.8
- net V5: now also U100.13 (Q1), U101.10, U93.3
- net V6: now also U100.12 (Q2), U101.12, U93.5
- net V7: now also U100.11 (Q3), U101.13, U52.12, U93.9
- net VCC: now also U120.19 (CE3), U52.13, U53.4 (I2a)
- net ~{BRIDGE (DBu)}: now also U6.5 (4)
- net ~{BRIDGE (Y)}: now also U6.3 (2)
- net ~{EXT.500}: now also U25.8 (~{Q}); no longer U25.2 (D), U25.9 (Q)
- net ~{H5}: now also U114.10, U115.3
- net ~{SLIP}: now also U59.12
- net ~{TV-BLANKING}: now also U101.6
- net ~{V4}: now also U93.2
- net at R16.1, U18.7 (RCext): now also C4.1
- net ~{0-AREA}: now reaches U66.4, U82.10
- net ~{0-AREA}: now also U10.13
- net FH: now reaches U53.11 (I1b)
- net FH: now also U107.12 (Q2), U114.9, U115.4, U39.9, U53.12 (I2b)
- net at U53.13 (I3b): now also U39.8
- net at U53.14 (S0): now also U46.3 (QA), U52.2
- net at U53.2 (S1): now also U46.2 (QB), U52.1
- net F7: now reaches U53.5 (I1a)
- net F7: now also U107.13 (Q1), U114.11, U39.10, J3.7 (Pin_7)
- net FD: now reaches U81.11
- net FD: now also U87.13, U88.11 (C)
- net at U201.13 (CP), U201.6 (Q3): now also U120.21 (A10)
- net at U66.9: now also U73.8
- net ~{M-ROAD}: now reaches U88.8 (~{Q}), U94.10
- net ~{M-ROAD}: now also U73.2, U73.5
- net at U59.13: now also U73.12
- net F2: now reaches U114.8
- net F2: now also J3.2 (Pin_2)
- net at U16.1: now also U23.12, U23.2, U23.5, U23.9, U28.1, U28.5, U52.11
- net F4: now reaches U16.3
- net F4: now also J3.4 (Pin_4)
- net ~{V5}: now reaches U93.4
- net FC: now reaches U88.13 (~{R})
- net FC: now also U81.3, U87.12
- net at U101.8: now also U101.5
- net at U119.9 (Zb), U58.13, U72.13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: no longer U119.7 (Za), U58.11, U60.11, U72.9
- net at U100.3 (D0): now also U100.4 (D1), U100.5 (D2), U100.6 (D3)
- net at U31.12 (D), U31.6 (~{Q}): now also U73.1
- net at U46.11 (~{LOAD}): now also U59.2
- net at U46.13 (~{BO}): now also U59.5
- net ED: now reaches U46.14 (CLR)
- net ED: now also J2.26 (Pin_26)
- net at U46.5 (UP): now also U39.6
- net ~{BRIDGE (Bu)}: now reaches U6.1 (0)
- net ~{BRIDGE (R)}: now reaches U6.2 (1)
- net EH: now reaches U6.6 (5)
- net EH: now also J2.30 (Pin_30)
- net F5: now reaches U16.11
- net F5: now also J3.5 (Pin_5)
- net ~{V7}: now reaches U16.12
- net ~{V7}: now also U93.8
- net at U96.6 (5): now also U95.5; no longer U95.4
- net at U96.7 (6): now also U95.4; no longer U95.5
- net at U52.3: now also U39.4
- net at U18.6 (Cext): now also C4.2
- net EW: now reaches U94.1
- net EB: now reaches J2.24 (Pin_24)
- net EC: now reaches J2.25 (Pin_25)
- net EE: now reaches J2.27 (Pin_27)
- net EF: now reaches J2.28 (Pin_28)
- net EG: now reaches J2.29 (Pin_29)
- net at U38.3 (C), U40.9 (Q): now also U201.1 (CP)
- net at U56.13, U81.5, U87.8: now also U81.10
- net at U115.6: now also U95.2
- net ~{HOUSE (R)}: now reaches U97.2 (1)
- net ~{HOUSE (R)}: now also U44.13
- net ~{HOUSE (Mu)}: now reaches U97.3 (2)
- net ~{HOUSE (Mu)}: now also U58.9
- net ~{HOUSE (St)}: now reaches U97.4 (3)
- net ~{HOUSE (St)}: now also U14.13
- net ~{HOUSE (W)}: now reaches U97.5 (4)
- net ~{HOUSE (W)}: now also U27.12
- net at U25.6 (~{Q}): now also U80.2
- net IC204_5: now reaches U201.5 (Q2)
- net ~{GRASS}: now reaches U20.11 (I0c)
- net at U94.4: now also U87.11
- net at U94.6: now also U80.9
- net EM: now reaches U59.1
- net F8: now reaches U107.14 (Q0)
- net F8: now also J3.8 (Pin_8)
- net at U118.10 (CET): now also U118.7 (CEP)
- net F1: now reaches U39.5
- net F1: now also J3.1 (Pin_1)
- net ~{V6}: now reaches U93.6
- net ~{EXPLO. AREA} renamed F15
- net F15: now also J3.15 (Pin_15)
- removed net ~{HOUSE}: U14.13, U27.12, U44.13, U58.9
- net ~{OTHER BODY} renamed ER
- net ~{RESCUE(Bc)} renamed ~{RESCUE (Bc)}
- net ~{RESCUE(Bl)} renamed ~{RESCUE (Bl)}
- net ~{RESCUE(R)} renamed ~{RESCUE (R)}
- net ~{RESCUE(W)} renamed ~{RESCUE (W)}
- net ~{RESCUE (W)}: now also U27.2
- new net: U58.11, U60.11
- new net: U119.7 (Za), U72.9
- new net F12: J3.12 (Pin_12)
- new net F13: J3.13 (Pin_13)
- new net F14: J3.14 (Pin_14)
- new net F16: J3.16 (Pin_16)
- new net F17: J3.17 (Pin_17)
- new net F18: J3.18 (Pin_18)
- new net F19: J3.19 (Pin_19)
- new net F20: J3.20 (Pin_20)
- new net F21: J3.21 (Pin_21)
- new net F22: J3.22 (Pin_22)
- new net F3: J3.3 (Pin_3)
- new net F6: J3.6 (Pin_6)
- no-connect marks 47 -> 59
Other:
- moved on the sheet: R16, U101A, U101B, U101C, U102, U107, U114A, U114B, U114C, U114D, U114E, U114F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

Commit message: vor
Parts:
- removed RN1: 560, Resistor_THT:R_Array_SIP9, symbol Device:R_Network08_US
- added C1: 470p, Capacitor_THT:C_Disc_D3.0mm_W1.6mm_P2.50mm, symbol Device:C_Polarized_US
- added C13, C14, C8: 470p, Capacitor_THT:C_Disc_D4.3mm_W1.9mm_P5.00mm, symbol Device:C
- added C18, C9, C998: 470p, Capacitor_THT:C_Disc_D3.0mm_W1.6mm_P2.50mm, symbol Device:C
- added R2077: 470, Resistor_THT:R_Axial_DIN0204_L3.6mm_D1.6mm_P7.62mm_Horizontal, symbol Device:R
- added RN2: 560, Resistor_THT:R_Array_SIP9, symbol Device:R_Network08_Split
Connections:
- net 7M is gone; now on net 7MHz: U103.2 (CP), U118.2 (CP), U14.4, U79.9 (Cp)
- net D6 is gone; now on net 14MHz_EXT: J1.6 (Pin_6)
- net F1 is gone; now on net E2: J3.1 (Pin_1), U39.5, U72.4
- net F13 is gone; now on net 7MHz: J3.13 (Pin_13)
- net F18 is gone; now on net BRIDGE AP: J3.18 (Pin_18)
- net H8 is gone; now on net FF: U53.1 (Ea), U55.4, U64.1 (A7)
- net Vs/64 is gone; now on net EV: U47.10, U49.1 (CP)
- net ~{CAR NO CONT} is gone; now on net F3: U59.9
- net ~{H8} is gone; now on net FB: U42.13, U71.9
- net ~{Hs} is gone; now on net FJ: U35.2 (D), U47.2, U76.2 (CP), U77.2 (CP), U85.2 (CP), U91.2 (CP)
- net ~{M.ROAD} is gone; now on net ~{M-ROAD}: U58.2
- net ~{TUNNEL&BRIDGE} is gone; now on net EF: U31.8 (~{Q}), U34.4, U38.12 (D), U80.11, U95.9
- net ~{Vb} is gone; now on net FN: U74.2 (D), U85.10 (CET), U88.12 (D), U91.10 (CET)
- net AREA 1: now also J3.32 (Pin_32)
- net AREA 2: now also J3.31 (Pin_31)
- net D10: now also RN2.2 (R1.2)
- net D14: now also U202.13 (I1d), RN2.3 (R2.2)
- net D15: now also U202.10 (I1c), RN2.4 (R3.2)
- net D16: now also U202.6 (I1b), RN2.7 (R6.2)
- net D17: now also U202.3 (I1a), RN2.8 (R7.2)
- net D7: now also U1.10
- net D8: now also U1.12
- net E5: no longer U27.11
- net E9: no longer U26.4
- net EG: now also U5.13 (I1d), U6.6 (5)
- net EH: no longer U5.13 (I1d), U6.6 (5)
- net F12: now also U115.12, U28.10, C8.1
- net F16: now also U111.2 (I0a)
- net F17: now also U110.13, U111.11 (I0c)
- net F3: now also U24.6 (5), U25.3 (C)
- net F7: now also U1.13
- net FH: now also J3.29 (Pin_29)
- net GNDPWR: now also U102.3 (D0), U102.4 (D1), U106.20 (~{CE}1_(PVCE)), U107.5 (D2), U108.3 (D0), U108.4 (D1), U202.15 (E), U41.7 (~{E}), U43.10 (I1c), U43.15 (E), U43.2 (I0a), U48.7 (~{E}), C1.2, C13.2, C14.2, C18.1, C8.2, C9.2, C998.2
- net H0: now also U108.14 (Q0)
- net H1: now also U108.13 (Q1)
- net H2: now also U108.12 (Q2)
- net H3: now also U108.11 (Q3)
- net MH8: now also U55.11, U57.3 (Q)
- net TUNNEL AP: no longer U68.7 (Q), U73.13, U73.3, U80.12, U80.3, U80.5
- net V-2: now also U54.3 (2), U61.3, U68.15 (~{S})
- net V-4: now also U54.5 (4), U58.4, U65.3
- net V-CA: now also U100.15 (TC), U109.12 (C), U110.1, U93.13, C998.1
- net V2: now also U1.11, U115.1
- net V4: now also U26.13
- net VCC: now also J1.41 (Pin_41), J1.42 (Pin_42), J1.43 (Pin_43), J1.44 (Pin_44), U100.7 (CEP), U111.10 (I1c), U116.13 (~{R}), U118.10 (CET), U118.7 (CEP), R2077.2, RN2.1 (R1), RN2.1 (R1), RN2.1 (R1), RN2.1 (R1), RN2.1 (R1), RN2.1 (R1), RN2.1 (R1), RN2.1 (R1)
- net Vb: now also U114.4
- net ~{DUMMY AREA}: no longer U26.2, U27.1, U55.12
- net ~{GRASS}: now also U22.4
- net ~{HOUSE ST}: now also U81.8, U98.15 (E)
- net ~{ROAD}: now also C1.1
- net ~{SYNCRO}: now also U28.8
- net ~{Y-LINE}: now also U87.11, U94.4
- net V-1: now reaches U54.2 (1), U61.13
- net V-1: now also U53.15 (Eb)
- net V-3: now reaches U54.4 (3)
- net V-3: now also U15.12, U60.2
- net V-5: now reaches U54.6 (5), U70.2
- net V-5: now also U15.13
- net at U42.6, U43.1 (S): now also C9.1
- net FS: now reaches U111.1 (S)
- net FS: now also U110.3
- net FU: now reaches U110.12, U111.14 (I0d)
- net FT: now reaches U111.5 (I0b)
- net at U53.7 (Za): now also U26.10
- net at U53.9 (Zb): now also U26.9
- net ~{MHL0}: now reaches U48.3 (I1)
- net ~{MHL0}: now also U40.11 (C), U41.12 (I7)
- net at U201.10 (Q1): now also U202.5 (I0b)
- net at U201.11 (Q0): now also U202.2 (I0a)
- net at U201.12 (MR), U201.2 (MR): now also U202.1 (S)
- net at U201.8 (Q3): now also U202.14 (I0d)
- net at U201.9 (Q2): now also U202.11 (I0c)
- net at D1.1 (K), D2.1 (K), D3.1 (K)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: now also RN2.5 (R4.2)
- net at Q1.3 (B), U7.2: now also RN2.6 (R5.2)
- net at U114.3: now also U100.3 (D0), U100.4 (D1), U100.5 (D2), U100.6 (D3), U109.2 (~{Q})
- net SLIP: now reaches U59.13, U73.12
- net FF: now reaches U116.10 (~{R}), U116.8 (J)
- net FF: now also U101.1, U102.6 (D3), U109.3 (Q), U110.2, U114.1, U115.10, U115.2, U116.11 (K), U116.3 (Q)
- net at U116.5 (Q): now also U101.4, U107.3 (D0), U108.6 (D3), U115.5, U116.4 (K)
- net at U116.6 (~{Q}): now also U107.4 (D1), U116.1 (J)
- net at U116.9 (C): now also U107.15 (TC), U115.9, U116.12 (C)
- net at U10.12: now also U15.11
- net at U28.9: now also U100.2 (CP), U102.2 (CP), U115.6, U95.2
- net ~{DUMMY (W)}: now reaches U55.1, U56.6
- net ~{DUMMY (W)}: now also U27.1
- net ~{DUMMY (R)}: now reaches U55.13, U56.8
- net at U114.12: now also U115.13
- net at U58.13, U72.13, U72.2: now also U119.7 (Za); no longer U119.9 (Zb)
- net FN: now reaches U114.2
- net FN: now also J3.34 (Pin_34)
- net at U100.10 (CET): now also U102.15 (TC)
- net at U100.9 (~{PE}): now also U102.9 (~{PE}), U93.12, C13.1
- net FJ: now reaches J3.30 (Pin_30)
- net FJ: now also U95.3
- net FM: now reaches J3.33 (Pin_33)
- net at U115.11: now also U107.7 (CEP), U108.15 (TC)
- net at U115.8: now also U107.9 (~{PE}), U108.9 (~{PE}), C14.1
- net at U46.11 (~{LOAD}): no longer U59.2
- net at U46.4 (DOWN): now also U59.2
- net at U72.9: now also U119.9 (Zb); no longer U119.7 (Za)
- net at U37.10 (CET), U44.9: now also U36.15 (TC)
- net 7MHz: now reaches U37.2 (CP)
- net 7MHz: now also U107.2 (CP), U108.2 (CP), U109.6 (~{Q}), U117.6, U36.2 (CP)
- net at U37.9 (~{PE}), U44.8: now also U36.9 (~{PE}), C18.2
- net at U56.1: now also U68.7 (Q), U73.13, U73.3, U80.12, U80.3, U80.5
- net 14MHz: now reaches U109.9 (C), U117.12
- net 14MHz: now also U1.9
- net ES: now reaches J2.37 (Pin_37)
- net ES: now also U27.11
- net ET: now reaches J2.38 (Pin_38)
- net EU: now reaches J2.39 (Pin_39)
- net EU: now also U26.4
- net EV: now reaches J2.40 (Pin_40)
- net FB: now reaches U116.2 (~{Q})
- net EXT. 500: now reaches U15.9
- net 14MHz_EXT: now reaches U1.8
- net 14MHz_EXT: now also R2077.1
- new net ~{DUMMY (BL)}: U26.2, U55.12
- no-connect marks 59 -> 92
Other:
- moved on the sheet: C16, C17, R17, R18, U100, U101A, U101B, U102, U104E, U108, U109A, U109B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

Commit message: almost done
Parts:
- added C19, C333, C5: 470p, Capacitor_THT:C_Disc_D3.0mm_W1.6mm_P2.50mm, symbol Device:C
- added C2: 470p, Capacitor_THT:C_Disc_D4.3mm_W1.9mm_P5.00mm, symbol Device:C
- added TP1: TestPoint, TestPoint:TestPoint_Loop_D2.60mm_Drill0.9mm_Beaded, symbol Connector:TestPoint
- added U203, U205: 74LS157, Package_DIP:DIP-16_W7.62mm, symbol 74xx:74LS157
Connections:
- net 100-C is gone; now on net S-100-D: U35.12 (D)
- net DUMMY is gone; now on net ~{DUMMY (R)}: U33.2
- net F20 is gone; now on net VCC: J3.20 (Pin_20)
- net F21 is gone; now on net VCC: J3.21 (Pin_21)
- net F22 is gone; now on net VCC: J3.22 (Pin_22)
- net M2V8 is gone; now on net M2V3: U78.13
- net RESCUE is gone; now on net ~{RESCUE (R)}: U33.1
- net V-(H) is gone; now on net V-4: U9.4
- net V4 is gone; now on net E21: U100.14 (Q0), U101.9, U26.13, U28.2, U51.4 (A4), U61.1, U64.5 (A3), U93.1
- net V6 is gone; now on net E12: U100.12 (Q2), U101.12, U28.4, U54.14 (A1), U64.3 (A5), U93.5
- net V7 is gone; now on net EN: U100.11 (Q3), U101.13, U104.1, U52.12, U54.13 (A2), U93.9
- net ~{EXT.500} is gone; now on net EJ: U25.8 (~{Q}), U65.2
- net ~{POOL} is gone; now on net FM: U14.12, U72.8
- net ~{RESCUE (Bc)} is gone; now on net F14: U15.5
- net ~{RESCUE (Bl)} is gone; now on net ~{RESCUE (BL)}: U22.10
- net ~{SIG} is gone; now on net ~{SIG. (BL)}: U26.1
- net ~{SLIDE} is gone; now on net FR: U65.4
- net ~{SLIP} is gone; now on net FA: U14.9, U59.12
- net ~{TREE&GRASS} is gone; now on net ~{TREE&GRASS (G)}: U20.2 (I0a), U20.6 (I1b), U21.5
- net ~{V5} is gone; now on net EY: U93.4
- net ~{V6} is gone; now on net E22: U93.6
- net ~{V7} is gone; now on net EZ: U16.12, U93.8
- net D9: now also U7.4
- net E18: no longer U30.23 (A8)
- net E3: now also U203.6 (I1b); no longer U10.10, U49.2 (MR)
- net E6: now also U203.10 (I1c)
- net E7: no longer U33.6
- net EB: now also U203.3 (I1a); no longer U20.1 (S), U25.12 (D), U26.12, U34.2, U40.2 (D)
- net ED: now also U206.1 (~{R}), U206.13 (~{R})
- net EK: now also J2.31 (Pin_31)
- net ER: now also J2.36 (Pin_36)
- net ET: now also U33.6
- net EW: now also J2.41 (Pin_41), U30.23 (A8)
- net EX: now also J2.42 (Pin_42)
- net F14: now also U72.11
- net F16: now also U205.3 (I1a); no longer U111.2 (I0a)
- net F17: now also U205.10 (I1c); no longer U110.13, U111.11 (I0c)
- net FB: now also J3.24 (Pin_24)
- net FC: now also J3.25 (Pin_25)
- net FD: now also J3.26 (Pin_26)
- net FF: now also J3.28 (Pin_28)
- net FS: now also J3.37 (Pin_37)
- net FT: now also J3.38 (Pin_38), U205.6 (I1b); no longer U111.5 (I0b)
- net FU: now also J3.39 (Pin_39), U205.13 (I1d); no longer U110.12, U111.14 (I0d)
- net GNDPWR: now also J1.32 (Pin_32), U113.20 (~{CE}1_(PVCE)), U37.5 (D2), C19.2, C2.2, C333.2, C5.2, U203.15 (E), U203.5 (I0b), U203.8 (GND), U205.11 (I0c), U205.15 (E), U205.2 (I0a), U205.5 (I0b), U205.8 (GND)
- net TUNNEL AP: now also U80.5
- net V-CA: now also C2.1
- net VCC: now also U30.18 (CE2), U30.19 (CE3), U37.4 (D1), U37.7 (CEP), U203.16 (VCC), U205.16 (VCC)
- net ~{DUMMY AREA}: now also C5.1
- net ~{MHL0}: now also U103.9 (~{PE}), U118.9 (~{PE}), U55.8
- net ~{SIDE LINE}: now also U104.8
- net at U56.1, U68.7 (Q), U73.13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: no longer U80.5
- net ~{SIG. (BL)}: now reaches U9.11
- net at U201.12 (MR), U201.2 (MR), U202.1 (S): now also U206.8 (~{Q}), U203.1 (S), U203.11 (I0c), U205.1 (S)
- net at U201.13 (CP), U201.6 (Q3): no longer U120.21 (A10)
- net at U201.8 (Q3): now also U203.2 (I0a); no longer U202.14 (I0d)
- net ~{TREE&GRASS (BL)}: now reaches U13.2, U19.11, U20.13 (I1d)
- net ~{TREE&GRASS (BL)}: now also U34.13
- net at U100.2 (CP), U102.2 (CP), U115.6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: now also C19.1
- net FA: now reaches J3.23 (Pin_23)
- net FE: now reaches J3.27 (Pin_27)
- net FE: now also U10.4, U59.10
- net FR: now reaches J3.36 (Pin_36)
- net FV: now reaches J3.40 (Pin_40)
- net FW: now reaches J3.41 (Pin_41)
- net FX: now reaches J3.42 (Pin_42)
- net FY: now reaches J3.43 (Pin_43)
- net FZ: now reaches J3.44 (Pin_44)
- net ~{TREE&GRASS (G)}: now reaches U60.8
- net at U58.6, U65.6: now also C333.1
- net EN: now reaches J2.34 (Pin_34)
- net EY: now reaches J2.43 (Pin_43)
- net EZ: now reaches J2.44 (Pin_44)
- net DF: now reaches J1.28 (Pin_28)
- net DM: now reaches J1.33 (Pin_33)
- net EH renamed EJ
- net FH renamed FG
- net SIG renamed ~{SIG. (Y)}
- net T.P: no longer names the net of U33.4
- net T.P: now also TP1.1
- net ~{GRAVEL} renamed ~{RESCUE (BL)}
- net ~{RESCUE (BL)}: no longer U72.11
- new net EXTEND: U20.1 (S), U203.4 (Za), U25.12 (D), U26.12, U34.2, U40.2 (D)
- new net SP.A: U111.2 (I0a), U205.4 (Za)
- new net SP.B: U111.5 (I0b), U205.7 (Zb)
- new net SP.C: U110.13, U111.11 (I0c), U205.9 (Zc)
- new net SP.D: U110.12, U111.14 (I0d), U205.12 (Zd)
- new net ~{EXTEND}: U10.10, U203.7 (Zb), U49.2 (MR)
- no-connect marks 92 -> 97
Other:
- note added: "TV-GND"
- moved on the sheet: J1, J2, RN2H, U206A, U206B, U206C
