File: Video/Video.kicad_sch (KiCad schematic)
At the start: 205 parts, among them J1 Conn_02x22_Top_Bottom, J2 Conn_02x22_Top_Bottom, J3 Conn_02x22_Top_Bottom, Q1 Q_NPN_BCE, U1 74LS07, U10 74LS32, U100 74LS161, U101 74LS20, U102 74LS161, U103 74LS161, U104 74LS32, U105 74LS153, U106 MB7137, U107 74LS161, U108 74LS161, U109 74LS107, U11 74LS157, U110 74LS00, U111 74LS157, U112 74LS153, U113 MB7137, U114 74LS06, U115 74LS10, U116 74LS107, U117 74LS06, U118 74LS161, U119 74LS153, U12 MB7137, U120 MB7137, U13 74LS30, U14 74LS20, U15 74LS09, U16 74LS00, U17 MB7137, U18 74LS123, U19 74LS12, U2 74LS147, U20 74LS157, U201 74LS393, U202 74LS157, U203 74LS157, U205 74LS157, U206 74LS74, U21 74LS11, U22 74LS06, U23 74LS86, U24 74LS42, U25 74LS74, U26 74LS20, U27 74LS30, U28 74LS86, U29 74LS157, U3 74LS04, U30 MB7137, U31 74LS74, U32 74LS21, U33 74LS30, U34 74LS02, U35 74LS74, U36 74LS161, U37 74LS161, U38 74LS74, U39 74LS32, U4 74LS30, U40 74LS74, U41 74LS151, U42 74LS10, U43 74LS157, U44 74LS10, U45 74LS00, U46 74LS193, U47 74LS08, U48 74LS151, U49 74LS393, U5 74LS157, U50 74LS157, U51 MB7137, U52 74LS08, U53 74LS153, U54 74LS42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

Commit message: finish video
Parts:
- added C12, C25: 470p, Capacitor_THT:C_Disc_D3.0mm_W1.6mm_P2.50mm, symbol Device:C
- added U204: 74LS86, Package_DIP:DIP-14_W7.62mm, symbol 74xx:74LS86
- renumbered C25 to C26
Connections:
- net EXT.500 is gone; now on net EXT. 500: U25.2 (D), U25.9 (Q)
- net FV is gone; now on net 14MHz: J3.40 (Pin_40)
- net ED: now also U203.9 (Zc)
- net F19: now also U206.3 (C)
- net GNDPWR: now also U103.6 (D3), C12.2, C25.2, U204.7 (GND); no longer U203.5 (I0b)
- net VCC: now also U17.18 (CE2), U204.14 (VCC)
- net ~{GREEN BELT}: now also U80.8, U94.8
- net ~{M1VL0}: now also C12.1
- net at U205.14 (I0d): now also U204.11
- net at U201.13 (CP), U201.6 (Q3): now also U204.4
- net at U201.8 (Q3), U203.2 (I0a): now also U204.9
- net at U12.19 (CE3), U17.20 (~{CE}1_(PVCE)): now also U10.11, U12.18 (CE2), U17.21 (A10)
- net at U202.14 (I0d): now also C25.1, U204.3
- net at U30.21 (A10): now also U204.5
- net at U32.6, U49.12 (MR): now also U204.12
- new net: U204.1, U204.10, U204.13
- new net: U204.2, U204.6
- new net: U203.5 (I0b), U204.8
- no-connect marks 97 -> 127
Other:
- moved on the sheet: U55D

Commit message: netlists
Parts:
- Cp1, Cp10, Cp11, Cp12, Cp13, Cp14, Cp15, Cp16, Cp17, Cp18, Cp19, Cp2, Cp20, Cp21, Cp22, Cp23, Cp24, Cp25, Cp26, Cp27, Cp28, Cp29, Cp3, Cp30, Cp31, Cp32, Cp33, Cp34, Cp35, Cp36, Cp4, Cp5, Cp6, Cp7, Cp8, Cp9: value C -> 100n
- renumbered RN2 to RN1
Connections:
- net EM: now also J2.33 (Pin_33)
- net EL: now reaches J2.32 (Pin_32)
- net DG: now reaches J1.29 (Pin_29)
- net DJ: now reaches J1.30 (Pin_30)
- net DK: now reaches J1.31 (Pin_31)
- net DN: now reaches J1.34 (Pin_34)
- net DR: now reaches J1.36 (Pin_36)
- net DS: now reaches J1.37 (Pin_37)
- net DT: now reaches J1.38 (Pin_38)
- net DU: now reaches J1.39 (Pin_39)
- net DV: now reaches J1.40 (Pin_40)
- no-connect marks 127 -> 141
